File: hardware/GFC/GFC/1-Wire_Connection.kicad_sch (KiCad schematic)
At the start: 3 parts

Commit message: sync
Parts:
- added TP44, TP45: Test Point, TestPoint:TestPoint_Pad_D1.0mm, symbol Connector:TestPoint_Small
Connections:
- net +3V3 renamed VCC
- net VCC: now also TP45.1
- net 1-Wire BUS 0 renamed 1-Wire
- net 1-Wire: now also TP44.1
Changed lines of the file:
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@@
 (kicad_sch (version 20211123) (generator eeschema)
   (paper "A4")
+  (junction (at 140.97 92.71) (diameter 0) (color 0 0 0 0)
+  )
   (junction (at 114.3 88.9) (diameter 0) (color 0 0 0 0)
+  )
+  (junction (at 109.22 88.9) (diameter 0) (color 0 0 0 0)
+  )
+  (junction (at 109.22 92.71) (diameter 0) (color 0 0 0 0)
+  )
+  (junction (at 116.84 92.71) (diameter 0) (color 0 0 0 0)
   )
   (junction (at 138.43 88.9) (diameter 0) (color 0 0 0 0)
@@
     (stroke (width 0) (type default) (color 0 0 0 0))
   )
+  (wire (pts (xy 140.97 92.71) (xy 140.97 83.82))
+    (stroke (width 0) (type default) (color 0 0 0 0))
+  )
   (wire (pts (xy 106.68 83.82) (xy 106.68 81.28))
     (stroke (width 0) (type default) (color 0 0 0 0))
   )
-  (wire (pts (xy 146.05 81.28) (xy 146.05 83.82))
+  (wire (pts (xy 109.22 88.9) (xy 114.3 88.9))
     (stroke (width 0) (type default) (color 0 0 0 0))
   )
@@
     (stroke (width 0) (type default) (color 0 0 0 0))
   )
+  (wire (pts (xy 140.97 92.71) (xy 166.37 92.71))
+    (stroke (width 0) (type default) (color 0 0 0 0))
+  )
+  (wire (pts (xy 109.22 92.71) (xy 116.84 92.71))
+    (stroke (width 0) (type default) (color 0 0 0 0))
+  )
   (wire (pts (xy 163.83 83.82) (xy 163.83 88.9))
     (stroke (width 0) (type default) (color 0 0 0 0))
   )
-  (wire (pts (xy 116.84 83.82) (xy 121.92 83.82))
+  (wire (pts (xy 116.84 92.71) (xy 140.97 92.71))
     (stroke (width 0) (type default) (color 0 0 0 0))
   )
@@
     (stroke (width 0) (type default) (color 0 0 0 0))
   )
-  (wire (pts (xy 166.37 83.82) (xy 171.45 83.82))
-    (stroke (width 0) (type default) (color 0 0 0 0))
-  )
-  (wire (pts (xy 121.92 81.28) (xy 121.92 83.82))
-    (stroke (width 0) (type default) (color 0 0 0 0))
-  )
-  (wire (pts (xy 171.45 81.28) (xy 171.45 83.82))
+  (wire (pts (xy 105.41 92.71) (xy 109.22 92.71))
     (stroke (width 0) (type default) (color 0 0 0 0))
   )
@@
     (stroke (width 0) (type default) (color 0 0 0 0))
   )
+  (wire (pts (xy 166.37 92.71) (xy 166.37 83.82))
+    (stroke (width 0) (type default) (color 0 0 0 0))
+  )
   (wire (pts (xy 106.68 83.82) (xy 111.76 83.82))
     (stroke (width 0) (type default) (color 0 0 0 0))
@@
     (stroke (width 0) (type default) (color 0 0 0 0))
   )
-  (wire (pts (xy 140.97 83.82) (xy 146.05 83.82))
+  (wire (pts (xy 116.84 92.71) (xy 116.84 83.82))
     (stroke (width 0) (type default) (color 0 0 0 0))
   )
-  (wire (pts (xy 105.41 88.9) (xy 114.3 88.9))
+  (wire (pts (xy 105.41 88.9) (xy 109.22 88.9))
     (stroke (width 0) (type default) (color 0 0 0 0))
   )
@@
     (stroke (width 0) (type default) (color 0 0 0 0))
   )
-  (global_label "1-Wire BUS 0" (shape input) (at 105.41 88.9 180) (fields_autoplaced)
+  (hierarchical_label "1-Wire" (shape input) (at 105.41 88.9 180)
     (effects (font (size 1.27 1.27)) (justify right))
-    (property "Intersheet References" "${INTERSHEET_REFS}" (id 0) (at 89.3293 88.8206 0)
-      (effects (font (size 1.27 1.27)) (justify right) hide)
+  )
+  (hierarchical_label "VCC" (shape input) (at 105.41 92.71 180)
+    (effects (font (size 1.27 1.27)) (justify right))
+  )
+  (symbol (lib_id "Connector:TestPoint_Small") (at 109.22 92.71 0) (mirror y) (unit 1)
+    (in_bom yes) (on_board yes)
+    (property "Reference" "TP45" (id 0) (at 113.03 91.44 0)
+      (effects (font (size 1.27 1.27)) (justify left))
     )
+    (property "Value" "Test Point" (id 1) (at 107.95 93.9799 0)
+      (effects (font (size 1.27 1.27)) (justify left) hide)
+    )
+    (property "Footprint" "TestPoint:TestPoint_Pad_D1.0mm" (id 2) (at 104.14 92.71 0)
+      (effects (font (size 1.27 1.27)) hide)
+    )
+    (property "Datasheet" "~" (id 3) (at 104.14 92.71 0)
+      (effects (font (size 1.27 1.27)) hide)
+    )
+    (pin "1")
   )
   (symbol (lib_id "Connector_Generic:Conn_01x03") (at 163.83 78.74 90) (unit 1)
@@
     (pin "3")
   )
-  (symbol (lib_id "power:+3V3") (at 146.05 81.28 0) (unit 1)
-    (in_bom yes) (on_board yes) (fields_autoplaced)
-    (property "Reference" "#PWR0124" (id 0) (at 146.05 85.09 0)
+  (symbol (lib_id "Connector:TestPoint_Small") (at 109.22 88.9 0) (mirror y) (unit 1)
+    (in_bom yes) (on_board yes)
+    (property "Reference" "TP44" (id 0) (at 113.03 87.63 0)
+      (effects (font (size 1.27 1.27)) (justify left))
+    )
+    (property "Value" "Test Point" (id 1) (at 107.95 90.1699 0)
+      (effects (font (size 1.27 1.27)) (justify left) hide)
+    )
+    (property "Footprint" "TestPoint:TestPoint_Pad_D1.0mm" (id 2) (at 104.14 88.9 0)
       (effects (font (size 1.27 1.27)) hide)
     )
-    (property "Value" "+3V3" (id 1) (at 146.05 76.2 0))
-    (property "Footprint" "" (id 2) (at 146.05 81.28 0)
-      (effects (font (size 1.27 1.27)) hide)
-    )
-    (property "Datasheet" "" (id 3) (at 146.05 81.28 0)
-      (effects (font (size 1.27 1.27)) hide)
-    )
-    (pin "1")
-  )
-  (symbol (lib_id "power:+3V3") (at 171.45 81.28 0) (unit 1)
-    (in_bom yes) (on_board yes) (fields_autoplaced)
-    (property "Reference" "#PWR0158" (id 0) (at 171.45 85.09 0)
-      (effects (font (size 1.27 1.27)) hide)
-    )
-    (property "Value" "+3V3" (id 1) (at 171.45 76.2 0))
-    (property "Footprint" "" (id 2) (at 171.45 81.28 0)
-      (effects (font (size 1.27 1.27)) hide)
-    )
-    (property "Datasheet" "" (id 3) (at 171.45 81.28 0)
+    (property "Datasheet" "~" (id 3) (at 104.14 88.9 0)
       (effects (font (size 1.27 1.27)) hide)
     )
@@
       (effects (font (size 1.27 1.27)) hide)
     )
-    (pin "1")
-  )
-  (symbol (lib_id "power:+3V3") (at 121.92 81.28 0) (unit 1)
-    (in_bom yes) (on_board yes) (fields_autoplaced)
-    (property "Reference" "#PWR0156" (id 0) (at 121.92 85.09 0)
-      (effects (font (size 1.27 1.27)) hide)
-    )
-    (property "Value" "+3V3" (id 1) (at 121.92 76.2 0))
-    (property "Footprint" "" (id 2) (at 121.92 81.28 0)
-      (effects (font (size 1.27 1.27)) hide)
-    )
-    (property "Datasheet" "" (id 3) (at 121.92 81.28 0)
-      (effects (font (size 1.27 1.27)) hide)
-    )
