File: hardware/GFC/GFC/BMP390.kicad_sch (KiCad schematic)
At the start: 5 parts

Commit message: Sync board
Parts:
- C? (x2): value C -> 100nF
- R? (x2): value R -> 4.7k
Connections:
- net VDDIO is gone; now on net VCC: C?.1, R?.1, R?.2, U?.1 (VDDIO), U?.6 (~{CS})
- net VDD renamed VCC
Changed lines of the file:
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@@
   (junction (at 129.54 67.31) (diameter 0) (color 0 0 0 0)
   )
+  (junction (at 144.78 43.18) (diameter 0) (color 0 0 0 0)
+  )
   (junction (at 129.54 73.66) (diameter 0) (color 0 0 0 0)
   )
@@
   (junction (at 129.54 59.69) (diameter 0) (color 0 0 0 0)
   )
-  (junction (at 83.82 34.29) (diameter 0) (color 0 0 0 0)
+  (junction (at 100.33 27.94) (diameter 0) (color 0 0 0 0)
   )
   (junction (at 129.54 77.47) (diameter 0) (color 0 0 0 0)
@@
     (stroke (width 0) (type default) (color 0 0 0 0))
   )
+  (wire (pts (xy 100.33 27.94) (xy 144.78 27.94))
+    (stroke (width 0) (type default) (color 0 0 0 0))
+  )
   (wire (pts (xy 78.74 38.1) (xy 95.25 38.1))
     (stroke (width 0) (type default) (color 0 0 0 0))
   )
-  (wire (pts (xy 100.33 38.1) (xy 100.33 31.75))
+  (wire (pts (xy 100.33 25.4) (xy 100.33 27.94))
     (stroke (width 0) (type default) (color 0 0 0 0))
   )
@@
     (stroke (width 0) (type default) (color 0 0 0 0))
   )
+  (wire (pts (xy 144.78 43.18) (xy 144.78 27.94))
+    (stroke (width 0) (type default) (color 0 0 0 0))
+  )
   (wire (pts (xy 144.78 43.18) (xy 144.78 91.44))
     (stroke (width 0) (type default) (color 0 0 0 0))
@@
     (stroke (width 0) (type default) (color 0 0 0 0))
   )
-  (wire (pts (xy 95.25 31.75) (xy 95.25 38.1))
+  (wire (pts (xy 95.25 25.4) (xy 95.25 38.1))
     (stroke (width 0) (type default) (color 0 0 0 0))
   )
@@
     (stroke (width 0) (type default) (color 0 0 0 0))
   )
-  (wire (pts (xy 83.82 34.29) (xy 92.71 34.29))
-    (stroke (width 0) (type default) (color 0 0 0 0))
-  )
   (wire (pts (xy 72.39 34.29) (xy 83.82 34.29))
     (stroke (width 0) (type default) (color 0 0 0 0))
@@
     (stroke (width 0) (type default) (color 0 0 0 0))
   )
-  (wire (pts (xy 97.79 31.75) (xy 97.79 50.8))
+  (wire (pts (xy 97.79 25.4) (xy 97.79 50.8))
+    (stroke (width 0) (type default) (color 0 0 0 0))
+  )
+  (wire (pts (xy 100.33 27.94) (xy 100.33 38.1))
     (stroke (width 0) (type default) (color 0 0 0 0))
   )
@@
     (stroke (width 0) (type default) (color 0 0 0 0))
   )
-  (wire (pts (xy 92.71 34.29) (xy 92.71 31.75))
-    (stroke (width 0) (type default) (color 0 0 0 0))
-  )
-  (hierarchical_label "SCL" (shape input) (at 97.79 31.75 90)
+  (label "VDDIO" (at 102.87 27.94 0)
+    (effects (font (size 1.27 1.27)) (justify left bottom))
+  )
+  (label "VDD" (at 102.87 38.1 0)
+    (effects (font (size 1.27 1.27)) (justify left bottom))
+  )
+  (hierarchical_label "SCL" (shape input) (at 97.79 25.4 90)
     (effects (font (size 1.27 1.27)) (justify left))
   )
-  (hierarchical_label "VDD" (shape input) (at 100.33 31.75 90)
+  (hierarchical_label "VCC" (shape input) (at 100.33 25.4 90)
     (effects (font (size 1.27 1.27)) (justify left))
   )
-  (hierarchical_label "SDA" (shape input) (at 95.25 31.75 90)
+  (hierarchical_label "SDA" (shape input) (at 95.25 25.4 90)
     (effects (font (size 1.27 1.27)) (justify left))
   )
-  (hierarchical_label "VDDIO" (shape input) (at 92.71 31.75 90)
-    (effects (font (size 1.27 1.27)) (justify left))
-  )
   (symbol (lib_id "Device:R") (at 72.39 60.96 0) (unit 1)
     (in_bom yes) (on_board yes) (fields_autoplaced)
@@
       (effects (font (size 1.27 1.27)) (justify left))
     )
-    (property "Value" "R" (id 1) (at 74.93 62.2299 0)
+    (property "Value" "4.7k" (id 1) (at 74.93 62.2299 0)
       (effects (font (size 1.27 1.27)) (justify left))
     )
@@
       (effects (font (size 1.27 1.27)) (justify left))
     )
-    (property "Value" "C" (id 1) (at 133.35 64.7699 0)
+    (property "Value" "100nF" (id 1) (at 133.35 64.7699 0)
       (effects (font (size 1.27 1.27)) (justify left))
     )
@@
     (in_bom yes) (on_board yes)
     (property "Reference" "R?" (id 0) (at 106.68 45.72 90))
-    (property "Value" "R" (id 1) (at 106.68 48.26 90))
+    (property "Value" "4.7k" (id 1) (at 106.68 48.26 90))
     (property "Footprint" "" (id 2) (at 106.68 52.578 90)
       (effects (font (size 1.27 1.27)) hide)
@@
       (effects (font (size 1.27 1.27)) (justify left))
     )
-    (property "Value" "C" (id 1) (at 87.63 52.0699 0)
-      (effects (font (size 1.27 1.27)) (justify left))
-    )
+    (property "Value" "100nF" (id 1) (at 87.63 52.0699 0)
+      (effects (font (size 1.27 1.27)) (justify left))
+    )

Commit message: Some hardware changes, started to add footprints and part links to digikey. Switching most to SMD
Parts:
- C15, C16: renamed from C?; value 100nF -> 0.1uF; footprint (none) -> Capacitor_SMD:C_0603_1608Metric_Pad1.08x0.95mm_HandSolder; Digikey (none) -> https://www.digikey.com/short/3wn2fdb2; Unit Price (none) -> 0.10
- U3: renamed from U?; footprint XDCR_BMP390L -> BMP390:XDCR_BMP390L; Digikey (none) -> https://www.digikey.com/short/43pj78n5; Unit Price (none) -> 5.18
- gave numbers to parts that had none: 2
Changed lines of the file:
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@@
     (stroke (width 0) (type default) (color 0 0 0 0))
-  )
-  (label "VDDIO" (at 102.87 27.94 0)
-    (effects (font (size 1.27 1.27)) (justify left bottom))
-  )
-  (label "VDD" (at 102.87 38.1 0)
-    (effects (font (size 1.27 1.27)) (justify left bottom))
   )
   (hierarchical_label "SCL" (shape input) (at 97.79 25.4 90)
@@
   (symbol (lib_id "Device:R") (at 72.39 60.96 0) (unit 1)
     (in_bom yes) (on_board yes) (fields_autoplaced)
-    (property "Reference" "R?" (id 0) (at 74.93 59.6899 0)
+    (property "Reference" "R9" (id 0) (at 74.93 59.6899 0)
       (effects (font (size 1.27 1.27)) (justify left))
     )
@@
   (symbol (lib_id "Device:C") (at 129.54 63.5 0) (unit 1)
     (in_bom yes) (on_board yes) (fields_autoplaced)
-    (property "Reference" "C?" (id 0) (at 133.35 62.2299 0)
+    (property "Reference" "C16" (id 0) (at 133.35 62.2299 0)
       (effects (font (size 1.27 1.27)) (justify left))
     )
-    (property "Value" "100nF" (id 1) (at 133.35 64.7699 0)
+    (property "Value" "0.1uF" (id 1) (at 133.35 64.7699 0)
       (effects (font (size 1.27 1.27)) (justify left))
     )
-    (property "Footprint" "" (id 2) (at 130.5052 67.31 0)
+    (property "Footprint" "Capacitor_SMD:C_0603_1608Metric_Pad1.08x0.95mm_HandSolder" (id 2) (at 130.5052 67.31 0)
       (effects (font (size 1.27 1.27)) hide)
     )
     (property "Datasheet" "~" (id 3) (at 129.54 63.5 0)
+      (effects (font (size 1.27 1.27)) hide)
+    )
+    (property "Digikey" "https://www.digikey.com/short/3wn2fdb2" (id 4) (at 129.54 63.5 0)
+      (effects (font (size 1.27 1.27)) hide)
+    )
+    (property "Unit Price" "0.10" (id 5) (at 129.54 63.5 0)
       (effects (font (size 1.27 1.27)) hide)
     )
@@
   (symbol (lib_id "power:GND") (at 129.54 81.28 0) (unit 1)
     (in_bom yes) (on_board yes) (fields_autoplaced)
-    (property "Reference" "#PWR?" (id 0) (at 129.54 87.63 0)
+    (property "Reference" "#PWR0148" (id 0) (at 129.54 87.63 0)
       (effects (font (size 1.27 1.27)) hide)
     )
@@
   (symbol (lib_id "Device:R") (at 106.68 50.8 90) (unit 1)
     (in_bom yes) (on_board yes)
-    (property "Reference" "R?" (id 0) (at 106.68 45.72 90))
+    (property "Reference" "R10" (id 0) (at 106.68 45.72 90))
     (property "Value" "4.7k" (id 1) (at 106.68 48.26 90))
     (property "Footprint" "" (id 2) (at 106.68 52.578 90)
@@
   (symbol (lib_id "BMP390L:BMP390L") (at 106.68 68.58 0) (unit 1)
     (in_bom yes) (on_board yes)
-    (property "Reference" "U?" (id 0) (at 106.68 63.5 0))
+    (property "Reference" "U3" (id 0) (at 106.68 63.5 0))
     (property "Value" "BMP390L" (id 1) (at 106.68 66.04 0))
-    (property "Footprint" "XDCR_BMP390L" (id 2) (at 106.68 68.58 0)
+    (property "Footprint" "BMP390:XDCR_BMP390L" (id 2) (at 106.68 68.58 0)
       (effects (font (size 1.27 1.27)) (justify bottom) hide)
     )
@@
       (effects (font (size 1.27 1.27)) (justify bottom) hide)
     )
+    (property "Digikey" "https://www.digikey.com/short/43pj78n5" (id 9) (at 106.68 68.58 0)
+      (effects (font (size 1.27 1.27)) hide)
+    )
+    (property "Unit Price" "5.18" (id 10) (at 106.68 68.58 0)
+      (effects (font (size 1.27 1.27)) hide)
+    )
     (pin "1")
     (pin "10")
@@
   (symbol (lib_id "power:GND") (at 83.82 60.96 0) (unit 1)
     (in_bom yes) (on_board yes) (fields_autoplaced)
-    (property "Reference" "#PWR?" (id 0) (at 83.82 67.31 0)
+    (property "Reference" "#PWR0147" (id 0) (at 83.82 67.31 0)
       (effects (font (size 1.27 1.27)) hide)
     )
@@
   (symbol (lib_id "Device:C") (at 83.82 50.8 0) (unit 1)
     (in_bom yes) (on_board yes) (fields_autoplaced)
-    (property "Reference" "C?" (id 0) (at 87.63 49.5299 0)
+    (property "Reference" "C15" (id 0) (at 87.63 49.5299 0)
       (effects (font (size 1.27 1.27)) (justify left))
     )
-    (property "Value" "100nF" (id 1) (at 87.63 52.0699 0)
+    (property "Value" "0.1uF" (id 1) (at 87.63 52.0699 0)
       (effects (font (size 1.27 1.27)) (justify left))
     )
-    (property "Footprint" "" (id 2) (at 84.7852 54.61 0)
+    (property "Footprint" "Capacitor_SMD:C_0603_1608Metric_Pad1.08x0.95mm_HandSolder" (id 2) (at 84.7852 54.61 0)
       (effects (font (size 1.27 1.27)) hide)
     )
@@
       (effects (font (size 1.27 1.27)) hide)
     )
+    (property "Digikey" "https://www.digikey.com/short/3wn2fdb2" (id 4) (at 83.82 50.8 0)
+      (effects (font (size 1.27 1.27)) hide)
+    )
+    (property "Unit Price" "0.10" (id 5) (at 83.82 50.8 0)
+      (effects (font (size 1.27 1.27)) hide)
+    )

Commit message: Updated footprints - Started work on PCB layout
Parts:
- R10, R9: footprint (none) -> Resistor_SMD:R_0603_1608Metric_Pad0.98x0.95mm_HandSolder; Digikey (none) -> https://www.digikey.com/short/4bjthv3d; Unit Price (none) -> 0.10
Changed lines of the file:
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@@
       (effects (font (size 1.27 1.27)) (justify left))
     )
-    (property "Footprint" "" (id 2) (at 70.612 60.96 90)
+    (property "Footprint" "Resistor_SMD:R_0603_1608Metric_Pad0.98x0.95mm_HandSolder" (id 2) (at 70.612 60.96 90)
       (effects (font (size 1.27 1.27)) hide)
     )
     (property "Datasheet" "~" (id 3) (at 72.39 60.96 0)
+      (effects (font (size 1.27 1.27)) hide)
+    )
+    (property "Digikey" "https://www.digikey.com/short/4bjthv3d" (id 4) (at 72.39 60.96 0)
+      (effects (font (size 1.27 1.27)) hide)
+    )
+    (property "Unit Price" "0.10" (id 5) (at 72.39 60.96 0)
       (effects (font (size 1.27 1.27)) hide)
     )
@@
     (property "Reference" "R10" (id 0) (at 106.68 45.72 90))
     (property "Value" "4.7k" (id 1) (at 106.68 48.26 90))
-    (property "Footprint" "" (id 2) (at 106.68 52.578 90)
+    (property "Footprint" "Resistor_SMD:R_0603_1608Metric_Pad0.98x0.95mm_HandSolder" (id 2) (at 106.68 52.578 90)
       (effects (font (size 1.27 1.27)) hide)
     )
@@
       (effects (font (size 1.27 1.27)) hide)
     )
+    (property "Digikey" "https://www.digikey.com/short/4bjthv3d" (id 4) (at 106.68 50.8 0)
+      (effects (font (size 1.27 1.27)) hide)
+    )
+    (property "Unit Price" "0.10" (id 5) (at 106.68 50.8 0)
+      (effects (font (size 1.27 1.27)) hide)
+    )

Commit message: Schematic Update - ADC/DAC & GPIO Config EEPROM
Parts:
- added TP30, TP31, TP32: TestPoint, TestPoint:TestPoint_Pad_D1.0mm, symbol Connector:TestPoint
Connections:
- net SCL: now also TP31.1
- net SDA: now also TP30.1
- net VCC: now also TP32.1
Changed lines of the file:
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@@
   (junction (at 129.54 73.66) (diameter 0) (color 0 0 0 0)
   )
+  (junction (at 90.17 38.1) (diameter 0) (color 0 0 0 0)
+  )
   (junction (at 83.82 59.69) (diameter 0) (color 0 0 0 0)
   )
@@
   )
   (junction (at 101.6 50.8) (diameter 0) (color 0 0 0 0)
+  )
+  (junction (at 135.89 43.18) (diameter 0) (color 0 0 0 0)
   )
   (no_connect (at 111.76 83.82))
@@
     (stroke (width 0) (type default) (color 0 0 0 0))
   )
-  (wire (pts (xy 78.74 38.1) (xy 95.25 38.1))
+  (wire (pts (xy 78.74 38.1) (xy 90.17 38.1))
     (stroke (width 0) (type default) (color 0 0 0 0))
   )
@@
     (stroke (width 0) (type default) (color 0 0 0 0))
   )
-  (wire (pts (xy 111.76 43.18) (xy 144.78 43.18))
+  (wire (pts (xy 111.76 43.18) (xy 135.89 43.18))
     (stroke (width 0) (type default) (color 0 0 0 0))
   )
@@
     (stroke (width 0) (type default) (color 0 0 0 0))
   )
+  (wire (pts (xy 90.17 38.1) (xy 95.25 38.1))
+    (stroke (width 0) (type default) (color 0 0 0 0))
+  )
   (wire (pts (xy 83.82 54.61) (xy 83.82 59.69))
     (stroke (width 0) (type default) (color 0 0 0 0))
@@
   )
   (wire (pts (xy 97.79 25.4) (xy 97.79 50.8))
+    (stroke (width 0) (type default) (color 0 0 0 0))
+  )
+  (wire (pts (xy 135.89 43.18) (xy 144.78 43.18))
     (stroke (width 0) (type default) (color 0 0 0 0))
   )
@@
     )
     (property "Datasheet" "" (id 3) (at 129.54 81.28 0)
+      (effects (font (size 1.27 1.27)) hide)
+    )
+    (pin "1")
+  )
+  (symbol (lib_id "Connector:TestPoint") (at 135.89 43.18 0) (unit 1)
+    (in_bom yes) (on_board yes) (fields_autoplaced)
+    (property "Reference" "TP32" (id 0) (at 138.43 38.6079 0)
+      (effects (font (size 1.27 1.27)) (justify left))
+    )
+    (property "Value" "TestPoint" (id 1) (at 138.43 41.1479 0)
+      (effects (font (size 1.27 1.27)) (justify left))
+    )
+    (property "Footprint" "TestPoint:TestPoint_Pad_D1.0mm" (id 2) (at 140.97 43.18 0)
+      (effects (font (size 1.27 1.27)) hide)
+    )
+    (property "Datasheet" "~" (id 3) (at 140.97 43.18 0)
+      (effects (font (size 1.27 1.27)) hide)
+    )
+    (pin "1")
+  )
+  (symbol (lib_id "Connector:TestPoint") (at 90.17 38.1 0) (unit 1)
+    (in_bom yes) (on_board yes) (fields_autoplaced)
+    (property "Reference" "TP30" (id 0) (at 92.71 33.5279 0)
+      (effects (font (size 1.27 1.27)) (justify left))
+    )
+    (property "Value" "TestPoint" (id 1) (at 92.71 36.0679 0)
+      (effects (font (size 1.27 1.27)) (justify left))
+    )
+    (property "Footprint" "TestPoint:TestPoint_Pad_D1.0mm" (id 2) (at 95.25 38.1 0)
+      (effects (font (size 1.27 1.27)) hide)
+    )
+    (property "Datasheet" "~" (id 3) (at 95.25 38.1 0)
       (effects (font (size 1.27 1.27)) hide)
     )
@@
       (effects (font (size 1.27 1.27)) hide)
     )
+    (pin "1")
+  )
+  (symbol (lib_id "Connector:TestPoint") (at 101.6 50.8 0) (unit 1)
+    (in_bom yes) (on_board yes)
+    (property "Reference" "TP31" (id 0) (at 100.33 40.64 0)
+      (effects (font (size 1.27 1.27)) (justify left))
+    )
+    (property "Value" "TestPoint" (id 1) (at 100.33 43.18 0)
+      (effects (font (size 1.27 1.27)) (justify left))
+    )
+    (property "Footprint" "TestPoint:TestPoint_Pad_D1.0mm" (id 2) (at 106.68 50.8 0)
+      (effects (font (size 1.27 1.27)) hide)
+    )
+    (property "Datasheet" "~" (id 3) (at 106.68 50.8 0)
+      (effects (font (size 1.27 1.27)) hide)
+    )
