File: hardware/GFC/GFC/BMP390.kicad_sch (KiCad schematic)
At the start: 8 parts, among them U3 BMP390L

Commit message: sync
Parts:
- removed TP30, TP31, TP32: TestPoint, TestPoint:TestPoint_Pad_D1.0mm, symbol Connector:TestPoint
- added TP37, TP38, TP39, TP40, TP41: Test Point, TestPoint:TestPoint_Pad_D1.0mm, symbol Connector:TestPoint_Small
Connections:
- net GND: now also TP37.1
- net VCC: now also TP40.1, TP41.1
- net SCL renamed I2C0.SCL
- net I2C0.SCL: now also TP39.1
- net SDA renamed I2C0.SDA
- net I2C0.SDA: now also TP38.1
Changed lines of the file:
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@@
   (junction (at 144.78 43.18) (diameter 0) (color 0 0 0 0)
   )
+  (junction (at 86.36 67.31) (diameter 0) (color 0 0 0 0)
+  )
   (junction (at 129.54 73.66) (diameter 0) (color 0 0 0 0)
   )
-  (junction (at 90.17 38.1) (diameter 0) (color 0 0 0 0)
-  )
   (junction (at 83.82 59.69) (diameter 0) (color 0 0 0 0)
   )
@@
   (junction (at 101.6 50.8) (diameter 0) (color 0 0 0 0)
   )
-  (junction (at 135.89 43.18) (diameter 0) (color 0 0 0 0)
-  )
   (no_connect (at 111.76 83.82))
+  (bus_entry (at 67.31 13.97) (size 2.54 2.54)
+    (stroke (width 0) (type default) (color 0 0 0 0))
+  )
+  (bus_entry (at 72.39 13.97) (size 2.54 2.54)
+    (stroke (width 0) (type default) (color 0 0 0 0))
+  )
   (wire (pts (xy 127 67.31) (xy 129.54 67.31))
     (stroke (width 0) (type default) (color 0 0 0 0))
@@
     (stroke (width 0) (type default) (color 0 0 0 0))
   )
-  (wire (pts (xy 78.74 38.1) (xy 90.17 38.1))
-    (stroke (width 0) (type default) (color 0 0 0 0))
-  )
   (wire (pts (xy 100.33 25.4) (xy 100.33 27.94))
     (stroke (width 0) (type default) (color 0 0 0 0))
@@
     (stroke (width 0) (type default) (color 0 0 0 0))
   )
-  (wire (pts (xy 111.76 43.18) (xy 135.89 43.18))
+  (wire (pts (xy 111.76 43.18) (xy 144.78 43.18))
     (stroke (width 0) (type default) (color 0 0 0 0))
   )
@@
     (stroke (width 0) (type default) (color 0 0 0 0))
   )
+  (bus (pts (xy 59.69 13.97) (xy 67.31 13.97))
+    (stroke (width 0) (type default) (color 0 0 0 0))
+  )
   (wire (pts (xy 144.78 43.18) (xy 144.78 91.44))
     (stroke (width 0) (type default) (color 0 0 0 0))
@@
     (stroke (width 0) (type default) (color 0 0 0 0))
   )
-  (wire (pts (xy 95.25 25.4) (xy 95.25 38.1))
+  (wire (pts (xy 95.25 19.05) (xy 95.25 38.1))
+    (stroke (width 0) (type default) (color 0 0 0 0))
+  )
+  (bus (pts (xy 67.31 13.97) (xy 72.39 13.97))
     (stroke (width 0) (type default) (color 0 0 0 0))
   )
@@
     (stroke (width 0) (type default) (color 0 0 0 0))
   )
-  (wire (pts (xy 90.17 38.1) (xy 95.25 38.1))
+  (wire (pts (xy 78.74 38.1) (xy 95.25 38.1))
     (stroke (width 0) (type default) (color 0 0 0 0))
   )
@@
     (stroke (width 0) (type default) (color 0 0 0 0))
   )
+  (wire (pts (xy 74.93 16.51) (xy 97.79 16.51))
+    (stroke (width 0) (type default) (color 0 0 0 0))
+  )
   (wire (pts (xy 129.54 38.1) (xy 129.54 59.69))
     (stroke (width 0) (type default) (color 0 0 0 0))
@@
     (stroke (width 0) (type default) (color 0 0 0 0))
   )
+  (wire (pts (xy 69.85 16.51) (xy 69.85 19.05))
+    (stroke (width 0) (type default) (color 0 0 0 0))
+  )
   (wire (pts (xy 127 59.69) (xy 129.54 59.69))
     (stroke (width 0) (type default) (color 0 0 0 0))
   )
-  (wire (pts (xy 97.79 25.4) (xy 97.79 50.8))
-    (stroke (width 0) (type default) (color 0 0 0 0))
-  )
-  (wire (pts (xy 135.89 43.18) (xy 144.78 43.18))
+  (wire (pts (xy 97.79 16.51) (xy 97.79 50.8))
     (stroke (width 0) (type default) (color 0 0 0 0))
   )
@@
     (stroke (width 0) (type default) (color 0 0 0 0))
   )
-  (hierarchical_label "SCL" (shape input) (at 97.79 25.4 90)
-    (effects (font (size 1.27 1.27)) (justify left))
+  (wire (pts (xy 69.85 19.05) (xy 95.25 19.05))
+    (stroke (width 0) (type default) (color 0 0 0 0))
+  )
+  (label "I2C0.SDA" (at 85.09 19.05 180)
+    (effects (font (size 1.27 1.27)) (justify right bottom))
+  )
+  (label "I2C0.SCL" (at 85.09 16.51 180)
+    (effects (font (size 1.27 1.27)) (justify right bottom))
   )
   (hierarchical_label "VCC" (shape input) (at 100.33 25.4 90)
     (effects (font (size 1.27 1.27)) (justify left))
   )
-  (hierarchical_label "SDA" (shape input) (at 95.25 25.4 90)
-    (effects (font (size 1.27 1.27)) (justify left))
+  (hierarchical_label "I2C{SDA SCL}" (shape input) (at 59.69 13.97 180)
+    (effects (font (size 1.27 1.27)) (justify right))
+  )
+  (symbol (lib_id "Connector:TestPoint_Small") (at 101.6 50.8 0) (mirror y) (unit 1)
+    (in_bom yes) (on_board yes)
+    (property "Reference" "TP39" (id 0) (at 105.41 49.53 0)
+      (effects (font (size 1.27 1.27)) (justify left))
+    )
+    (property "Value" "Test Point" (id 1) (at 100.33 52.0699 0)
+      (effects (font (size 1.27 1.27)) (justify left) hide)
+    )
+    (property "Footprint" "TestPoint:TestPoint_Pad_D1.0mm" (id 2) (at 96.52 50.8 0)
+      (effects (font (size 1.27 1.27)) hide)
+    )
+    (property "Datasheet" "~" (id 3) (at 96.52 50.8 0)
+      (effects (font (size 1.27 1.27)) hide)
+    )
+    (pin "1")
+  )
+  (symbol (lib_id "Connector:TestPoint_Small") (at 111.76 50.8 0) (mirror y) (unit 1)
+    (in_bom yes) (on_board yes)
+    (property "Reference" "TP40" (id 0) (at 115.57 49.53 0)
+      (effects (font (size 1.27 1.27)) (justify left))
+    )
+    (property "Value" "Test Point" (id 1) (at 110.49 52.0699 0)
+      (effects (font (size 1.27 1.27)) (justify left) hide)
+    )
+    (property "Footprint" "TestPoint:TestPoint_Pad_D1.0mm" (id 2) (at 106.68 50.8 0)
+      (effects (font (size 1.27 1.27)) hide)
+    )
+    (property "Datasheet" "~" (id 3) (at 106.68 50.8 0)
+      (effects (font (size 1.27 1.27)) hide)
+    )
+    (pin "1")
   )
   (symbol (lib_id "Device:R") (at 72.39 60.96 0) (unit 1)
@@
     (pin "1")
   )
-  (symbol (lib_id "Connector:TestPoint") (at 135.89 43.18 0) (unit 1)
-    (in_bom yes) (on_board yes) (fields_autoplaced)
-    (property "Reference" "TP32" (id 0) (at 138.43 38.6079 0)
-      (effects (font (size 1.27 1.27)) (justify left))
-    )
-    (property "Value" "TestPoint" (id 1) (at 138.43 41.1479 0)
-      (effects (font (size 1.27 1.27)) (justify left))
-    )
-    (property "Footprint" "TestPoint:TestPoint_Pad_D1.0mm" (id 2) (at 140.97 43.18 0)
-      (effects (font (size 1.27 1.27)) hide)
-    )
-    (property "Datasheet" "~" (id 3) (at 140.97 43.18 0)
-      (effects (font (size 1.27 1.27)) hide)
-    )
-    (pin "1")
-  )
-  (symbol (lib_id "Connector:TestPoint") (at 90.17 38.1 0) (unit 1)
-    (in_bom yes) (on_board yes) (fields_autoplaced)
-    (property "Reference" "TP30" (id 0) (at 92.71 33.5279 0)
-      (effects (font (size 1.27 1.27)) (justify left))
-    )
-    (property "Value" "TestPoint" (id 1) (at 92.71 36.0679 0)
-      (effects (font (size 1.27 1.27)) (justify left))
-    )
-    (property "Footprint" "TestPoint:TestPoint_Pad_D1.0mm" (id 2) (at 95.25 38.1 0)
-      (effects (font (size 1.27 1.27)) hide)
-    )
-    (property "Datasheet" "~" (id 3) (at 95.25 38.1 0)
+  (symbol (lib_id "Connector:TestPoint_Small") (at 129.54 59.69 0) (mirror y) (unit 1)
+    (in_bom yes) (on_board yes)
+    (property "Reference" "TP41" (id 0) (at 133.35 58.42 0)
+      (effects (font (size 1.27 1.27)) (justify left))
+    )
+    (property "Value" "Test Point" (id 1) (at 128.27 60.9599 0)
+      (effects (font (size 1.27 1.27)) (justify left) hide)
+    )
+    (property "Footprint" "TestPoint:TestPoint_Pad_D1.0mm" (id 2) (at 124.46 59.69 0)
+      (effects (font (size 1.27 1.27)) hide)
+    )
+    (property "Datasheet" "~" (id 3) (at 124.46 59.69 0)
       (effects (font (size 1.27 1.27)) hide)
     )
@@
     (pin "1")
     (pin "2")
+  )
+  (symbol (lib_id "Connector:TestPoint_Small") (at 83.82 59.69 0) (mirror y) (unit 1)
+    (in_bom yes) (on_board yes)
+    (property "Reference" "TP37" (id 0) (at 87.63 58.42 0)
+      (effects (font (size 1.27 1.27)) (justify left))
+    )
+    (property "Value" "Test Point" (id 1) (at 82.55 60.9599 0)
+      (effects (font (size 1.27 1.27)) (justify left) hide)
+    )
+    (property "Footprint" "TestPoint:TestPoint_Pad_D1.0mm" (id 2) (at 78.74 59.69 0)
+      (effects (font (size 1.27 1.27)) hide)
+    )
+    (property "Datasheet" "~" (id 3) (at 78.74 59.69 0)
+      (effects (font (size 1.27 1.27)) hide)
+    )
+    (pin "1")
   )
   (symbol (lib_id "BMP390L:BMP390L") (at 106.68 68.58 0) (unit 1)
@@
     (pin "9")
   )
+  (symbol (lib_id "Connector:TestPoint_Small") (at 86.36 67.31 0) (mirror y) (unit 1)
+    (in_bom yes) (on_board yes)
+    (property "Reference" "TP38" (id 0) (at 90.17 66.04 0)
+      (effects (font (size 1.27 1.27)) (justify left))
+    )
+    (property "Value" "Test Point" (id 1) (at 85.09 68.5799 0)
+      (effects (font (size 1.27 1.27)) (justify left) hide)
+    )
+    (property "Footprint" "TestPoint:TestPoint_Pad_D1.0mm" (id 2) (at 81.28 67.31 0)
+      (effects (font (size 1.27 1.27)) hide)
+    )
+    (property "Datasheet" "~" (id 3) (at 81.28 67.31 0)
+      (effects (font (size 1.27 1.27)) hide)
+    )
+    (pin "1")
+  )
   (symbol (lib_id "power:GND") (at 83.82 60.96 0) (unit 1)
     (in_bom yes) (on_board yes) (fields_autoplaced)
@@
       (effects (font (size 1.27 1.27)) hide)
     )
-    (pin "1")
-  )
-  (symbol (lib_id "Connector:TestPoint") (at 101.6 50.8 0) (unit 1)
-    (in_bom yes) (on_board yes)
-    (property "Reference" "TP31" (id 0) (at 100.33 40.64 0)
-      (effects (font (size 1.27 1.27)) (justify left))
-    )
-    (property "Value" "TestPoint" (id 1) (at 100.33 43.18 0)
-      (effects (font (size 1.27 1.27)) (justify left))
-    )
-    (property "Footprint" "TestPoint:TestPoint_Pad_D1.0mm" (id 2) (at 106.68 50.8 0)
-      (effects (font (size 1.27 1.27)) hide)
-    )
-    (property "Datasheet" "~" (id 3) (at 106.68 50.8 0)
-      (effects (font (size 1.27 1.27)) hide)
-    )
