File: hardware/GFC/GFC/EEPROM.kicad_sch (KiCad schematic)
At the start: 4 parts, among them U6 CAT24C32WI-GT3

Commit message: sync
Changed lines of the file:
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@@
     (effects (font (size 1.27 1.27)) (justify left))
   )
-  (hierarchical_label "EEPROM Interface" (shape input) (at 203.2 82.55 0)
+  (hierarchical_label "EEPROM{SDA SCL}" (shape input) (at 203.2 82.55 0)
     (effects (font (size 1.27 1.27)) (justify left))
   )
