File: hardware/GFC/GFC/SPI0_Expansion.kicad_sch (KiCad schematic)
At the start: 0 parts

Commit message: sync
Connections:
- no-connect marks 0 -> 2
Changed lines of the file:
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@@
 (kicad_sch (version 20211123) (generator eeschema)
   (paper "A4")
+  (no_connect (at 184.15 67.31))
+  (no_connect (at 184.15 72.39))
+  (wire (pts (xy 184.15 72.39) (xy 196.85 72.39))
+    (stroke (width 0) (type default) (color 0 0 0 0))
+  )
+  (bus (pts (xy 184.15 67.31) (xy 196.85 67.31))
+    (stroke (width 0) (type default) (color 0 0 0 0))
+  )
+  (hierarchical_label "SPI0{CE1 CE0 MISO MOSI SCLK}" (shape input) (at 196.85 67.31 0)
+    (effects (font (size 1.27 1.27)) (justify left))
+  )
+  (hierarchical_label "VCC" (shape input) (at 196.85 72.39 0)
+    (effects (font (size 1.27 1.27)) (justify left))
+  )
 )
