File: hardware/GFC/GFC/dac.kicad_sch (KiCad schematic)
At the start: 25 parts, among them J2 USB, U5 PCM2902C, Y1 12MHz

Commit message: sync
Parts:
- C21, C26, C29, C30, C33: footprint (none) -> Capacitor_SMD:C_0603_1608Metric_Pad1.08x0.95mm_HandSolder
Connections:
- no-connect marks 8 -> 12
Changed lines of the file:
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@@
   (junction (at 71.12 133.35) (diameter 0) (color 0 0 0 0)
   )
+  (no_connect (at 111.76 160.02))
   (no_connect (at 124.46 96.52))
-  (no_connect (at 99.06 147.32))
-  (no_connect (at 114.3 144.78))
+  (no_connect (at 104.14 160.02))
+  (no_connect (at 177.8 62.23))
   (no_connect (at 88.9 109.22))
   (no_connect (at 88.9 106.68))
+  (no_connect (at 177.8 54.61))
   (no_connect (at 124.46 106.68))
   (no_connect (at 88.9 111.76))
+  (no_connect (at 177.8 57.15))
+  (no_connect (at 177.8 59.69))
   (no_connect (at 124.46 104.14))
-  (bus_entry (at 114.3 162.56) (size -2.54 -2.54)
-    (stroke (width 0) (type default) (color 0 0 0 0))
-  )
-  (bus_entry (at 106.68 162.56) (size -2.54 -2.54)
+  (bus_entry (at 203.2 64.77) (size -2.54 -2.54)
+    (stroke (width 0) (type default) (color 0 0 0 0))
+  )
+  (bus_entry (at 198.12 64.77) (size -2.54 -2.54)
+    (stroke (width 0) (type default) (color 0 0 0 0))
+  )
+  (bus_entry (at 200.66 64.77) (size -2.54 -2.54)
+    (stroke (width 0) (type default) (color 0 0 0 0))
+  )
+  (bus_entry (at 205.74 64.77) (size -2.54 -2.54)
     (stroke (width 0) (type default) (color 0 0 0 0))
   )
@@
     (stroke (width 0) (type default) (color 0 0 0 0))
   )
+  (bus (pts (xy 198.12 64.77) (xy 200.66 64.77))
+    (stroke (width 0) (type default) (color 0 0 0 0))
+  )
   (wire (pts (xy 45.72 96.52) (xy 69.85 96.52))
     (stroke (width 0) (type default) (color 0 0 0 0))
@@
     (stroke (width 0) (type default) (color 0 0 0 0))
   )
-  (bus (pts (xy 114.3 162.56) (xy 210.82 162.56))
+  (bus (pts (xy 111.76 162.56) (xy 210.82 162.56))
     (stroke (width 0) (type default) (color 0 0 0 0))
   )
@@
     (stroke (width 0) (type default) (color 0 0 0 0))
   )
+  (wire (pts (xy 200.66 62.23) (xy 200.66 57.15))
+    (stroke (width 0) (type default) (color 0 0 0 0))
+  )
   (bus (pts (xy 109.22 162.56) (xy 106.68 162.56))
     (stroke (width 0) (type default) (color 0 0 0 0))
@@
     (stroke (width 0) (type default) (color 0 0 0 0))
   )
+  (wire (pts (xy 198.12 59.69) (xy 177.8 59.69))
+    (stroke (width 0) (type default) (color 0 0 0 0))
+  )
   (wire (pts (xy 124.46 101.6) (xy 146.05 101.6))
     (stroke (width 0) (type default) (color 0 0 0 0))
@@
     (stroke (width 0) (type default) (color 0 0 0 0))
   )
+  (wire (pts (xy 198.12 62.23) (xy 198.12 59.69))
+    (stroke (width 0) (type default) (color 0 0 0 0))
+  )
   (wire (pts (xy 153.67 114.3) (xy 153.67 113.03))
     (stroke (width 0) (type default) (color 0 0 0 0))
@@
     (stroke (width 0) (type default) (color 0 0 0 0))
   )
+  (bus (pts (xy 200.66 64.77) (xy 203.2 64.77))
+    (stroke (width 0) (type default) (color 0 0 0 0))
+  )
   (wire (pts (xy 69.85 87.63) (xy 69.85 96.52))
     (stroke (width 0) (type default) (color 0 0 0 0))
@@
     (stroke (width 0) (type default) (color 0 0 0 0))
   )
+  (wire (pts (xy 203.2 54.61) (xy 177.8 54.61))
+    (stroke (width 0) (type default) (color 0 0 0 0))
+  )
   (wire (pts (xy 144.78 120.65) (xy 144.78 123.19))
     (stroke (width 0) (type default) (color 0 0 0 0))
@@
     (stroke (width 0) (type default) (color 0 0 0 0))
   )
+  (wire (pts (xy 177.8 62.23) (xy 195.58 62.23))
+    (stroke (width 0) (type default) (color 0 0 0 0))
+  )
+  (wire (pts (xy 200.66 57.15) (xy 177.8 57.15))
+    (stroke (width 0) (type default) (color 0 0 0 0))
+  )
   (wire (pts (xy 138.43 133.35) (xy 138.43 130.81))
     (stroke (width 0) (type default) (color 0 0 0 0))
@@
     (stroke (width 0) (type default) (color 0 0 0 0))
   )
+  (bus (pts (xy 203.2 64.77) (xy 205.74 64.77))
+    (stroke (width 0) (type default) (color 0 0 0 0))
+  )
+  (bus (pts (xy 205.74 64.77) (xy 214.63 64.77))
+    (stroke (width 0) (type default) (color 0 0 0 0))
+  )
   (wire (pts (xy 129.54 123.19) (xy 132.08 123.19))
     (stroke (width 0) (type default) (color 0 0 0 0))
@@
     (stroke (width 0) (type default) (color 0 0 0 0))
   )
+  (wire (pts (xy 203.2 62.23) (xy 203.2 54.61))
+    (stroke (width 0) (type default) (color 0 0 0 0))
+  )
   (wire (pts (xy 62.23 128.27) (xy 59.69 128.27))
     (stroke (width 0) (type default) (color 0 0 0 0))
@@
   )
   (wire (pts (xy 71.12 133.35) (xy 71.12 137.16))
-    (stroke (width 0) (type default) (color 0 0 0 0))
-  )
-  (bus (pts (xy 114.3 162.56) (xy 111.76 162.56))
     (stroke (width 0) (type default) (color 0 0 0 0))
   )
@@
     (effects (font (size 1.27 1.27)) (justify right bottom))
   )
+  (label "DAC.BCLK" (at 177.8 62.23 0)
+    (effects (font (size 1.27 1.27)) (justify left bottom))
+  )
   (label "D+" (at 45.72 96.52 0)
     (effects (font (size 1.27 1.27)) (justify left bottom))
   )
+  (label "DAC.DIN" (at 177.8 57.15 0)
+    (effects (font (size 1.27 1.27)) (justify left bottom))
+  )
   (label "V_BUS" (at 45.72 101.6 0)
     (effects (font (size 1.27 1.27)) (justify left bottom))
@@
     (effects (font (size 1.27 1.27)) (justify right bottom))
   )
+  (label "DAC.LRC" (at 177.8 59.69 0)
+    (effects (font (size 1.27 1.27)) (justify left bottom))
+  )
   (label "D-" (at 45.72 99.06 0)
     (effects (font (size 1.27 1.27)) (justify left bottom))
@@
     (effects (font (size 1.27 1.27)) (justify left bottom))
   )
-  (global_label "AUDIO{SC_IN_L SC_IN_R SC_OUT_L SC_OUR_R" (shape input) (at 210.82 73.66 0) (fields_autoplaced)
+  (label "DAC.DOUT" (at 177.8 54.61 0)
+    (effects (font (size 1.27 1.27)) (justify left bottom))
+  )
+  (hierarchical_label "AUDIO{SC_IN_L SC_IN_R SC_OUT_L SC_OUT_R}" (shape input) (at 214.63 68.58 0)
     (effects (font (size 1.27 1.27)) (justify left))
-    (property "Intersheet References" "${INTERSHEET_REFS}" (id 0) (at 257.1388 73.5806 0)
-      (effects (font (size 1.27 1.27)) (justify left) hide)
-    )
-  )
-  (hierarchical_label "Analog Audio" (shape input) (at 214.63 68.58 0)
+  )
+  (hierarchical_label "DAC{BCLK LRC DIN DOUT}" (shape input) (at 214.63 64.77 0)
     (effects (font (size 1.27 1.27)) (justify left))
   )
@@
       (effects (font (size 1.27 1.27)) (justify left))
     )
-    (property "Footprint" "" (id 2) (at 69.85 104.14 0)
+    (property "Footprint" "Capacitor_SMD:C_0603_1608Metric_Pad1.08x0.95mm_HandSolder" (id 2) (at 69.85 104.14 0)
       (effects (font (size 1.27 1.27)) hide)
     )
@@
       (effects (font (size 1.27 1.27)) (justify left))
     )
-    (property "Footprint" "" (id 2) (at 163.83 124.46 0)
+    (property "Footprint" "Capacitor_SMD:C_0603_1608Metric_Pad1.08x0.95mm_HandSolder" (id 2) (at 163.83 124.46 0)
       (effects (font (size 1.27 1.27)) hide)
     )
@@
       (effects (font (size 1.27 1.27)) (justify left))
     )
-    (property "Footprint" "" (id 2) (at 148.59 109.22 0)
+    (property "Footprint" "Capacitor_SMD:C_0603_1608Metric_Pad1.08x0.95mm_HandSolder" (id 2) (at 148.59 109.22 0)
       (effects (font (size 1.27 1.27)) hide)
     )
@@
       (effects (font (size 1.27 1.27)) (justify left))
     )
-    (property "Footprint" "" (id 2) (at 134.62 123.19 0)
+    (property "Footprint" "Capacitor_SMD:C_0603_1608Metric_Pad1.08x0.95mm_HandSolder" (id 2) (at 134.62 123.19 0)
       (effects (font (size 1.27 1.27)) hide)
     )
@@
       (effects (font (size 1.27 1.27)) (justify left))
     )
-    (property "Footprint" "" (id 2) (at 143.51 99.06 0)
-      (effects (font (size 1.27 1.27)) hide)
-    )
+    (property "Footprint" "Capacitor_SMD:C_0603_1608Metric_Pad1.08x0.95mm_HandSolder" (id 2) (at 143.51 99.06 0)
+      (effects (font (size 1.27 1.27)) hide)
+    )
