File: hardware/GFC/EEPROM.kicad_sch (KiCad schematic)
At the start: 4 parts, among them U6 CAT24C32WI-GT3

Commit message: Cleaning up the hardware directory
Parts:
- C34: footprint (none) -> Capacitor_SMD:C_0603_1608Metric_Pad1.08x0.95mm_HandSolder; Digikey (none) -> https://www.digikey.com/short/3wn2fdb2
- R23, R24: footprint (none) -> Resistor_SMD:R_0603_1608Metric_Pad0.98x0.95mm_HandSolder
Changed lines of the file:
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@@
     (property "Reference" "C34" (id 0) (at 121.92 90.17 90))
     (property "Value" "0.1uF" (id 1) (at 121.92 92.71 90))
-    (property "Footprint" "" (id 2) (at 125.73 96.8248 0)
+    (property "Footprint" "Capacitor_SMD:C_0603_1608Metric_Pad1.08x0.95mm_HandSolder" (id 2) (at 125.73 96.8248 0)
       (effects (font (size 1.27 1.27)) hide)
     )
     (property "Datasheet" "~" (id 3) (at 121.92 97.79 0)
+      (effects (font (size 1.27 1.27)) hide)
+    )
+    (property "Digikey" "https://www.digikey.com/short/3wn2fdb2" (id 4) (at 121.92 97.79 0)
       (effects (font (size 1.27 1.27)) hide)
     )
@@
       (effects (font (size 1.27 1.27)) (justify left))
     )
-    (property "Footprint" "" (id 2) (at 173.482 92.71 90)
+    (property "Footprint" "Resistor_SMD:R_0603_1608Metric_Pad0.98x0.95mm_HandSolder" (id 2) (at 173.482 92.71 90)
       (effects (font (size 1.27 1.27)) hide)
     )
@@
       (effects (font (size 1.27 1.27)) (justify left))
     )
-    (property "Footprint" "" (id 2) (at 167.132 96.52 90)
+    (property "Footprint" "Resistor_SMD:R_0603_1608Metric_Pad0.98x0.95mm_HandSolder" (id 2) (at 167.132 96.52 90)
       (effects (font (size 1.27 1.27)) hide)
     )
