File: hardware/GFC/SAM-M8Q.kicad_sch (KiCad schematic)
At the start: 4 parts, among them U4 SAM-M8Q

Commit message: Cleaning up the hardware directory
Parts:
- removed TP42, TP43: Test Point, TestPoint:TestPoint_Pad_D1.0mm, symbol Connector:TestPoint_Small
Changed lines of the file:
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@@
   (junction (at 130.81 63.5) (diameter 0) (color 0 0 0 0)
   )
-  (junction (at 147.3561 92.71) (diameter 0) (color 0 0 0 0)
-  )
   (junction (at 130.81 68.58) (diameter 0) (color 0 0 0 0)
-  )
-  (junction (at 147.32 90.17) (diameter 0) (color 0 0 0 0)
   )
   (junction (at 130.81 71.12) (diameter 0) (color 0 0 0 0)
@@
     (stroke (width 0) (type default) (color 0 0 0 0))
   )
-  (wire (pts (xy 146.05 90.17) (xy 147.32 90.17))
+  (wire (pts (xy 146.05 90.17) (xy 152.4 90.17))
     (stroke (width 0) (type default) (color 0 0 0 0))
   )
@@
     (stroke (width 0) (type default) (color 0 0 0 0))
   )
-  (wire (pts (xy 146.05 92.71) (xy 147.3561 92.71))
-    (stroke (width 0) (type default) (color 0 0 0 0))
-  )
-  (wire (pts (xy 147.32 90.17) (xy 152.4 90.17))
-    (stroke (width 0) (type default) (color 0 0 0 0))
-  )
   (wire (pts (xy 130.81 60.96) (xy 130.81 63.5))
     (stroke (width 0) (type default) (color 0 0 0 0))
@@
     (stroke (width 0) (type default) (color 0 0 0 0))
   )
-  (wire (pts (xy 147.3561 92.71) (xy 152.4 92.71))
+  (wire (pts (xy 146.05 92.71) (xy 152.4 92.71))
     (stroke (width 0) (type default) (color 0 0 0 0))
   )
@@
     (effects (font (size 1.27 1.27)) (justify left))
   )
-  (symbol (lib_id "Connector:TestPoint_Small") (at 147.3561 92.71 0) (mirror y) (unit 1)
-    (in_bom yes) (on_board yes)
-    (property "Reference" "TP43" (id 0) (at 151.1661 91.44 0)
-      (effects (font (size 1.27 1.27)) (justify left))
-    )
-    (property "Value" "Test Point" (id 1) (at 146.0861 93.9799 0)
-      (effects (font (size 1.27 1.27)) (justify left) hide)
-    )
-    (property "Footprint" "TestPoint:TestPoint_Pad_D1.0mm" (id 2) (at 142.2761 92.71 0)
-      (effects (font (size 1.27 1.27)) hide)
-    )
-    (property "Datasheet" "~" (id 3) (at 142.2761 92.71 0)
-      (effects (font (size 1.27 1.27)) hide)
-    )
-    (pin "1")
-  )
   (symbol (lib_id "Device:C") (at 123.19 63.5 90) (unit 1)
     (in_bom yes) (on_board yes) (fields_autoplaced)
@@
     (pin "2")
   )
-  (symbol (lib_id "Connector:TestPoint_Small") (at 147.32 90.17 0) (mirror y) (unit 1)
-    (in_bom yes) (on_board yes)
-    (property "Reference" "TP42" (id 0) (at 151.13 88.9 0)
-      (effects (font (size 1.27 1.27)) (justify left))
-    )
-    (property "Value" "Test Point" (id 1) (at 146.05 91.4399 0)
-      (effects (font (size 1.27 1.27)) (justify left) hide)
-    )
-    (property "Footprint" "TestPoint:TestPoint_Pad_D1.0mm" (id 2) (at 142.24 90.17 0)
-      (effects (font (size 1.27 1.27)) hide)
-    )
-    (property "Datasheet" "~" (id 3) (at 142.24 90.17 0)
-      (effects (font (size 1.27 1.27)) hide)
-    )
-    (pin "1")
-  )
   (symbol (lib_id "power:GND") (at 116.84 66.04 0) (unit 1)

Commit message: PCB Prototype
Parts:
- removed C17: 0.1uF, Capacitor_SMD:C_0603_1608Metric_Pad1.08x0.95mm_HandSolder, symbol Device:C
- removed U4: SAM-M8Q, RF_GPS:ublox_SAM-M8Q, symbol RF_GPS:SAM-M8Q
Connections:
- no-connect marks 6 -> 0
Changed lines of the file:
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@@
 (kicad_sch (version 20211123) (generator eeschema)
   (paper "A4")
-  (junction (at 130.81 63.5) (diameter 0) (color 0 0 0 0)
-  )
-  (junction (at 130.81 68.58) (diameter 0) (color 0 0 0 0)
-  )
-  (junction (at 130.81 71.12) (diameter 0) (color 0 0 0 0)
-  )
-  (no_connect (at 120.65 92.71))
-  (no_connect (at 120.65 90.17))
-  (no_connect (at 120.65 87.63))
-  (no_connect (at 146.05 82.55))
-  (no_connect (at 146.05 85.09))
-  (no_connect (at 120.65 85.09))
-  (bus_entry (at 151.13 43.18) (size -2.54 2.54)
-    (stroke (width 0) (type default) (color 0 0 0 0))
-  )
-  (bus_entry (at 151.13 46.99) (size -2.54 2.54)
-    (stroke (width 0) (type default) (color 0 0 0 0))
-  )
-  (wire (pts (xy 152.4 93.98) (xy 166.37 93.98))
-    (stroke (width 0) (type default) (color 0 0 0 0))
-  )
-  (wire (pts (xy 146.05 90.17) (xy 152.4 90.17))
-    (stroke (width 0) (type default) (color 0 0 0 0))
-  )
-  (bus (pts (xy 152.4 43.18) (xy 151.13 43.18))
-    (stroke (width 0) (type default) (color 0 0 0 0))
-  )
-  (wire (pts (xy 130.81 71.12) (xy 130.81 74.93))
-    (stroke (width 0) (type default) (color 0 0 0 0))
-  )
-  (wire (pts (xy 152.4 90.17) (xy 152.4 87.63))
-    (stroke (width 0) (type default) (color 0 0 0 0))
-  )
-  (wire (pts (xy 166.37 63.5) (xy 135.89 63.5))
-    (stroke (width 0) (type default) (color 0 0 0 0))
-  )
-  (wire (pts (xy 148.59 45.72) (xy 133.35 45.72))
-    (stroke (width 0) (type default) (color 0 0 0 0))
-  )
-  (wire (pts (xy 127 63.5) (xy 130.81 63.5))
-    (stroke (width 0) (type default) (color 0 0 0 0))
-  )
-  (wire (pts (xy 119.38 63.5) (xy 116.84 63.5))
-    (stroke (width 0) (type default) (color 0 0 0 0))
-  )
-  (wire (pts (xy 135.89 74.93) (xy 135.89 68.58))
-    (stroke (width 0) (type default) (color 0 0 0 0))
-  )
-  (wire (pts (xy 152.4 92.71) (xy 152.4 93.98))
-    (stroke (width 0) (type default) (color 0 0 0 0))
-  )
-  (wire (pts (xy 130.81 68.58) (xy 130.81 71.12))
-    (stroke (width 0) (type default) (color 0 0 0 0))
-  )
-  (wire (pts (xy 163.83 87.63) (xy 163.83 66.04))
-    (stroke (width 0) (type default) (color 0 0 0 0))
-  )
-  (wire (pts (xy 130.81 60.96) (xy 130.81 63.5))
-    (stroke (width 0) (type default) (color 0 0 0 0))
-  )
-  (bus (pts (xy 151.13 43.18) (xy 151.13 46.99))
-    (stroke (width 0) (type default) (color 0 0 0 0))
-  )
-  (wire (pts (xy 146.05 92.71) (xy 152.4 92.71))
-    (stroke (width 0) (type default) (color 0 0 0 0))
-  )
-  (wire (pts (xy 133.35 71.12) (xy 130.81 71.12))
-    (stroke (width 0) (type default) (color 0 0 0 0))
-  )
-  (wire (pts (xy 130.81 63.5) (xy 130.81 68.58))
-    (stroke (width 0) (type default) (color 0 0 0 0))
-  )
-  (wire (pts (xy 135.89 49.53) (xy 148.59 49.53))
-    (stroke (width 0) (type default) (color 0 0 0 0))
-  )
-  (wire (pts (xy 163.83 66.04) (xy 133.35 66.04))
-    (stroke (width 0) (type default) (color 0 0 0 0))
-  )
-  (wire (pts (xy 116.84 63.5) (xy 116.84 66.04))
-    (stroke (width 0) (type default) (color 0 0 0 0))
-  )
-  (wire (pts (xy 135.89 68.58) (xy 130.81 68.58))
-    (stroke (width 0) (type default) (color 0 0 0 0))
-  )
-  (wire (pts (xy 166.37 93.98) (xy 166.37 63.5))
-    (stroke (width 0) (type default) (color 0 0 0 0))
-  )
-  (wire (pts (xy 133.35 74.93) (xy 133.35 71.12))
-    (stroke (width 0) (type default) (color 0 0 0 0))
-  )
-  (wire (pts (xy 135.89 49.53) (xy 135.89 63.5))
-    (stroke (width 0) (type default) (color 0 0 0 0))
-  )
-  (wire (pts (xy 133.35 100.33) (xy 133.35 104.14))
-    (stroke (width 0) (type default) (color 0 0 0 0))
-  )
-  (wire (pts (xy 152.4 87.63) (xy 163.83 87.63))
-    (stroke (width 0) (type default) (color 0 0 0 0))
-  )
-  (wire (pts (xy 133.35 45.72) (xy 133.35 66.04))
-    (stroke (width 0) (type default) (color 0 0 0 0))
-  )
-  (label "I2C0.SDA" (at 139.7 45.72 0)
-    (effects (font (size 1.27 1.27)) (justify left bottom))
-  )
-  (label "I2C0.SCL" (at 139.7 49.53 0)
-    (effects (font (size 1.27 1.27)) (justify left bottom))
-  )
-  (hierarchical_label "I2C0{SDA SCL}" (shape input) (at 152.4 43.18 0)
-    (effects (font (size 1.27 1.27)) (justify left))
-  )
-  (hierarchical_label "VCC" (shape input) (at 130.81 60.96 90)
-    (effects (font (size 1.27 1.27)) (justify left))
-  )
-  (symbol (lib_id "Device:C") (at 123.19 63.5 90) (unit 1)
-    (in_bom yes) (on_board yes) (fields_autoplaced)
-    (property "Reference" "C17" (id 0) (at 123.19 55.88 90))
-    (property "Value" "0.1uF" (id 1) (at 123.19 58.42 90))
-    (property "Footprint" "Capacitor_SMD:C_0603_1608Metric_Pad1.08x0.95mm_HandSolder" (id 2) (at 127 62.5348 0)
-      (effects (font (size 1.27 1.27)) hide)
-    )
-    (property "Datasheet" "~" (id 3) (at 123.19 63.5 0)
-      (effects (font (size 1.27 1.27)) hide)
-    )
-    (property "Digikey" "https://www.digikey.com/short/3wn2fdb2" (id 4) (at 123.19 63.5 0)
-      (effects (font (size 1.27 1.27)) hide)
-    )
-    (property "Unit Price" "0.10" (id 5) (at 123.19 63.5 0)
-      (effects (font (size 1.27 1.27)) hide)
-    )
-    (pin "1")
-    (pin "2")
-  )
-  (symbol (lib_id "power:GND") (at 116.84 66.04 0) (unit 1)
-    (in_bom yes) (on_board yes) (fields_autoplaced)
-    (property "Reference" "#PWR0149" (id 0) (at 116.84 72.39 0)
-      (effects (font (size 1.27 1.27)) hide)
-    )
-    (property "Value" "GND" (id 1) (at 116.84 71.12 0))
-    (property "Footprint" "" (id 2) (at 116.84 66.04 0)
-      (effects (font (size 1.27 1.27)) hide)
-    )
-    (property "Datasheet" "" (id 3) (at 116.84 66.04 0)
-      (effects (font (size 1.27 1.27)) hide)
-    )
-    (pin "1")
-  )
-  (symbol (lib_id "RF_GPS:SAM-M8Q") (at 133.35 87.63 0) (unit 1)
-    (in_bom yes) (on_board yes) (fields_autoplaced)
-    (property "Reference" "U4" (id 0) (at 135.3694 100.33 0)
-      (effects (font (size 1.27 1.27)) (justify left))
-    )
-    (property "Value" "SAM-M8Q" (id 1) (at 135.3694 102.87 0)
-      (effects (font (size 1.27 1.27)) (justify left))
-    )
-    (property "Footprint" "RF_GPS:ublox_SAM-M8Q" (id 2) (at 146.05 99.06 0)
-      (effects (font (size 1.27 1.27)) hide)
-    )
-    (property "Datasheet" "https://www.u-blox.com/sites/default/files/SAM-M8Q_DataSheet_%28UBX-16012619%29.pdf" (id 3) (at 133.35 87.63 0)
-      (effects (font (size 1.27 1.27)) hide)
-    )
-    (property "Digikey" "https://www.digikey.com/short/n7wwdb37" (id 4) (at 133.35 87.63 0)
-      (effects (font (size 1.27 1.27)) hide)
-    )
-    (property "Unit Price" "31.50" (id 5) (at 133.35 87.63 0)
-      (effects (font (size 1.27 1.27)) hide)
-    )
-    (pin "1")
-    (pin "10")
-    (pin "11")
-    (pin "12")
-    (pin "13")
-    (pin "14")
-    (pin "15")
-    (pin "16")
-    (pin "17")
-    (pin "18")
-    (pin "19")
-    (pin "2")
-    (pin "20")
-    (pin "3")
-    (pin "4")
-    (pin "5")
-    (pin "6")
-    (pin "7")
-    (pin "8")
-    (pin "9")
-  )
-  (symbol (lib_id "power:GND") (at 133.35 104.14 0) (unit 1)
-    (in_bom yes) (on_board yes) (fields_autoplaced)
-    (property "Reference" "#PWR0150" (id 0) (at 133.35 110.49 0)
-      (effects (font (size 1.27 1.27)) hide)
-    )
-    (property "Value" "GND" (id 1) (at 133.35 109.22 0))
-    (property "Footprint" "" (id 2) (at 133.35 104.14 0)
-      (effects (font (size 1.27 1.27)) hide)
-    )
-    (property "Datasheet" "" (id 3) (at 133.35 104.14 0)
-      (effects (font (size 1.27 1.27)) hide)
-    )
-    (pin "1")
-  )
 )
