File: hardware/GFC/GFC.kicad_pcb (KiCad board)
At the start: 2 copper layers, 103 parts, among them J1 BAT, Q1 Q_NPN_BCE, Q2 DMN67D8LW-13, Q3 Q_NPN_BCE, SW1 H/L_DIP_SW, U2 LTV-356T, U4 SAM-M8Q, U5 PCM2902C, U6 CAT24C32WI-GT3

Commit message: Cleaning up the hardware directory
Parts:
- removed TP30, TP32, TP33, TP37, TP40, TP41, TP42, TP43: Test Point, TestPoint:TestPoint_Pad_D1.0mm
- added C20: 100nF, Capacitor_SMD:C_0603_1608Metric_Pad1.08x0.95mm_HandSolder, F.Cu at (36.3, 26.4)
- added C22: 4.7uF, Capacitor_SMD:C_0603_1608Metric_Pad1.08x0.95mm_HandSolder, F.Cu at (94.2, 56.1)
- added C23: 4.7uF, Capacitor_SMD:C_0603_1608Metric_Pad1.08x0.95mm_HandSolder, F.Cu at (94.2, 54.6)
- added C24: 10uF, Capacitor_SMD:C_0603_1608Metric_Pad1.08x0.95mm_HandSolder, F.Cu at (90.4, 51.3)
- added C25: 10uF, Capacitor_SMD:C_0603_1608Metric_Pad1.08x0.95mm_HandSolder, F.Cu at (90.4, 53.1)
- added C27: 4.7uF, Capacitor_SMD:C_0603_1608Metric_Pad1.08x0.95mm_HandSolder, F.Cu at (106.1, 56.6)
- added C28: 4.7uF, Capacitor_SMD:C_0603_1608Metric_Pad1.08x0.95mm_HandSolder, F.Cu at (106.1, 58.4)
- added C31: 10pF, Capacitor_SMD:C_0603_1608Metric_Pad1.08x0.95mm_HandSolder, F.Cu at (113.0, 47.8)
- added C32: 10pF, Capacitor_SMD:C_0603_1608Metric_Pad1.08x0.95mm_HandSolder, F.Cu at (112.5, 52.1)
- added C34: 0.1uF, Capacitor_SMD:C_0603_1608Metric_Pad1.08x0.95mm_HandSolder, F.Cu at (84.9, 34.8)
- added J2: USB, Connector_PinHeader_2.54mm:PinHeader_1x04_P2.54mm_Vertical, F.Cu at (82.8, 50.3)
- added LED1: Status LED, LED_SMD:LED_0805_2012Metric, F.Cu at (62.5, 30.0)
- added Op_R1: R, Resistor_SMD:R_0603_1608Metric_Pad0.98x0.95mm_HandSolder, F.Cu at (35.6, 17.3)
- added Op_R2: R, Resistor_SMD:R_0603_1608Metric_Pad0.98x0.95mm_HandSolder, F.Cu at (50.8, 17.8)
- added R14: OR 1M, Resistor_SMD:R_0603_1608Metric_Pad0.98x0.95mm_HandSolder, F.Cu at (91.4, 57.4)
- added R15: OR 1M, Resistor_SMD:R_0603_1608Metric_Pad0.98x0.95mm_HandSolder, F.Cu at (89.6, 57.4)
- added R16: 2.2, Resistor_SMD:R_0603_1608Metric_Pad0.98x0.95mm_HandSolder, F.Cu at (86.8, 47.2)
- added R17: 1.5k, Resistor_SMD:R_0603_1608Metric_Pad0.98x0.95mm_HandSolder, F.Cu at (86.8, 41.7)
- added R18: 22, Resistor_SMD:R_0603_1608Metric_Pad0.98x0.95mm_HandSolder, F.Cu at (89.4, 42.7)
- added R19: 22, Resistor_SMD:R_0603_1608Metric_Pad0.98x0.95mm_HandSolder, F.Cu at (89.4, 44.5)
- added R2: R, Resistor_SMD:R_0603_1608Metric_Pad0.98x0.95mm_HandSolder, F.Cu at (58.9, 30.0)
- added R20: OR 1M, Resistor_SMD:R_0603_1608Metric_Pad0.98x0.95mm_HandSolder, F.Cu at (112.0, 59.2)
- added R21: 1M, Resistor_SMD:R_0603_1608Metric_Pad0.98x0.95mm_HandSolder, F.Cu at (104.9, 49.3)
- added R22: OR 1M, Resistor_SMD:R_0603_1608Metric_Pad0.98x0.95mm_HandSolder, F.Cu at (112.0, 55.6)
- added R23: 3.9K, Resistor_SMD:R_0603_1608Metric_Pad0.98x0.95mm_HandSolder, F.Cu at (82.1, 32.5)
- added R24: 3.9K, Resistor_SMD:R_0603_1608Metric_Pad0.98x0.95mm_HandSolder, F.Cu at (80.3, 30.2)
- added TP46: Test Point, TestPoint:TestPoint_Pad_D1.0mm, F.Cu at (93.5, 58.2)
- added TP47: Test Point, TestPoint:TestPoint_Pad_D1.0mm, F.Cu at (114.3, 56.4)
- added U1: MAX17048G+T10, MAX17048G_T10:SON50P200X200X80-9N, F.Cu at (33.5, 36.6)
- added U3: BMP390L, BMP390:XDCR_BMP390L, F.Cu at (32.9, 64.0)
- CPU1: footprint Connector_PinSocket_2.54mm:PinSocket_2x20_P2.54mm_Vertical -> Connector_PinSocket_2.54mm:PinSocket_2x20_P2.54mm_Vertical_SMD
- R11: footprint Resistor_SMD:R_1206_3216Metric_Pad1.30x1.75mm_HandSolder -> Resistor_SMD:R_0603_1608Metric_Pad0.98x0.95mm_HandSolder
- moved TP19 205.8 mm to (121.7, 39.4)
- moved TP25 205.5 mm to (120.7, 63.5), turned to -90 degrees
- moved TP21 202.3 mm to (121.4, 45.2)
- moved TP24 201.8 mm to (132.6, 64.5)
- moved TP27 201.4 mm to (117.6, 33.8)
- moved R13 201.1 mm to (111.8, 28.7)
- moved C10 200.8 mm to (124.2, 22.1)
- moved C11 200.8 mm to (125.7, 22.1)
- moved C12 200.8 mm to (127.3, 22.1)
- moved C9 200.8 mm to (152.4, 53.1)
- moved L1 200.8 mm to (153.4, 32.8)
- moved L3 200.8 mm to (153.4, 49.0)
- moved Q3 200.8 mm to (120.7, 51.6)
- moved R3 200.8 mm to (115.8, 21.1)
- moved R5 200.8 mm to (120.7, 33.8)
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Connections:
- R10 pad 1: /BMP390 (I2C)/I2C0.SCL -> I2C0.SCL
- R9 pad 2: /BMP390 (I2C)/I2C0.SDA -> I2C0.SDA
- TP38 pad 1: /BMP390 (I2C)/I2C0.SDA -> I2C0.SDA
- TP39 pad 1: /BMP390 (I2C)/I2C0.SCL -> I2C0.SCL
Routing:
- net +3V3: track 17.6 -> 246.4 mm, vias 0 -> 14
- net UART0.PI_TXD: track 0.00 -> 169.4 mm, vias 0 -> 4
- net UART0.PI_RXD: track 0.00 -> 160.7 mm, vias 0 -> 4
- net +4V3: track 31.7 -> 169.7 mm
- net I2C0.SCL: track 0.00 -> 100.5 mm, vias 0 -> 4
- net I2C0.SDA: track 0.00 -> 85.2 mm, vias 0 -> 5
- net GND: track 16.1 -> 97.6 mm, vias 0 -> 31
- net 1-Wire: track 17.6 -> 81.7 mm
- net /DAC/AUDIO.SC_IN_R: track 0.00 -> 53.6 mm
- net GPIO.DRA_SQ: track 0.00 -> 38.8 mm, vias 0 -> 2
- net +5V: track 27.7 -> 58.1 mm
- net Net-(C29-Pad1): track 0.00 -> 29.8 mm, vias 0 -> 2
- net /DAC/AUDIO.SC_OUT_R: track 0.00 -> 22.4 mm, vias 0 -> 2
- net GPIO.DRA_PTT: track 0.00 -> 22.4 mm
- net EEPROM.SDA: track 0.00 -> 22.4 mm, vias 0 -> 2
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- added copper zone on B.Cu, net GND
- added copper zone on F.Cu, net GND

Commit message: PCB Prototype
Parts:
- removed AE1: Antenna, footprints:LINX_CONSMA001-G
- removed C1, C10, C13, C4, C5: 0.1uF, Capacitor_SMD:C_0603_1608Metric_Pad1.08x0.95mm_HandSolder
- removed C11: 10kpF, Capacitor_SMD:C_0603_1608Metric_Pad1.08x0.95mm_HandSolder
- removed C12: 1kpF, Capacitor_SMD:C_0603_1608Metric_Pad1.08x0.95mm_HandSolder
- removed C2: 100uF, Capacitor_THT:CP_Radial_D6.3mm_P2.50mm
- removed C20: 100nF, Capacitor_SMD:C_0603_1608Metric_Pad1.08x0.95mm_HandSolder
- removed C24, C25: 10uF, Capacitor_SMD:C_0603_1608Metric_Pad1.08x0.95mm_HandSolder
- removed C26, C29, C3, C30, C33: 1uF, Capacitor_SMD:C_0603_1608Metric_Pad1.08x0.95mm_HandSolder
- removed C27, C28: 4.7uF, Capacitor_SMD:C_0603_1608Metric_Pad1.08x0.95mm_HandSolder
- removed C31, C32: 10pF, Capacitor_SMD:C_0603_1608Metric_Pad1.08x0.95mm_HandSolder
- removed C6, C9: 20pF, Capacitor_SMD:C_0603_1608Metric_Pad1.08x0.95mm_HandSolder
- removed C7, C8: 36pF, Capacitor_SMD:C_0603_1608Metric_Pad1.08x0.95mm_HandSolder
- removed CPU1: Pi Zero/Zero W, Connector_PinSocket_2.54mm:PinSocket_2x20_P2.54mm_Vertical_SMD
- removed J1: BAT, TerminalBlock_Phoenix:TerminalBlock_Phoenix_PT-1,5-2-5.0-H_1x02_P5.00mm_Horizontal
- removed L1, L3: 56nH, footprints:IND_AIAC-1812-33NK-T
- removed L2: 68nH, footprints:IND_AIAC-1812-33NK-T
- removed LED1: Status LED, LED_SMD:LED_0805_2012Metric
- removed Op_R1, Op_R2, R2: R, Resistor_SMD:R_0603_1608Metric_Pad0.98x0.95mm_HandSolder
- removed Q1, Q3: Q_NPN_BCE, Package_TO_SOT_SMD:SOT-23
- removed Q2: DMN67D8LW-13, Package_TO_SOT_SMD:SOT-323_SC-70_Handsoldering
- removed R1, R10, R9: 4.7k, Resistor_SMD:R_0603_1608Metric_Pad0.98x0.95mm_HandSolder
- removed R11: 40k, Resistor_SMD:R_0603_1608Metric_Pad0.98x0.95mm_HandSolder
- removed R14, R15, R20, R22: OR 1M, Resistor_SMD:R_0603_1608Metric_Pad0.98x0.95mm_HandSolder
- removed R16: 2.2, Resistor_SMD:R_0603_1608Metric_Pad0.98x0.95mm_HandSolder
- removed R17: 1.5k, Resistor_SMD:R_0603_1608Metric_Pad0.98x0.95mm_HandSolder
- removed R18, R19: 22, Resistor_SMD:R_0603_1608Metric_Pad0.98x0.95mm_HandSolder
- removed R21: 1M, Resistor_SMD:R_0603_1608Metric_Pad0.98x0.95mm_HandSolder
- removed R23, R24: 3.9K, Resistor_SMD:R_0603_1608Metric_Pad0.98x0.95mm_HandSolder
- removed R3: 100, Resistor_SMD:R_0805_2012Metric_Pad1.20x1.40mm_HandSolder
- removed R4: 10k, Resistor_SMD:R_0805_2012Metric_Pad1.20x1.40mm_HandSolder
- removed R5: 10K, Resistor_SMD:R_0805_2012Metric_Pad1.20x1.40mm_HandSolder
- removed R6: 100K, Resistor_SMD:R_0603_1608Metric_Pad0.98x0.95mm_HandSolder
- removed R7: 56K, Resistor_SMD:R_0603_1608Metric_Pad0.98x0.95mm_HandSolder
- removed R8: 1K, Resistor_SMD:R_0603_1608Metric_Pad0.98x0.95mm_HandSolder
- removed RV1: 100k, footprints:TRIM_3361P-1-104GLF
- removed SW1: H/L_DIP_SW, Button_Switch_THT:SW_DIP_SPSTx01_Slide_6.7x4.1mm_W7.62mm_P2.54mm_LowProfile
- removed TP1, TP10, TP11, TP12, TP13, TP14, TP15, TP16, TP17, TP18, TP19, TP2, TP20, TP21, TP22, TP23, TP24, TP25, TP26, TP27, TP28, TP29, TP3, TP31, TP34, TP35, TP36, TP38, TP39, TP4, TP44, TP45, TP46, TP47, TP5, TP6, TP7, TP8, TP9: Test Point, TestPoint:TestPoint_Pad_D1.0mm
- removed TX1: DRA818V, footprints:DORJI_DRA818V
- removed U1: MAX17048G+T10, MAX17048G_T10:SON50P200X200X80-9N
- removed U4: SAM-M8Q, RF_GPS:ublox_SAM-M8Q
- removed U5: PCM2902C, Package_SO:SSOP-28_5.3x10.2mm_P0.65mm
- removed VR2: LD29150PTR, footprints:LD29150PTR
- added C35: 100nF, Capacitor_SMD:C_0603_1608Metric_Pad1.08x0.95mm_HandSolder, B.Cu at (38.9, 39.9)
- added C38: 0.1uF, Capacitor_SMD:C_0603_1608Metric_Pad1.08x0.95mm_HandSolder, F.Cu at (64.8, 55.1)
- added C39: 0.1uF, Capacitor_SMD:C_0603_1608Metric_Pad1.08x0.95mm_HandSolder, F.Cu at (72.4, 55.1)
- added CPU2: Pi Zero/Zero W, Connector_PinSocket_2.54mm:PinSocket_2x20_P2.54mm_Vertical, B.Cu at (41.7, 42.7)
- added I2C1: I2C0, Connector_PinHeader_2.00mm:PinHeader_1x04_P2.00mm_Vertical, F.Cu at (52.8, 54.1)
- added I2C2: I2C0, Connector_PinHeader_2.00mm:PinHeader_1x04_P2.00mm_Vertical, F.Cu at (59.4, 54.1)
- added I2C3: I2C0, Connector_PinHeader_2.00mm:PinHeader_1x04_P2.00mm_Vertical, F.Cu at (56.1, 54.1)
- added PR1: R, Resistor_SMD:R_0603_1608Metric_Pad0.98x0.95mm_HandSolder, F.Cu at (47.6, 45.5)
- added PR2: R, Resistor_SMD:R_0603_1608Metric_Pad0.98x0.95mm_HandSolder, F.Cu at (43.4, 45.5)
- added R25: 4.7k, Resistor_SMD:R_0603_1608Metric_Pad0.98x0.95mm_HandSolder, F.Cu at (50.3, 49.5)
- added SPI1: SPI, Connector_PinHeader_2.00mm:PinHeader_1x06_P2.00mm_Vertical, F.Cu at (67.1, 56.1)
- added SPI2: SPI, Connector_PinHeader_2.00mm:PinHeader_1x06_P2.00mm_Vertical, F.Cu at (70.1, 56.1)
- added TP43: Test Point, TestPoint:TestPoint_Pad_D1.0mm, F.Cu at (50.3, 46.7)
- C14, C21: value 1uF -> 0.1uF
- C15: value 0.1uF -> 100uF; footprint Capacitor_SMD:C_0603_1608Metric_Pad1.08x0.95mm_HandSolder -> Capacitor_THT:CP_Radial_D6.3mm_P2.50mm
- C16: value 0.1uF -> 1uF; moved to B.Cu
- C17, D1, VR1: moved to B.Cu
- C18: value 0.33uF -> 0.1uF; moved to B.Cu
- C19: value 10uF -> 0.1uF; footprint Capacitor_SMD:C_0805_2012Metric_Pad1.18x1.45mm_HandSolder -> Capacitor_SMD:C_0603_1608Metric_Pad1.08x0.95mm_HandSolder
- C22, C23: value 4.7uF -> 0.1uF
- J2: value USB -> BAT; footprint Connector_PinHeader_2.54mm:PinHeader_1x04_P2.54mm_Vertical -> Connector_PinHeader_2.54mm:PinHeader_1x02_P2.54mm_Vertical
- R12: value 100k -> 3.9K
- R13: value ? -> 3.9K
- TMP1, TMP2, TMP3: value DS18B20 - Connector -> 1-Wire Bus; footprint Connector_JST:JST_XH_B3B-XH-AM_1x03_P2.50mm_Vertical -> Connector_PinHeader_2.00mm:PinHeader_1x03_P2.00mm_Vertical
- U2: value LTV-356T -> MAX17048G+T10; footprint Package_SO:SO-4_4.4x3.6mm_P2.54mm -> MAX17048G_T10:SON50P200X200X80-9N
- U3: value BMP390L -> CAT24C32WI-GT3; footprint BMP390:XDCR_BMP390L -> footprints:SOIC127P600X175-8N
- U6: value CAT24C32WI-GT3 -> BME280; footprint footprints:SOIC127P600X175-8N -> footprints:PSON65P250X250X100-8N
- moved R12 75.5 mm to (94.2, 43.2), turned to 180 degrees
- moved C14 71.6 mm to (61.3, 64.5), turned to 180 degrees
- moved C19 69.0 mm to (90.4, 47.2), turned to 90 degrees
- moved U2 67.0 mm to (62.5, 62.0), turned to 90 degrees
- moved U3 63.4 mm to (94.5, 48.8), turned to 90 degrees
- moved C22 49.6 mm to (44.8, 51.4)
- moved TMP3 47.7 mm to (56.1, 46.5)
- moved C21 47.4 mm to (42.2, 50.6), turned to 90 degrees
- moved U6 46.1 mm to (44.7, 49.0), turned to 90 degrees
- moved TMP1 46.1 mm to (52.8, 46.5)
- moved TMP2 41.7 mm to (59.4, 46.5)
- moved J2 38.5 mm to (46.0, 61.7), turned to 90 degrees
- moved C34 38.3 mm to (58.4, 62.5), turned to 0 degrees
- moved D1 34.5 mm to (41.1, 65.8), turned to 0 degrees
- moved C23 32.8 mm to (61.7, 49.8), turned to 90 degrees
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Connections:
- C14 pad 1: Net-(C14-Pad1) -> VCC
- C14 pad 2: Net-(C14-Pad2) -> GND
- C15 pad 1: +3V3 -> /GFC_HAT/Power/VCC_P
- C16 pad 1: +3V3 -> /GFC_HAT/Power/VCC_P
- C17 pad 1: GND -> /GFC_HAT/Power/VCC_P
- C17 pad 2: +3V3 -> GND
- C19 pad 1: +4V3 -> GND
- C19 pad 2: GND -> +3V3
- C21 pad 1: Net-(C21-Pad1) -> GND
- C21 pad 2: GND -> +3V3
- C22 pad 1: Net-(C22-Pad1) -> +3V3
- C22 pad 2: /DAC/AUDIO.SC_IN_L -> GND
- C23 pad 1: Net-(C23-Pad1) -> +3V3
- C23 pad 2: /DAC/AUDIO.SC_IN_R -> GND
- D1 pad 1: /Power/VCC_P -> /GFC_HAT/Power/VCC_P
- J2 pad 1: GND -> VCC
- J2 pad 2: /DAC/V_BUS -> GND
- R12 pad 1: +4V3 -> EEPROM.SCL
- R12 pad 2: Net-(R11-Pad1) -> +3V3
- R13 pad 1: Net-(Q1-Pad1) -> EEPROM.SDA
- R13 pad 2: GPIO.DRA_PWR_CONTROL -> +3V3
- U2 pad 1: Net-(R3-Pad1) -> GND
- U2 pad 2: Net-(Q1-Pad2) -> VCC
- U2 pad 3: /DRA818/4V3 Controlled -> +3V3
- U2 pad 4: +4V3 -> GND
- U3 pad 1: +3V3 -> GND
- U3 pad 2: I2C0.SCL -> GND
- U3 pad 4: I2C0.SDA -> GND
- U3 pad 5: GND -> EEPROM.SDA
- U3 pad 6: +3V3 -> EEPROM.SCL
- U3 pad 8: GND -> +3V3
- U6 pad 2: GND -> +3V3
- U6 pad 3: GND -> I2C0.SDA
- U6 pad 4: GND -> I2C0.SCL
- U6 pad 5: EEPROM.SDA -> GND
- U6 pad 6: EEPROM.SCL -> +3V3
- U6 pad 7: unconnected-(U6-Pad7) -> GND
- VR1 pad 1: /Power/VCC_P -> /GFC_HAT/Power/VCC_P
Routing:
- net +4V3: track 169.7 -> 0.00 mm
- net UART0.PI_TXD: track 169.4 -> 0.00 mm, vias 4 -> 0
- net UART0.PI_RXD: track 160.7 -> 0.00 mm, vias 4 -> 0
- net +3V3: track 246.4 -> 166.3 mm, vias 14 -> 2
- net 1-Wire: track 81.7 -> 15.5 mm
- net I2C0.SCL: track 100.5 -> 34.7 mm, vias 4 -> 0
- net /DAC/AUDIO.SC_IN_R: track 53.6 -> 0.00 mm
- net I2C0.SDA: track 85.2 -> 34.9 mm, vias 5 -> 0
- net GND: track 97.6 -> 48.9 mm, vias 31 -> 68
- net GPIO.DRA_SQ: track 38.8 -> 0.00 mm, vias 2 -> 0
- net +5V: track 58.1 -> 22.7 mm
- net Net-(C29-Pad1): track 29.8 -> 0.00 mm, vias 2 -> 0
- net /Power/VCC_P: track 25.9 -> 0.00 mm
- net /DAC/AUDIO.SC_OUT_R: track 22.4 -> 0.00 mm, vias 2 -> 0
- net GPIO.DRA_PTT: track 22.4 -> 0.00 mm
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Other:
- board outline added: 65 x 30 mm
- board text added: "GFC V0.1"
- board text added: "HAT"
- board text added: "github.com/joshua-jerred/Giraffe"

Commit message: Hardware Update
Parts:
- added G***: LOGO, footprints:logo, F.Cu at (82.0, 52.6)
Routing:
- net GND: vias 68 -> 67
Other:
- board text added: "GFC PROTOTYPE 1"
- board text removed: "GFC V0.1"
