File: hardware/GFC/DRA818.kicad_sch (KiCad schematic)
At the start: 38 parts, among them Q1 Q_NPN_BCE, Q2 DMN67D8LW-13, Q3 Q_NPN_BCE, SW1 H/L_DIP_SW, U2 LTV-356T

Commit message: Cleaning up the hardware directory
Changed lines of the file:
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@@
   (junction (at 119.38 123.19) (diameter 0) (color 0 0 0 0)
   )
+  (junction (at 154.94 31.75) (diameter 0) (color 0 0 0 0)
+  )
   (bus_entry (at 214.63 107.95) (size -2.54 2.54)
     (stroke (width 0) (type default) (color 0 0 0 0))
@@
     (stroke (width 0) (type default) (color 0 0 0 0))
   )
-  (wire (pts (xy 166.37 31.75) (xy 110.49 31.75))
+  (wire (pts (xy 166.37 31.75) (xy 154.94 31.75))
     (stroke (width 0) (type default) (color 0 0 0 0))
   )
@@
   )
   (wire (pts (xy 165.1 66.04) (xy 165.1 73.66))
+    (stroke (width 0) (type default) (color 0 0 0 0))
+  )
+  (wire (pts (xy 154.94 31.75) (xy 110.49 31.75))
     (stroke (width 0) (type default) (color 0 0 0 0))
   )
@@
     (pin "2")
   )
+  (symbol (lib_id "power:PWR_FLAG") (at 154.94 31.75 0) (unit 1)
+    (in_bom yes) (on_board yes) (fields_autoplaced)
+    (property "Reference" "#FLG0106" (id 0) (at 154.94 29.845 0)
+      (effects (font (size 1.27 1.27)) hide)
+    )
+    (property "Value" "PWR_FLAG" (id 1) (at 154.94 26.67 0))
+    (property "Footprint" "" (id 2) (at 154.94 31.75 0)
+      (effects (font (size 1.27 1.27)) hide)
+    )
+    (property "Datasheet" "~" (id 3) (at 154.94 31.75 0)
+      (effects (font (size 1.27 1.27)) hide)
+    )
+    (pin "1")
+  )
   (symbol (lib_id "Transistor_FET:2N7002K") (at 44.45 96.52 270) (unit 1)

Commit message: Update
Parts:
- renumbered C6 to C25, C7 to C26, C14 to C27, C8 to C28, C9 to C29, C10 to C30, C11 to C31, C12 to C32, C13 to C33, Q2 to Q1, Q3 to Q2, Q1 to Q3, R4 to R16, R5 to R17, R6 to R18, R7 to R19, R8 to R20, R3 to R21, R13 to R22, TP1 to TP29, TP19 to TP30, TP20 to TP31, TP21 to TP32, TP22 to TP33, TP23 to TP34, TP24 to TP35, TP25 to TP36, TP26 to TP37, TP27 to TP38, TP28 to TP39, U2 to U5
