File: hardware/GFC/GFC_HAT.kicad_sch (KiCad schematic)
At the start: 30 parts, among them U3 CAT24C32WI-GT3, U6 BME280

Commit message: Hardware Update
Parts:
- removed TP40: Test Point, TestPoint:TestPoint_Pad_D1.0mm, symbol Connector:TestPoint_Small
- added C24, C40: 0.1uF, Capacitor_SMD:C_0603_1608Metric_Pad1.08x0.95mm_HandSolder, symbol Device:C
- gave numbers to parts that had none: 2
- renumbered Op_R3 to PR1, Op_R4 to PR2
Connections:
- net VCC is gone; now on net +3V3: C20.2, U4.17 (VCC), U4.2 (VCC_IO), U4.3 (V_BCKP)
- net +3V3: now also C24.1, C40.1
- net GND: now also C24.2, C40.2

Commit message: Update
Other:
- removed sheet SAM-M8Q (I2C)
Changed lines of the file:
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@@
-    (stroke (width 0) (type default) (color 0 0 0 0))
-  )
-  (bus (pts (xy 85.09 30.48) (xy 83.82 30.48))
     (stroke (width 0) (type default) (color 0 0 0 0))
   )
@@
   )
   (wire (pts (xy 157.48 73.66) (xy 157.48 72.39))
-    (stroke (width 0) (type default) (color 0 0 0 0))
-  )
-  (wire (pts (xy 81.28 22.86) (xy 85.09 22.86))
     (stroke (width 0) (type default) (color 0 0 0 0))
   )
@@
     (property "Intersheet References" "${INTERSHEET_REFS}" (id 0) (at 283.1436 45.7994 0)
       (effects (font (size 1.27 1.27)) (justify left) hide)
-    )
-  )
-  (global_label "I2C0{SDA SCL}" (shape input) (at 83.82 30.48 180) (fields_autoplaced)
-    (effects (font (size 1.27 1.27)) (justify right))
-    (property "Intersheet References" "${INTERSHEET_REFS}" (id 0) (at 67.3764 30.5594 0)
-      (effects (font (size 1.27 1.27)) (justify right) hide)
     )
   )
@@
     (pin "2")
     (pin "3")
-  )
-  (symbol (lib_id "power:+3V3") (at 81.28 22.86 0) (unit 1)
-    (in_bom yes) (on_board yes) (fields_autoplaced)
-    (property "Reference" "#PWR0181" (id 0) (at 81.28 26.67 0)
-      (effects (font (size 1.27 1.27)) hide)
-    )
-    (property "Value" "+3V3" (id 1) (at 81.28 17.78 0))
-    (property "Footprint" "" (id 2) (at 81.28 22.86 0)
-      (effects (font (size 1.27 1.27)) hide)
-    )
-    (property "Datasheet" "" (id 3) (at 81.28 22.86 0)
-      (effects (font (size 1.27 1.27)) hide)
-    )
-    (pin "1")
   )
   (symbol (lib_id "power:+3V3") (at 204.47 22.86 0) (unit 1)
@@
     )
   )
-  (sheet (at 85.09 17.78) (size 22.86 19.05) (fields_autoplaced)
-    (stroke (width 0.1524) (type solid) (color 0 0 0 0))
-    (fill (color 0 0 0 0.0000))
-    (property "Sheet name" "SAM-M8Q (I2C)" (id 0) (at 85.09 17.0684 0)
-      (effects (font (size 1.27 1.27)) (justify left bottom))
-    )
-    (property "Sheet file" "SAM-M8Q.kicad_sch" (id 1) (at 85.09 37.4146 0)
-      (effects (font (size 1.27 1.27)) (justify left top))
-    )
-    (pin "VCC" input (at 85.09 22.86 180)
-      (effects (font (size 1.27 1.27)) (justify left))
-    )
-    (pin "I2C0{SDA SCL}" input (at 85.09 30.48 180)
-      (effects (font (size 1.27 1.27)) (justify left))
-    )
-  )
