File: hardware/GFC/dac.kicad_sch (KiCad schematic)
At the start: 25 parts, among them J2 USB, U5 PCM2902C, Y1 12MHz

Commit message: Cleaning up the hardware directory
Parts:
- added TP46, TP47: Test Point, TestPoint:TestPoint_Pad_D1.0mm, symbol Connector:TestPoint_Small
- C22, C23, C24, C25, C27, C28: footprint (none) -> Capacitor_SMD:C_0603_1608Metric_Pad1.08x0.95mm_HandSolder
- C31, C32: value 10-33pF -> 10pF; footprint (none) -> Capacitor_SMD:C_0603_1608Metric_Pad1.08x0.95mm_HandSolder
- J2: footprint (none) -> Connector_PinHeader_2.54mm:PinHeader_1x04_P2.54mm_Vertical
- R14, R15, R16, R17, R18, R19, R20, R21, R22: footprint (none) -> Resistor_SMD:R_0603_1608Metric_Pad0.98x0.95mm_HandSolder
Connections:
- net AUDIO.SC_IN_L: now also TP46.1
- net AUDIO.SC_OUT_L: now also TP47.1
- no-connect marks 12 -> 10
Changed lines of the file:
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@@
   (junction (at 85.09 114.3) (diameter 0) (color 0 0 0 0)
   )
+  (junction (at 53.34 101.6) (diameter 0) (color 0 0 0 0)
+  )
   (junction (at 166.37 124.46) (diameter 0) (color 0 0 0 0)
   )
@@
   (junction (at 71.12 133.35) (diameter 0) (color 0 0 0 0)
   )
-  (no_connect (at 111.76 160.02))
   (no_connect (at 124.46 96.52))
-  (no_connect (at 104.14 160.02))
   (no_connect (at 177.8 62.23))
   (no_connect (at 88.9 109.22))
@@
     (stroke (width 0) (type default) (color 0 0 0 0))
   )
+  (wire (pts (xy 53.34 93.98) (xy 53.34 101.6))
+    (stroke (width 0) (type default) (color 0 0 0 0))
+  )
   (wire (pts (xy 128.27 129.54) (xy 128.27 130.81))
     (stroke (width 0) (type default) (color 0 0 0 0))
@@
     (stroke (width 0) (type default) (color 0 0 0 0))
   )
+  (wire (pts (xy 53.34 101.6) (xy 59.69 101.6))
+    (stroke (width 0) (type default) (color 0 0 0 0))
+  )
   (wire (pts (xy 124.46 99.06) (xy 128.27 99.06))
     (stroke (width 0) (type default) (color 0 0 0 0))
@@
     (stroke (width 0) (type default) (color 0 0 0 0))
   )
-  (wire (pts (xy 45.72 101.6) (xy 59.69 101.6))
+  (wire (pts (xy 45.72 101.6) (xy 53.34 101.6))
     (stroke (width 0) (type default) (color 0 0 0 0))
   )
@@
     (property "Reference" "R18" (id 0) (at 83.82 95.25 90))
     (property "Value" "22" (id 1) (at 74.93 95.25 90))
-    (property "Footprint" "" (id 2) (at 80.01 98.298 90)
+    (property "Footprint" "Resistor_SMD:R_0603_1608Metric_Pad0.98x0.95mm_HandSolder" (id 2) (at 80.01 98.298 90)
       (effects (font (size 1.27 1.27)) hide)
     )
@@
       (effects (font (size 1.27 1.27)) (justify left))
     )
-    (property "Footprint" "" (id 2) (at 60.452 132.08 90)
+    (property "Footprint" "Resistor_SMD:R_0603_1608Metric_Pad0.98x0.95mm_HandSolder" (id 2) (at 60.452 132.08 90)
       (effects (font (size 1.27 1.27)) hide)
     )
@@
     (property "Reference" "C24" (id 0) (at 76.2 120.65 90))
     (property "Value" "10uF" (id 1) (at 83.82 120.65 90))
-    (property "Footprint" "" (id 2) (at 80.01 119.38 0)
+    (property "Footprint" "Capacitor_SMD:C_0603_1608Metric_Pad1.08x0.95mm_HandSolder" (id 2) (at 80.01 119.38 0)
       (effects (font (size 1.27 1.27)) hide)
     )
@@
     (property "Reference" "R16" (id 0) (at 67.31 100.33 90))
     (property "Value" "2.2" (id 1) (at 58.42 100.33 90))
-    (property "Footprint" "" (id 2) (at 63.5 103.378 90)
+    (property "Footprint" "Resistor_SMD:R_0603_1608Metric_Pad0.98x0.95mm_HandSolder" (id 2) (at 63.5 103.378 90)
       (effects (font (size 1.27 1.27)) hide)
     )
@@
       (effects (font (size 1.27 1.27)) (justify left))
     )
-    (property "Value" "10-33pF" (id 1) (at 175.26 113.03 90)
-      (effects (font (size 1.27 1.27)) (justify left))
-    )
-    (property "Footprint" "" (id 2) (at 163.83 113.03 0)
+    (property "Value" "10pF" (id 1) (at 175.26 113.03 90)
+      (effects (font (size 1.27 1.27)) (justify left))
+    )
+    (property "Footprint" "Capacitor_SMD:C_0603_1608Metric_Pad1.08x0.95mm_HandSolder" (id 2) (at 163.83 113.03 0)
       (effects (font (size 1.27 1.27)) hide)
     )
@@
       (effects (font (size 1.27 1.27)) (justify left))
     )
-    (property "Footprint" "" (id 2) (at 68.072 83.82 90)
+    (property "Footprint" "Resistor_SMD:R_0603_1608Metric_Pad0.98x0.95mm_HandSolder" (id 2) (at 68.072 83.82 90)
       (effects (font (size 1.27 1.27)) hide)
     )
@@
     (property "Reference" "C27" (id 0) (at 132.08 125.73 90))
     (property "Value" "4.7uF" (id 1) (at 138.43 125.73 90))
-    (property "Footprint" "" (id 2) (at 134.62 127 0)
+    (property "Footprint" "Capacitor_SMD:C_0603_1608Metric_Pad1.08x0.95mm_HandSolder" (id 2) (at 134.62 127 0)
       (effects (font (size 1.27 1.27)) hide)
     )
@@
     (property "Reference" "R21" (id 0) (at 133.35 115.57 90))
     (property "Value" "1M" (id 1) (at 144.78 115.57 90))
-    (property "Footprint" "" (id 2) (at 139.7 117.348 90)
+    (property "Footprint" "Resistor_SMD:R_0603_1608Metric_Pad0.98x0.95mm_HandSolder" (id 2) (at 139.7 117.348 90)
       (effects (font (size 1.27 1.27)) hide)
     )
@@
     (pin "1")
     (pin "2")
+  )
+  (symbol (lib_id "Connector:TestPoint_Small") (at 111.76 160.02 270) (unit 1)
+    (in_bom yes) (on_board yes)
+    (property "Reference" "TP47" (id 0) (at 113.03 156.21 0)
+      (effects (font (size 1.27 1.27)) (justify left))
+    )
+    (property "Value" "Test Point" (id 1) (at 110.4901 161.29 0)
+      (effects (font (size 1.27 1.27)) (justify left) hide)
+    )
+    (property "Footprint" "TestPoint:TestPoint_Pad_D1.0mm" (id 2) (at 111.76 165.1 0)
+      (effects (font (size 1.27 1.27)) hide)
+    )
+    (property "Datasheet" "~" (id 3) (at 111.76 165.1 0)
+      (effects (font (size 1.27 1.27)) hide)
+    )
+    (pin "1")
+  )
+  (symbol (lib_id "power:PWR_FLAG") (at 53.34 93.98 0) (unit 1)
+    (in_bom yes) (on_board yes) (fields_autoplaced)
+    (property "Reference" "#FLG0105" (id 0) (at 53.34 92.075 0)
+      (effects (font (size 1.27 1.27)) hide)
+    )
+    (property "Value" "PWR_FLAG" (id 1) (at 53.34 88.9 0))
+    (property "Footprint" "" (id 2) (at 53.34 93.98 0)
+      (effects (font (size 1.27 1.27)) hide)
+    )
+    (property "Datasheet" "~" (id 3) (at 53.34 93.98 0)
+      (effects (font (size 1.27 1.27)) hide)
+    )
+    (pin "1")
   )
   (symbol (lib_id "Device:Crystal") (at 156.21 116.84 90) (unit 1)
@@
       (effects (font (size 1.27 1.27)) (justify left))
     )
-    (property "Footprint" "" (id 2) (at 141.732 130.81 90)
+    (property "Footprint" "Resistor_SMD:R_0603_1608Metric_Pad0.98x0.95mm_HandSolder" (id 2) (at 141.732 130.81 90)
       (effects (font (size 1.27 1.27)) hide)
     )
@@
     (property "Reference" "J2" (id 0) (at 40.64 90.17 0))
     (property "Value" "USB" (id 1) (at 40.64 92.71 0))
-    (property "Footprint" "" (id 2) (at 40.64 101.6 0)
+    (property "Footprint" "Connector_PinHeader_2.54mm:PinHeader_1x04_P2.54mm_Vertical" (id 2) (at 40.64 101.6 0)
       (effects (font (size 1.27 1.27)) hide)
     )
@@
     (property "Reference" "C25" (id 0) (at 76.2 134.62 90))
     (property "Value" "10uF" (id 1) (at 83.82 134.62 90))
-    (property "Footprint" "" (id 2) (at 80.01 133.35 0)
+    (property "Footprint" "Capacitor_SMD:C_0603_1608Metric_Pad1.08x0.95mm_HandSolder" (id 2) (at 80.01 133.35 0)
       (effects (font (size 1.27 1.27)) hide)
     )
@@
     (property "Reference" "C22" (id 0) (at 73.66 125.73 90))
     (property "Value" "4.7uF" (id 1) (at 81.28 125.73 90))
-    (property "Footprint" "" (id 2) (at 77.47 124.46 0)
+    (property "Footprint" "Capacitor_SMD:C_0603_1608Metric_Pad1.08x0.95mm_HandSolder" (id 2) (at 77.47 124.46 0)
       (effects (font (size 1.27 1.27)) hide)
     )
@@
     (property "Reference" "R19" (id 0) (at 83.82 97.79 90))
     (property "Value" "22" (id 1) (at 74.93 97.79 90))
-    (property "Footprint" "" (id 2) (at 80.01 100.838 90)
+    (property "Footprint" "Resistor_SMD:R_0603_1608Metric_Pad0.98x0.95mm_HandSolder" (id 2) (at 80.01 100.838 90)
       (effects (font (size 1.27 1.27)) hide)
     )
@@
     (property "Reference" "C28" (id 0) (at 132.08 129.54 90))
     (property "Value" "4.7uF" (id 1) (at 138.43 129.54 90))
-    (property "Footprint" "" (id 2) (at 134.62 130.81 0)
+    (property "Footprint" "Capacitor_SMD:C_0603_1608Metric_Pad1.08x0.95mm_HandSolder" (id 2) (at 134.62 130.81 0)
       (effects (font (size 1.27 1.27)) hide)
     )
@@
     (pin "1")
   )
+  (symbol (lib_id "Connector:TestPoint_Small") (at 104.14 160.02 180) (unit 1)
+    (in_bom yes) (on_board yes)
+    (property "Reference" "TP46" (id 0) (at 107.95 161.29 0)
+      (effects (font (size 1.27 1.27)) (justify left))
+    )
+    (property "Value" "Test Point" (id 1) (at 102.87 158.7501 0)
+      (effects (font (size 1.27 1.27)) (justify left) hide)
+    )
+    (property "Footprint" "TestPoint:TestPoint_Pad_D1.0mm" (id 2) (at 99.06 160.02 0)
+      (effects (font (size 1.27 1.27)) hide)
+    )
+    (property "Datasheet" "~" (id 3) (at 99.06 160.02 0)
+      (effects (font (size 1.27 1.27)) hide)
+    )
+    (pin "1")
+  )
   (symbol (lib_id "Device:C_Polarized_Small") (at 77.47 128.27 270) (unit 1)
     (in_bom yes) (on_board yes)
     (property "Reference" "C23" (id 0) (at 73.66 129.54 90))
     (property "Value" "4.7uF" (id 1) (at 81.28 129.54 90))
-    (property "Footprint" "" (id 2) (at 77.47 128.27 0)
+    (property "Footprint" "Capacitor_SMD:C_0603_1608Metric_Pad1.08x0.95mm_HandSolder" (id 2) (at 77.47 128.27 0)
       (effects (font (size 1.27 1.27)) hide)
     )
@@
       (effects (font (size 1.27 1.27)) (justify right))
     )
-    (property "Footprint" "" (id 2) (at 58.928 128.27 90)
+    (property "Footprint" "Resistor_SMD:R_0603_1608Metric_Pad0.98x0.95mm_HandSolder" (id 2) (at 58.928 128.27 90)
       (effects (font (size 1.27 1.27)) hide)
     )
@@
       (effects (font (size 1.27 1.27)) (justify left))
     )
-    (property "Value" "10-33pF" (id 1) (at 175.26 119.38 90)
-      (effects (font (size 1.27 1.27)) (justify left))
-    )
-    (property "Footprint" "" (id 2) (at 163.83 120.65 0)
+    (property "Value" "10pF" (id 1) (at 175.26 119.38 90)
+      (effects (font (size 1.27 1.27)) (justify left))
+    )
+    (property "Footprint" "Capacitor_SMD:C_0603_1608Metric_Pad1.08x0.95mm_HandSolder" (id 2) (at 163.83 120.65 0)
       (effects (font (size 1.27 1.27)) hide)
     )
@@
       (effects (font (size 1.27 1.27)) (justify left))
     )
-    (property "Footprint" "" (id 2) (at 136.652 137.16 90)
-      (effects (font (size 1.27 1.27)) hide)
-    )
+    (property "Footprint" "Resistor_SMD:R_0603_1608Metric_Pad0.98x0.95mm_HandSolder" (id 2) (at 136.652 137.16 90)
+      (effects (font (size 1.27 1.27)) hide)
+    )

Commit message: Update
Parts:
- renumbered C21 to C1, C30 to C10, C31 to C11, C32 to C12, C33 to C13, C22 to C2, C23 to C3, C24 to C4, C25 to C5, C26 to C6, C27 to C7, C28 to C8, C29 to C9, J2 to J1, R21 to R10, R22 to R11, R14 to R3, R15 to R4, R16 to R5, R17 to R6, R18 to R7, R19 to R8, R20 to R9, TP46 to TP1, TP47 to TP19, U5 to U1
