File: hardware/GFC Shoe/GFC Shoe.kicad_pcb (KiCad board)
At the start: 4 copper layers, 65.8 x 30 mm, 51 parts, among them J1 USB, K1 TLP241A, Q1 BSS138, Q2 BSS138, Q3 DMN67D8LW-13, Q4 Q_NPN_BCE, U1 PCM2902C, Y1 12MHz

Commit message: Minor hardware updates
Parts:
- AE1: moved to B.Cu
- J1: footprint Connector_PinHeader_2.54mm:PinHeader_1x04_P2.54mm_Vertical -> Connector_PinHeader_2.54mm:PinHeader_1x02_P2.54mm_Vertical_SMD_Pin1Left
- R6: moved to F.Cu
- Y1: value 12MHz -> Crystal ECS33B; footprint Crystal:Crystal_SMD_HC49-SD_HandSoldering -> Crystal:Crystal_SMD_3225-4Pin_3.2x2.5mm
- moved R12 81.6 mm to (90.5, 36.7), turned to 180 degrees
- moved C14 73.4 mm to (99.9, 49.4), turned to -90 degrees
- moved U1 71.1 mm to (93.5, 43.2)
- moved R13 68.5 mm to (86.7, 37.3)
- moved C9 63.5 mm to (87.4, 41.7), turned to -90 degrees
- moved C12 60.2 mm to (85.3, 45.4), turned to 180 degrees
- moved C10 59.8 mm to (86.4, 48.2), turned to 180 degrees
- moved J1 59.0 mm to (81.3, 39.6), turned to 180 degrees
- moved R14 58.4 mm to (86.7, 38.9)
- moved C11 57.6 mm to (87.4, 50.2), turned to 180 degrees
- moved R15 55.3 mm to (99.8, 43.4), turned to 90 degrees
- moved C21 54.2 mm to (101.9, 49.4), turned to -90 degrees
- moved C17 52.9 mm to (98.3, 36.6)
- moved R11 50.9 mm to (85.6, 41.7), turned to 90 degrees
- moved C16 50.5 mm to (95.8, 50.7), turned to -90 degrees
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Connections:
- net /Sound Card/IN_Left renamed /Sound Card/Audio In Left
- J1 pad 1: /Sound Card/V_BUS -> /Sound Card/D-
- J1 pad 2: /Sound Card/D- -> /Sound Card/D+
- PI_HDR1 pad 11: unconnected-(PI_HDR1-Pad11) -> Radio Power Control
- PI_HDR1 pad 16: /SA868/GPIO SQ -> unconnected-(PI_HDR1-Pad16)
- PI_HDR1 pad 18: /SA868/GPIO PTT -> unconnected-(PI_HDR1-Pad18)
- PI_HDR1 pad 22: /SA868/GPIO PWR_CTRL -> unconnected-(PI_HDR1-Pad22)
- PI_HDR1 pad 31: unconnected-(PI_HDR1-Pad31) -> GPIO PTT
- PI_HDR1 pad 40: unconnected-(PI_HDR1-Pad40) -> GPIO SQ
- Q1 pad 1: +3.3V -> +3V3
- Q2 pad 1: +3.3V -> +3V3
- Q4 pad 2: /SA868/GPIO SQ -> GPIO SQ
- R1 pad 2: /SA868/GPIO PWR_CTRL -> Radio Power Control
- R10 pad 1: +3.3V -> +3V3
- R10 pad 2: /SA868/GPIO SQ -> GPIO SQ
- R11 pad 1: /Sound Card/V_BUS -> +5V
- R2 pad 1: +3.3V -> +3V3
- R3 pad 1: +3.3V -> +3V3
- R8 pad 1: /SA868/GPIO PTT -> GPIO PTT
- Y1 pad 2: Net-(C19-Pad1) -> GND
Routing:
- net +3V3: track 0.00 -> 61.8 mm, vias 0 -> 2
- net /SA868/RXD 5V: track 0.00 -> 49.9 mm, vias 0 -> 2
- net /SA868/TXD 5V: track 0.00 -> 49.5 mm, vias 0 -> 2
- net +5V: track 0.00 -> 49.3 mm, vias 0 -> 1
- net 5VC: track 0.00 -> 32.5 mm, vias 0 -> 3
- net /SA868/A_OUT: track 0.00 -> 29.9 mm, vias 0 -> 2
- net /SA868/A_IN: track 0.00 -> 24.5 mm, vias 0 -> 2
- net GND: track 0.00 -> 20.5 mm, vias 0 -> 496
- net Net-(K1-Pad1): track 0.00 -> 19.1 mm, vias 0 -> 2
- net Net-(C17-Pad1): track 0.00 -> 19.1 mm
- net /SA868/RF OUT: track 0.00 -> 14.9 mm
- net /Sound Card/D+: track 0.00 -> 11.2 mm
- net Net-(R15-Pad1): track 0.00 -> 11.0 mm
- net GPIO SQ: track 0.00 -> 10.8 mm
- net /SA868/Radio UART RX: track 0.00 -> 8.38 mm, vias 0 -> 1
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- added copper zone on B.Cu, net GND
- added copper zone on F.Cu, net GND
- added copper zone on In1.Cu, net GND
- added copper zone on In2.Cu, net GND
Other:
- board size 65.8 x 30 mm -> 65 x 30 mm
