File: hardware/GFC Shoe/SA868.kicad_sch (KiCad schematic)
At the start: 29 parts, among them K1 TLP241A, Q1 BSS138, Q2 BSS138, Q3 DMN67D8LW-13, Q4 Q_NPN_BCE

Commit message: PCB Reference Updates
Parts:
- gave numbers to parts that had none: 1
- renumbered R11 to R10, R8 to R7, R9 to R8, R10 to R9
Changed lines of the file:
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@@
   (symbol (lib_id "Device:R") (at 182.88 118.11 0) (unit 1)
     (in_bom yes) (on_board yes)
-    (property "Reference" "R10" (id 0) (at 179.07 116.84 0)
+    (property "Reference" "R9" (id 0) (at 179.07 116.84 0)
       (effects (font (size 1.27 1.27)) (justify left))
     )
@@
   (symbol (lib_name "GND_8") (lib_id "power:GND") (at 190.5 123.19 0) (unit 1)
     (in_bom yes) (on_board yes) (fields_autoplaced)
-    (property "Reference" "#PWR018" (id 0) (at 190.5 129.54 0)
+    (property "Reference" "#PWR017" (id 0) (at 190.5 129.54 0)
       (effects (font (size 1.27 1.27)) hide)
     )
@@
   (symbol (lib_name "GND_1") (lib_id "power:GND") (at 190.5 85.09 0) (mirror y) (unit 1)
     (in_bom yes) (on_board yes)
-    (property "Reference" "#PWR016" (id 0) (at 190.5 91.44 0)
+    (property "Reference" "#PWR015" (id 0) (at 190.5 91.44 0)
       (effects (font (size 1.27 1.27)) hide)
     )
@@
   (symbol (lib_name "GND_5") (lib_id "power:GND") (at 212.725 57.785 0) (unit 1)
     (in_bom yes) (on_board yes)
-    (property "Reference" "#PWR020" (id 0) (at 212.725 64.135 0)
+    (property "Reference" "#PWR019" (id 0) (at 212.725 64.135 0)
       (effects (font (size 1.27 1.27)) hide)
     )
@@
   (symbol (lib_name "GND_10") (lib_id "power:GND") (at 182.88 132.08 0) (unit 1)
     (in_bom yes) (on_board yes)
-    (property "Reference" "#PWR015" (id 0) (at 182.88 138.43 0)
+    (property "Reference" "#PWR014" (id 0) (at 182.88 138.43 0)
       (effects (font (size 1.27 1.27)) hide)
     )
@@
   (symbol (lib_id "Device:R") (at 177.165 114.3 90) (unit 1)
     (in_bom yes) (on_board yes)
-    (property "Reference" "R8" (id 0) (at 177.165 110.49 90))
+    (property "Reference" "R7" (id 0) (at 177.165 110.49 90))
     (property "Value" "100K" (id 1) (at 177.165 112.395 90))
     (property "Footprint" "Resistor_SMD:R_0603_1608Metric_Pad0.98x0.95mm_HandSolder" (id 2) (at 177.165 116.078 90)
@@
   (symbol (lib_name "GND_4") (lib_id "power:GND") (at 197.485 57.785 0) (unit 1)
     (in_bom yes) (on_board yes)
-    (property "Reference" "#PWR019" (id 0) (at 197.485 64.135 0)
+    (property "Reference" "#PWR018" (id 0) (at 197.485 64.135 0)
       (effects (font (size 1.27 1.27)) hide)
     )
@@
   (symbol (lib_id "power:+3.3V") (at 190.5 98.425 0) (unit 1)
     (in_bom yes) (on_board yes)
-    (property "Reference" "#PWR017" (id 0) (at 190.5 102.235 0)
+    (property "Reference" "#PWR016" (id 0) (at 190.5 102.235 0)
       (effects (font (size 1.27 1.27)) hide)
     )
@@
   (symbol (lib_id "Device:R") (at 180.34 142.24 270) (unit 1)
     (in_bom yes) (on_board yes)
-    (property "Reference" "R9" (id 0) (at 180.34 144.145 90))
+    (property "Reference" "R8" (id 0) (at 180.34 144.145 90))
     (property "Value" "10k" (id 1) (at 180.34 146.05 90))
     (property "Footprint" "Resistor_SMD:R_0603_1608Metric_Pad0.98x0.95mm_HandSolder" (id 2) (at 180.34 140.462 90)
@@
   (symbol (lib_name "GND_6") (lib_id "power:GND") (at 235.585 43.815 0) (unit 1)
     (in_bom yes) (on_board yes)
-    (property "Reference" "#PWR021" (id 0) (at 235.585 50.165 0)
+    (property "Reference" "#PWR020" (id 0) (at 235.585 50.165 0)
       (effects (font (size 1.27 1.27)) hide)
     )
@@
   (symbol (lib_name "Antenna_Shield_1") (lib_id "Device:Antenna_Shield") (at 233.045 36.83 0) (unit 1)
     (in_bom yes) (on_board yes) (fields_autoplaced)
-    (property "Reference" "AE?" (id 0) (at 236.22 34.9249 0)
+    (property "Reference" "AE1" (id 0) (at 236.22 34.9249 0)
       (effects (font (size 1.27 1.27)) (justify left))
     )
@@
   (symbol (lib_id "Device:R") (at 190.5 104.14 0) (unit 1)
     (in_bom yes) (on_board yes) (fields_autoplaced)
-    (property "Reference" "R11" (id 0) (at 193.04 102.8699 0)
+    (property "Reference" "R10" (id 0) (at 193.04 102.8699 0)
       (effects (font (size 1.27 1.27)) (justify left))
     )
@@
   (symbol (lib_name "GND_2") (lib_id "power:GND") (at 182.245 57.785 0) (unit 1)
     (in_bom yes) (on_board yes)
-    (property "Reference" "#PWR014" (id 0) (at 182.245 64.135 0)
+    (property "Reference" "#PWR013" (id 0) (at 182.245 64.135 0)
       (effects (font (size 1.27 1.27)) hide)
     )
@@
   (symbol (lib_name "GND_3") (lib_id "power:GND") (at 167.005 57.785 0) (unit 1)
     (in_bom yes) (on_board yes)
-    (property "Reference" "#PWR013" (id 0) (at 167.005 64.135 0)
-      (effects (font (size 1.27 1.27)) hide)
-    )
+    (property "Reference" "#PWR012" (id 0) (at 167.005 64.135 0)
+      (effects (font (size 1.27 1.27)) hide)
+    )

Commit message: Minor hardware updates
Connections:
- net +3.3V renamed +3V3
Changed lines of the file:
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@@
-    (pin "1")
-  )
-  (symbol (lib_id "power:+3.3V") (at 74.295 116.205 0) (unit 1)
-    (in_bom yes) (on_board yes)
-    (property "Reference" "#PWR04" (id 0) (at 74.295 120.015 0)
-      (effects (font (size 1.27 1.27)) hide)
-    )
-    (property "Value" "+3.3V" (id 1) (at 74.295 112.395 0))
-    (property "Footprint" "" (id 2) (at 74.295 116.205 0)
-      (effects (font (size 1.27 1.27)) hide)
-    )
-    (property "Datasheet" "" (id 3) (at 74.295 116.205 0)
-      (effects (font (size 1.27 1.27)) hide)
-    )
     (pin "1")
   )
@@
     (pin "2")
   )
+  (symbol (lib_id "power:+3V3") (at 74.295 135.255 0) (unit 1)
+    (in_bom yes) (on_board yes)
+    (property "Reference" "#PWR?" (id 0) (at 74.295 139.065 0)
+      (effects (font (size 1.27 1.27)) hide)
+    )
+    (property "Value" "+3V3" (id 1) (at 73.66 131.445 0))
+    (property "Footprint" "" (id 2) (at 74.295 135.255 0)
+      (effects (font (size 1.27 1.27)) hide)
+    )
+    (property "Datasheet" "" (id 3) (at 74.295 135.255 0)
+      (effects (font (size 1.27 1.27)) hide)
+    )
+    (pin "1")
+  )
   (symbol (lib_id "Device:C") (at 101.6 85.09 180) (unit 1)
     (in_bom yes) (on_board yes)
@@
     (pin "3")
   )
-  (symbol (lib_id "power:+3.3V") (at 74.295 135.255 0) (unit 1)
-    (in_bom yes) (on_board yes)
-    (property "Reference" "#PWR05" (id 0) (at 74.295 139.065 0)
-      (effects (font (size 1.27 1.27)) hide)
-    )
-    (property "Value" "+3.3V" (id 1) (at 74.295 131.445 0))
-    (property "Footprint" "" (id 2) (at 74.295 135.255 0)
-      (effects (font (size 1.27 1.27)) hide)
-    )
-    (property "Datasheet" "" (id 3) (at 74.295 135.255 0)
-      (effects (font (size 1.27 1.27)) hide)
-    )
-    (pin "1")
-  )
   (symbol (lib_name "GND_11") (lib_id "power:GND") (at 78.74 49.53 0) (mirror y) (unit 1)
     (in_bom yes) (on_board yes)
@@
     (pin "2")
   )
-  (symbol (lib_id "power:+3.3V") (at 190.5 98.425 0) (unit 1)
-    (in_bom yes) (on_board yes)
-    (property "Reference" "#PWR016" (id 0) (at 190.5 102.235 0)
-      (effects (font (size 1.27 1.27)) hide)
-    )
-    (property "Value" "+3.3V" (id 1) (at 190.5 94.615 0))
-    (property "Footprint" "" (id 2) (at 190.5 98.425 0)
-      (effects (font (size 1.27 1.27)) hide)
-    )
-    (property "Datasheet" "" (id 3) (at 190.5 98.425 0)
-      (effects (font (size 1.27 1.27)) hide)
-    )
-    (pin "1")
-  )
   (symbol (lib_id "Device:R") (at 180.34 142.24 270) (unit 1)
     (in_bom yes) (on_board yes)
@@
     (pin "2")
   )
+  (symbol (lib_id "power:+3V3") (at 190.5 98.425 0) (unit 1)
+    (in_bom yes) (on_board yes)
+    (property "Reference" "#PWR?" (id 0) (at 190.5 102.235 0)
+      (effects (font (size 1.27 1.27)) hide)
+    )
+    (property "Value" "+3V3" (id 1) (at 189.865 94.615 0))
+    (property "Footprint" "" (id 2) (at 190.5 98.425 0)
+      (effects (font (size 1.27 1.27)) hide)
+    )
+    (property "Datasheet" "" (id 3) (at 190.5 98.425 0)
+      (effects (font (size 1.27 1.27)) hide)
+    )
+    (pin "1")
+  )
   (symbol (lib_name "GND_2") (lib_id "power:GND") (at 182.245 57.785 0) (unit 1)
     (in_bom yes) (on_board yes)
@@
       (effects (font (size 1.27 1.27)) hide)
     )
+    (pin "1")
+  )
+  (symbol (lib_id "power:+3V3") (at 74.295 116.205 0) (unit 1)
+    (in_bom yes) (on_board yes)
+    (property "Reference" "#PWR?" (id 0) (at 74.295 120.015 0)
+      (effects (font (size 1.27 1.27)) hide)
+    )
+    (property "Value" "+3V3" (id 1) (at 73.66 112.395 0))
+    (property "Footprint" "" (id 2) (at 74.295 116.205 0)
+      (effects (font (size 1.27 1.27)) hide)
+    )
+    (property "Datasheet" "" (id 3) (at 74.295 116.205 0)
+      (effects (font (size 1.27 1.27)) hide)
+    )
