File: hardware/GFC Shoe/Sound Card.kicad_sch (KiCad schematic)
At the start: 21 parts, among them J1 USB, U1 PCM2902C, Y1 12MHz

Commit message: PCB Reference Updates
Parts:
- renumbered R12 to R11, R13 to R12, R14 to R13, R15 to R14, R16 to R15
Changed lines of the file:
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@@
   (symbol (lib_id "power:GND") (at 146.05 101.6 0) (unit 1)
     (in_bom yes) (on_board yes)
-    (property "Reference" "#PWR025" (id 0) (at 146.05 107.95 0)
+    (property "Reference" "#PWR024" (id 0) (at 146.05 107.95 0)
       (effects (font (size 1.27 1.27)) hide)
     )
@@
   (symbol (lib_id "Device:R") (at 80.01 96.52 90) (unit 1)
     (in_bom yes) (on_board yes)
-    (property "Reference" "R14" (id 0) (at 83.82 95.25 90))
+    (property "Reference" "R13" (id 0) (at 83.82 95.25 90))
     (property "Value" "22" (id 1) (at 74.93 95.25 90))
     (property "Footprint" "Capacitor_SMD:C_0603_1608Metric_Pad1.08x0.95mm_HandSolder" (id 2) (at 80.01 98.298 90)
@@
   (symbol (lib_id "power:GND") (at 144.78 123.19 0) (unit 1)
     (in_bom yes) (on_board yes)
-    (property "Reference" "#PWR024" (id 0) (at 144.78 129.54 0)
+    (property "Reference" "#PWR023" (id 0) (at 144.78 129.54 0)
       (effects (font (size 1.27 1.27)) hide)
     )
@@
   (symbol (lib_id "Device:R") (at 63.5 101.6 90) (unit 1)
     (in_bom yes) (on_board yes)
-    (property "Reference" "R12" (id 0) (at 67.31 100.33 90))
+    (property "Reference" "R11" (id 0) (at 67.31 100.33 90))
     (property "Value" "2.2" (id 1) (at 58.42 100.33 90))
     (property "Footprint" "Capacitor_SMD:C_0603_1608Metric_Pad1.08x0.95mm_HandSolder" (id 2) (at 63.5 103.378 90)
@@
   (symbol (lib_id "Device:R") (at 69.85 83.82 0) (unit 1)
     (in_bom yes) (on_board yes)
-    (property "Reference" "R13" (id 0) (at 71.12 82.55 0)
+    (property "Reference" "R12" (id 0) (at 71.12 82.55 0)
       (effects (font (size 1.27 1.27)) (justify left))
     )
@@
   (symbol (lib_id "power:GND") (at 48.26 104.14 0) (unit 1)
     (in_bom yes) (on_board yes) (fields_autoplaced)
-    (property "Reference" "#PWR022" (id 0) (at 48.26 110.49 0)
+    (property "Reference" "#PWR021" (id 0) (at 48.26 110.49 0)
       (effects (font (size 1.27 1.27)) hide)
     )
@@
   (symbol (lib_id "Device:R") (at 139.7 115.57 90) (unit 1)
     (in_bom yes) (on_board yes)
-    (property "Reference" "R16" (id 0) (at 133.35 115.57 90))
+    (property "Reference" "R15" (id 0) (at 133.35 115.57 90))
     (property "Value" "1M" (id 1) (at 144.78 115.57 90))
     (property "Footprint" "Capacitor_SMD:C_0603_1608Metric_Pad1.08x0.95mm_HandSolder" (id 2) (at 139.7 117.348 90)
@@
   (symbol (lib_id "power:GND") (at 71.12 137.16 0) (unit 1)
     (in_bom yes) (on_board yes) (fields_autoplaced)
-    (property "Reference" "#PWR023" (id 0) (at 71.12 143.51 0)
+    (property "Reference" "#PWR022" (id 0) (at 71.12 143.51 0)
       (effects (font (size 1.27 1.27)) hide)
     )
@@
   (symbol (lib_id "Device:R") (at 80.01 99.06 90) (unit 1)
     (in_bom yes) (on_board yes)
-    (property "Reference" "R15" (id 0) (at 83.82 97.79 90))
+    (property "Reference" "R14" (id 0) (at 83.82 97.79 90))
     (property "Value" "22" (id 1) (at 74.93 97.79 90))
     (property "Footprint" "Capacitor_SMD:C_0603_1608Metric_Pad1.08x0.95mm_HandSolder" (id 2) (at 80.01 100.838 90)
@@
   (symbol (lib_id "power:GND") (at 166.37 128.27 0) (unit 1)
     (in_bom yes) (on_board yes)
-    (property "Reference" "#PWR026" (id 0) (at 166.37 134.62 0)
-      (effects (font (size 1.27 1.27)) hide)
-    )
+    (property "Reference" "#PWR025" (id 0) (at 166.37 134.62 0)
+      (effects (font (size 1.27 1.27)) hide)
+    )

Commit message: Minor hardware updates
Parts:
- removed J1: USB, Connector_PinHeader_2.54mm:PinHeader_1x04_P2.54mm_Vertical, symbol Connector_Generic:Conn_01x04
- removed Y1: 12MHz, Crystal:Crystal_SMD_HC49-SD_HandSoldering, symbol Device:Crystal
- added J1: USB, Connector_PinHeader_2.54mm:PinHeader_1x02_P2.54mm_Vertical_SMD_Pin1Left, symbol Connector_Generic:Conn_01x02
- added Y1: Crystal ECS33B, Crystal:Crystal_SMD_3225-4Pin_3.2x2.5mm, symbol GFC-Symbols:Crystal_GND23
Connections:
- net D+: now also J1.2 (Pin_2)
- net D-: now also J1.1 (Pin_1)
- net GND: now also Y1.2, Y1.4
- net at C19.1, R15.2, U1.21 (XTI): now also Y1.3
- net at C20.1, R15.1, U1.20 (XTO): now also Y1.1
- net V_BUS renamed +5V
Other:
- moved on the sheet: C19, C20, C21
