File: hardware/Prototype Boards/5v Power Supply/5v Power Supply.kicad_pcb (KiCad board)
At the start: 2 copper layers, 23.4 x 11.2 mm, 12 parts

Commit message: [pre-commit.ci] auto fixes from pre-commit.com hooks
for more information, see https://pre-commit.ci
Parts:
- GND: footprint TestPoint:TestPoint_Keystone_5019_Minature -> TestPoint:TestPoint_Keystone_5019_Miniature
Changed lines of the file:
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@@
     )
   )
-  (footprint "TestPoint:TestPoint_Keystone_5019_Minature" (layer "B.Cu")
+  (footprint "TestPoint:TestPoint_Keystone_5019_Miniature" (layer "B.Cu")
     (at 97.028 75.438 180)
     (descr "SMT Test Point- Micro Miniature 5019, http://www.keyelco.com/product-pdf.cfm?p=1357")
