File: hardware/Prototype Boards/5v Power Supply/5v Power Supply.kicad_sch (KiCad schematic)
At the start: 12 parts

Commit message: [pre-commit.ci] auto fixes from pre-commit.com hooks
for more information, see https://pre-commit.ci
Parts:
- GNDREF: footprint TestPoint:TestPoint_Keystone_5019_Minature -> TestPoint:TestPoint_Keystone_5019_Miniature
Changed lines of the file:
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@@
       (effects (font (size 1.27 1.27)) (justify left))
     )
-    (property "Footprint" "TestPoint:TestPoint_Keystone_5019_Minature" (at 43.18 71.12 0)
+    (property "Footprint" "TestPoint:TestPoint_Keystone_5019_Miniature" (at 43.18 71.12 0)
       (effects (font (size 1.27 1.27)) hide)
     )
