File: hardware/giraffe_flight_computer/giraffe_flight_computer.kicad_sch (KiCad schematic)
At the start: 113 parts, among them J1 PI_HEADER_HAT, J2 BAT, J3 PI_HEADER_SHOE, J4 EEPROM, J5 USB, K1 ????, Q1 DMG2305UX, Q2 DMMT5401, Q3 NPN, Q4 BSS138, Q5 BSS138, Q6 DMN67D8LW-13, Q7 Q_NPN_BCE, SW1 Sliding Switch, U1 INA180A, U2 TPS61033, U3 CAT24C32, U4 SAM-M8Q, U5 BME280, U6 BMI088, U7 PCM2902C, Y1 Crystal ECS33B

Commit message: new PCB and Schematic
Parts:
- removed AE1: Antenna_Shield, Connector_Coaxial:SMA_Molex_73251-1153_EdgeMount_Horizontal, symbol Device:Antenna_Shield
- removed C2, C3: 0.1µF, Capacitor_SMD:C_0603_1608Metric, symbol Device:C_Small
- removed C20, C24: 20pF, Capacitor_SMD:C_0603_1608Metric_Pad1.08x0.95mm_HandSolder, symbol Device:C_Small
- removed C21: 1uF, Capacitor_SMD:C_0805_2012Metric_Pad1.18x1.45mm_HandSolder, symbol Device:C_Polarized_Small_US
- removed C22, C23: 36pF, Capacitor_SMD:C_0603_1608Metric_Pad1.08x0.95mm_HandSolder, symbol Device:C_Small
- removed C31: 1uF, Capacitor_SMD:C_0805_2012Metric_Pad1.18x1.45mm_HandSolder, symbol Device:C_Polarized_Small
- removed J5: USB, Connector_PinHeader_2.54mm:PinHeader_1x02_P2.54mm_Vertical_SMD_Pin1Left, symbol Connector_Generic:Conn_01x02
- removed K1: ????, Package_DIP:DIP-4_W8.89mm_SMDSocket_LongPads, symbol GFC-Symbols:TLP241A
- removed L2, L4: 56nH, Inductor_SMD:L_0603_1608Metric, symbol pspice:INDUCTOR
- removed L3: 68nH, Inductor_SMD:L_0603_1608Metric, symbol pspice:INDUCTOR
- removed Q4, Q5: BSS138, Package_TO_SOT_SMD:SOT-23, symbol Transistor_FET:BSS138
- removed Q6: DMN67D8LW-13, Package_TO_SOT_SMD:SOT-323_SC-70_Handsoldering, symbol Transistor_FET:2N7002K
- removed Q7: Q_NPN_BCE, Package_TO_SOT_SMD:SOT-23, symbol Device:Q_NPN_BCE
- removed R24: 0Ω, Resistor_SMD:R_0603_1608Metric, symbol Device:R_Small
- removed R25: 270Ω, Resistor_SMD:R_0603_1608Metric_Pad0.98x0.95mm_HandSolder, symbol Device:R_Small
- removed R26, R27, R28, R29, R32: 10k, Resistor_SMD:R_0603_1608Metric_Pad0.98x0.95mm_HandSolder, symbol Device:R_Small
- removed R31: 100K, Resistor_SMD:R_0603_1608Metric_Pad0.98x0.95mm_HandSolder, symbol Device:R_Small
- removed R33: 56K, Resistor_SMD:R_0603_1608Metric_Pad0.98x0.95mm_HandSolder, symbol Device:R_Small
- removed R34: 1K, Resistor_SMD:R_0603_1608Metric_Pad0.98x0.95mm_HandSolder, symbol Device:R_Small
- removed RV1: 100k, GFC-Footprints:TRIM_3361P-1-104GLF, symbol Device:R_Potentiometer
- added AE201: Antenna, giraffe_flight_computer_footprints:LINX_CONSMA001-G, symbol Device:Antenna_Shield
- added C10, C14, C15, C16, C17, C8, C9: 100pF, Capacitor_SMD:C_0603_1608Metric, symbol Device:C_Small
- added C19, C26, C27, C? (x6): 0.1µF, Capacitor_SMD:C_0603_1608Metric, symbol Device:C_Small
- added C218: 1μF, Resistor_SMD:R_0805_2012Metric, symbol Device:C_Polarized_Small
- added C221, C224: 20pF, Capacitor_SMD:C_0603_1608Metric, symbol Device:C_Small
- added C222, C223: 36pF, Capacitor_SMD:C_0603_1608Metric, symbol Device:C_Small
- added C? (x2): 10μF, Resistor_SMD:R_1210_3225Metric, symbol Device:C_Small
- added C?: 1μF, Resistor_SMD:R_0805_2012Metric, symbol Device:C_Small
- added D201: SHOE PWR LED, symbol Device:LED
- added J202: BAT, giraffe_flight_computer_footprints:OSTVN02A150 2x1 Terminal Block, symbol Connector:Screw_Terminal_01x02
- added J203: USB, symbol Connector_Generic:Conn_01x02
- added J204: Extra Audio, symbol Connector_Generic:Conn_01x02
- added J3: SHOE ADC, Connector_PinSocket_1.27mm:PinSocket_2x02_P1.27mm_Vertical, symbol Connector_Generic:Conn_02x02_Counter_Clockwise
- added L202, L204: 56nH, giraffe_flight_computer_footprints:IND_AIAC-1812-33NK-T, symbol Device:L
- added L203: 68nH, giraffe_flight_computer_footprints:IND_AIAC-1812-33NK-T, symbol Device:L
- added L?: 0.47uH, Inductor_SMD:L_Coilcraft_XAL4020-XXX, symbol Device:L
- added Q201: NPN, symbol Device:Q_NPN_BCE
- added Q202: Q_NPN_BCE, symbol Device:Q_NPN_BCE
- added R1, R2, R201, R202, R203, R205, R206, R207, R208, R209, R210, R211, R212, R215, R216: ?Ω, Resistor_SMD:R_0603_1608Metric, symbol Device:R_Small
- added R204: ?Ω, Potentiometer_SMD:Potentiometer_Bourns_TC33X_Vertical, symbol Device:R_Trim
- added R213, R217: ?kΩ, Resistor_SMD:R_0603_1608Metric, symbol Device:R_Small
- added R51, R53: 0Ω, Resistor_SMD:R_0603_1608Metric, symbol Device:R_Small
- added RV201, RV202: 100kΩ, Potentiometer_SMD:Potentiometer_Bourns_TC33X_Vertical, symbol Device:R_Potentiometer
- added SW201: ~, symbol Switch:SW_SPST
- added TP201, TP202: ~, TestPoint:TestPoint_Pad_D1.5mm, symbol Connector:TestPoint
- added U201: ?, Package_DIP:DIP-4_W8.89mm_SMDSocket_LongPads, symbol giraffe_symbols:Optical_Relay
- added U202: TPS61033, Package_TO_SOT_SMD:SOT-583-8, symbol giraffe_symbols:TPS61033
- added U203: INA180A1, Package_TO_SOT_SMD:SOT-23-5, symbol giraffe_symbols:INA180A
- added U204, U205: ISO6720B, Package_SO:SOIC-8_3.9x4.9mm_P1.27mm, symbol giraffe_symbols:ISO6721B
- added U3: MAX11615, Package_SO:QSOP-16_3.9x4.9mm_P0.635mm, symbol giraffe_symbols:MAX1161x
- added U4: DS18B20, Package_SO:MSOP-8_3x3mm_P0.65mm, symbol Sensor_Temperature:DS18B20Z
- added U5: AD1582B, Package_TO_SOT_SMD:SOT-23-3, symbol giraffe_symbols:AD1582
- 1W1: renamed from 1W2; footprint Connector_PinHeader_1.27mm:PinHeader_1x03_P1.27mm_Vertical -> giraffe_flight_computer_footprints:Molex-52745-0497; DESCRIPTION Breakaway Header -> (none); Digikey https://www.digikey.com/short/mwpz3z87 -> (none); Unit Price 0.18 -> (none)
- 1W2: renamed from 1W1; footprint Connector_PinHeader_1.27mm:PinHeader_1x03_P1.27mm_Vertical -> giraffe_flight_computer_footprints:Molex-52745-0497; DESCRIPTION Breakaway Header -> (none); Digikey https://www.digikey.com/short/mwpz3z87 -> (none); Unit Price 0.18 -> (none)
- C1: renamed from C12; footprint Capacitor_SMD:C_0603_1608Metric -> (none)
- C2: renamed from C11; value 10µF -> 10μF; footprint Capacitor_SMD:C_0603_1608Metric -> Resistor_SMD:R_1210_3225Metric
- C20: renamed from C15; DESCRIPTION CL10B104KB8NNWC -> (none); Digikey https://www.digikey.com/short/dz14934f -> (none); Unit Price 0.10 -> (none)
- C203: renamed from C17; value 0.1uF -> 0.1µF; footprint Capacitor_SMD:C_0603_1608Metric_Pad1.08x0.95mm_HandSolder -> Capacitor_SMD:C_0603_1608Metric; Digikey - -> (none); Unit Price 0.10 -> (none)
- C204: renamed from C18; footprint Capacitor_SMD:C_0603_1608Metric_Pad1.08x0.95mm_HandSolder -> Capacitor_SMD:C_0603_1608Metric; Digikey - -> (none); Unit Price 0.10 -> (none)
- C205: renamed from C19; footprint Capacitor_SMD:C_0603_1608Metric_Pad1.08x0.95mm_HandSolder -> Capacitor_SMD:C_0603_1608Metric; Digikey - -> (none); Unit Price 0.10 -> (none)
- C208: renamed from C33; value 1uF -> 1μF; footprint Capacitor_SMD:C_0805_2012Metric_Pad1.18x1.45mm_HandSolder -> Resistor_SMD:R_0805_2012Metric; Digikey https://www.digikey.com/short/rn5mbmcm -> (none)
- C209: renamed from C25; value 1uF -> 1μF; footprint Capacitor_SMD:C_0805_2012Metric_Pad1.18x1.45mm_HandSolder -> Resistor_SMD:R_0805_2012Metric; Digikey https://www.digikey.com/short/rn5mbmcm -> (none)
- C21: renamed from C16; DESCRIPTION CL10B104KB8NNWC -> (none); Digikey https://www.digikey.com/short/dz14934f -> (none); Unit Price 0.10 -> (none)
- C210: renamed from C34; value 1uF -> 1μF; footprint Capacitor_SMD:C_0805_2012Metric_Pad1.18x1.45mm_HandSolder -> Resistor_SMD:R_0805_2012Metric; Digikey https://www.digikey.com/short/rn5mbmcm -> (none)
- C211: renamed from C35; value 10pF -> ?pF; footprint Capacitor_SMD:C_0603_1608Metric_Pad1.08x0.95mm_HandSolder -> Capacitor_SMD:C_0603_1608Metric; Digikey https://www.digikey.com/short/dbpbjvrm -> (none)
- C212: renamed from C28; value 10uF -> 10μF; footprint Capacitor_SMD:C_1210_3225Metric_Pad1.33x2.70mm_HandSolder -> Resistor_SMD:R_1210_3225Metric; Digikey https://www.digikey.com/short/nm2875wp -> (none)
- C213: renamed from C26; value 1uF -> 1μF; footprint Capacitor_SMD:C_0805_2012Metric_Pad1.18x1.45mm_HandSolder -> Resistor_SMD:R_0805_2012Metric; Digikey https://www.digikey.com/short/rn5mbmcm -> (none)
- C214: renamed from C30; value 1uF -> 1μF; footprint Capacitor_SMD:C_0805_2012Metric_Pad1.18x1.45mm_HandSolder -> Resistor_SMD:R_0805_2012Metric; Digikey https://www.digikey.com/short/rn5mbmcm -> (none)
- C215: renamed from C36; value 10pF -> ?pF; footprint Capacitor_SMD:C_0603_1608Metric_Pad1.08x0.95mm_HandSolder -> Capacitor_SMD:C_0603_1608Metric; Digikey https://www.digikey.com/short/dbpbjvrm -> (none)
- C216: renamed from C27; value 1uF -> 1μF; footprint Capacitor_SMD:C_0805_2012Metric_Pad1.18x1.45mm_HandSolder -> Resistor_SMD:R_0805_2012Metric; Digikey https://www.digikey.com/short/rn5mbmcm -> (none)
- C217: renamed from C32; value 1uF -> 1μF; footprint Capacitor_SMD:C_0805_2012Metric_Pad1.18x1.45mm_HandSolder -> Resistor_SMD:R_0805_2012Metric; Digikey https://www.digikey.com/short/rn5mbmcm -> (none)
- C219: renamed from C29; value 10uF -> 10μF; footprint Capacitor_SMD:C_1210_3225Metric_Pad1.33x2.70mm_HandSolder -> Resistor_SMD:R_1210_3225Metric; Digikey https://www.digikey.com/short/nm2875wp -> (none)
- C22: renamed from C8; DESCRIPTION CL10B104KB8NNWC -> (none); Digikey https://www.digikey.com/short/dz14934f -> (none)
- C220: renamed from C37; value 1uF -> 1μF; footprint Capacitor_SMD:C_0805_2012Metric_Pad1.18x1.45mm_HandSolder -> Resistor_SMD:R_0805_2012Metric; Digikey https://www.digikey.com/short/rn5mbmcm -> (none)
- C23: renamed from C14; DESCRIPTION CL10B104KB8NNWC -> (none); Digikey https://www.digikey.com/short/dz14934f -> (none)
- C24: renamed from C5; DESCRIPTION CL10B104KB8NNWC -> (none); Digikey https://www.digikey.com/short/dz14934f -> (none); Unit Price 0.10 -> (none)
- C25: renamed from C6; DESCRIPTION CL10B104KB8NNWC -> (none); Digikey https://www.digikey.com/short/dz14934f -> (none); Unit Price 0.10 -> (none)
- C7: value 0.1µF -> 100pF; DESCRIPTION CL10B104KB8NNWC -> (none); Digikey https://www.digikey.com/short/dz14934f -> (none)
- C?: renamed from C1; value 10μf -> 10μF; footprint Capacitor_SMD:C_1210_3225Metric -> Resistor_SMD:R_1210_3225Metric
- C?: renamed from C2; value 10 μf -> 10μF; footprint Capacitor_SMD:C_1210_3225Metric -> Resistor_SMD:R_1210_3225Metric
- D2: renamed from D1; value PWR LED -> HAT PWR LED
- I2C1: footprint Connector_PinHeader_1.27mm:PinHeader_1x04_P1.27mm_Vertical -> giraffe_flight_computer_footprints:Molex-52745-0497; DESCRIPTION Breakaway Header -> (none); Digikey https://www.digikey.com/short/mwpz3z87 -> (none)
- J2: footprint GFC-Footprints:OSTVN02A150 2x1 Terminal Block -> (none)
- J4: value EEPROM -> EEPROM PROG
- Q1: footprint (none) -> Package_TO_SOT_SMD:SOT-23-3
- Q2: footprint (none) -> Package_TO_SOT_SMD:SOT-23-6
- Q3: symbol Simulation_SPICE:NPN -> Device:Q_NPN_BCE
- R10: renamed from R13; footprint (none) -> Resistor_SMD:R_0603_1608Metric
- R11: value ?KΩ -> ?Ω; footprint (none) -> Resistor_SMD:R_0603_1608Metric
- R12: renamed from R14; value 1KΩ -> 1kΩ; footprint (none) -> Potentiometer_SMD:Potentiometer_Bourns_TC33X_Vertical
- R13: renamed from R21; footprint (none) -> Resistor_SMD:R_0603_1608Metric
- R14: renamed from R16; value ?KΩ -> ?Ω; footprint (none) -> Resistor_SMD:R_0603_1608Metric
- R15: renamed from R12; value ?KΩ -> ?Ω; footprint (none) -> Resistor_SMD:R_0603_1608Metric
- R16: renamed from R15; value 3KΩ -> 3kΩ; footprint (none) -> Resistor_SMD:R_0603_1608Metric
- R17: renamed from R18; value ?KΩ -> ?Ω; footprint (none) -> Resistor_SMD:R_0603_1608Metric
- R18: renamed from R17; value ?KΩ -> ?Ω; footprint (none) -> Resistor_SMD:R_0603_1608Metric
- R19: renamed from R3; value ?KΩ -> ?Ω; footprint (none) -> Resistor_SMD:R_0603_1608Metric
- R20: renamed from R4; value ?KΩ -> ?Ω; footprint (none) -> Resistor_SMD:R_0603_1608Metric
- R21: renamed from R19; value ?KΩ -> ?Ω; footprint (none) -> Resistor_SMD:R_0603_1608Metric
- R214: renamed from R30; value 10K -> 10kΩ; footprint Resistor_SMD:R_0603_1608Metric_Pad0.98x0.95mm_HandSolder -> Resistor_SMD:R_0603_1608Metric; Digikey - -> (none); Unit Price 0.10 -> (none)
- R218: renamed from R36; value 1.5k -> 1.5kΩ; footprint Capacitor_SMD:C_0603_1608Metric_Pad1.08x0.95mm_HandSolder -> Resistor_SMD:R_0603_1608Metric; Digikey https://www.digikey.com/short/q2j089rj -> (none)
- R219: renamed from R37; value 22 -> 22Ω; footprint Capacitor_SMD:C_0603_1608Metric_Pad1.08x0.95mm_HandSolder -> Resistor_SMD:R_0603_1608Metric; Digikey https://www.digikey.com/short/v7c8qpnf -> (none)
- R220: renamed from R38; value 22 -> 22Ω; footprint Capacitor_SMD:C_0603_1608Metric_Pad1.08x0.95mm_HandSolder -> Resistor_SMD:R_0603_1608Metric; Digikey https://www.digikey.com/short/v7c8qpnf -> (none)
- R221: renamed from R35; value 2.2 -> 2.2Ω; footprint Capacitor_SMD:C_0603_1608Metric_Pad1.08x0.95mm_HandSolder -> Resistor_SMD:R_0603_1608Metric; Digikey https://www.digikey.com/short/4p2jz24h -> (none)
- R222: renamed from R39; value 1M -> 1MΩ; footprint Capacitor_SMD:C_0603_1608Metric_Pad1.08x0.95mm_HandSolder -> Resistor_SMD:R_0603_1608Metric; Digikey https://www.digikey.com/short/f7pn93f7 -> (none)
- R23: renamed from R22; value ?kΩ -> ?Ω
- R26: renamed from R23; value ?kΩ -> ?Ω
- R3: renamed from R2; footprint (none) -> Resistor_SMD:R_0603_1608Metric
- R4: renamed from R5; footprint (none) -> Resistor_SMD:R_0603_1608Metric
- R5: renamed from R20; footprint (none) -> Resistor_SMD:R_0603_1608Metric
- R9: renamed from R1; footprint (none) -> Resistor_SMD:R_0603_1608Metric
- SW1: value Sliding Switch -> ~
- TP1: renamed from TP3; footprint (none) -> TestPoint:TestPoint_Pad_D1.5mm
- TP2: renamed from TP1; footprint TestPoint:TestPoint_Keystone_5019_Minature -> (none)
- TP3: renamed from TP2; footprint (none) -> TestPoint:TestPoint_Pad_D1.5mm
- TX201: renamed from TX1; footprint GFC-Footprints:DORJI_DRA818V -> giraffe_flight_computer_footprints:DORJI_DRA818V; symbol GFC-Symbols:SA868 -> giraffe_symbols:SA868; Digikey eBay -> (none); MANUFACTURER NiceRF -> (none); PART_REV 1.23 -> (none); STANDARD MANUFACTURER RECOMMENDATIONS -> (none); Unit Price 12.28 -> (none)
- U2: renamed from U1; value INA180A -> INA180A1; footprint (none) -> Package_TO_SOT_SMD:SOT-23-5
- U206: renamed from U7; symbol Audio:PCM2902 -> giraffe_symbols:PCM2902; Digikey TI -> (none)
- U6: footprint PQFN50P450X300X100-16N -> giraffe_flight_computer_footprints:BMI088; symbol GFC-Symbols:BMI088 -> giraffe_symbols:BMI088; AVAILABILITY In Stock -> (none); Digikey https://www.digikey.com/short/pfd3pm9q -> (none); MF Bosch Sensortec -> (none); MP BMI088 -> (none); PACKAGE VFLGA-16 Bosch Sensortec -> (none); PRICE None -> (none); PURCHASE-URL https://pricing.snapeda.com/search/part/BMI088/?ref=eda -> (none)
- U7: renamed from U5; footprint footprints:PSON65P250X250X100-8N -> giraffe_flight_computer_footprints:BME280; symbol GFC-Symbols:BME280 -> giraffe_symbols:BME280; AVAILABILITY Good -> (none); Digikey https://www.digikey.com/short/pjf7tjwh -> (none); MF Bosch -> (none); MP BME280 -> (none); PACKAGE LGA-8 Bosch -> (none); PRICE 4.94 USD -> (none); STANDARD IPC-7351B -> (none)
- U8: renamed from U4; symbol RF_GPS:SAM-M8Q -> giraffe_symbols:SAM-M8Q
- U9: renamed from U3; footprint SOIC127P600X175-8N -> giraffe_flight_computer_footprints:CAT24C32WI_GT3; symbol GFC-Symbols:CAT24C32WI-GT3 -> giraffe_symbols:CAT24C32WI-GT3
- Y201: renamed from Y1; value Crystal ECS33B -> 12MHz; footprint Crystal:Crystal_SMD_3225-4Pin_3.2x2.5mm -> Crystal:Crystal_SMD_0603-2Pin_6.0x3.5mm; symbol GFC-Symbols:Crystal_GND23 -> Device:Crystal_GND23
- renumbered C4 to C28, C1 to C29, C9 to C3, J3 to J201, L1 to L?, R7 to R24, R6 to R25, R9 to R6, R8 to R7, R10 to R8, U2 to U1
Connections:
- net +3V3 is gone; now on net H_3V3: 1W1.3 (Pin_3), 1W2.3 (Pin_3), I2C1.2 (Pin_2), U6.11 (VDDIO), U6.3 (VDD)
- net PD is gone; now on an unnamed net: TX201.6 (PD)
- net SAM_M8Q.RST is gone; now on net SAM-M8Q.RST: J1.33 (PWM1/GPIO13)
- net 1-Wire: now also R8.2, U4.4 (DQ)
- net ADC CH1: now also R17.2, R21.1, C9.2, U3.6 (AIN1); no longer R14.2, R18.1
- net ADC CH2: now also C8.2, U3.7 (AIN2)
- net ADC CH3: now also C7.2, R1.2, R2.1, U3.8 (AIN3); no longer R17.2, R21.1
- net BMI088.INT1: now also J1.29 (GCLK1/GPIO5)
- net BMI088.INT3: now also J1.31 (GCLK2/GPIO6)
- net EEPROM.SCL: now also R25.1
- net EEPROM.SDA: now also R24.1
- net H_3V3: now also C20.2, C21.2, C22.2, C23.2, C24.2, C25.2, R23.2, R24.2, R25.2, R6.2, R7.1, R8.1, U7.2 (CSB), C19.2, C26.1, C27.1, C?.1, C?.1, R1.1, R51.1, U3.16 (Vdd), U4.3 (V_{DD})
- net H_5V_HAT: now also C?.1, C?.1, U203.5 (VS), U5.3 (V_In)
- net H_GND: now also 1W1.1 (Pin_1), 1W2.1 (Pin_1), C20.1, C21.1, C22.1, C23.1, C24.1, C25.1, C7.1, I2C1.1 (Pin_1), C10.1, C14.1, C15.1, C16.1, C17.1, C19.1, C26.2, C27.2, C8.1, C9.1, C?.2, C?.2, C?.2, C?.2, C?.2, R2.2, R53.2, U3.15 (GND), U4.5 (GND), U5.2 (GND); no longer J201.14 (GND), J201.20 (GND), J201.25 (GND), J201.30 (GND), J201.34 (GND), J201.39 (GND), J201.6 (GND), J201.9 (GND), U7.5 (SDO)
- net I2C0.SCL: now also R7.2, U3.13 (SCL); no longer J201.5 (SCL/GPIO3)
- net I2C0.SDA: now also R6.1, U3.14 (SDA); no longer J201.3 (SDA/GPIO2)
- net PCM.CLK: no longer J201.12 (GPIO18/PWM0)
- net PCM.DIN: no longer J201.38 (GPIO20/MOSI1)
- net PCM.DOUT: no longer J201.40 (GPIO21/SCLK1)
- net PCM.FS: no longer J201.35 (GPIO19/MISO1)
- net RF_OUT_FILTERED: now also AE201.1 (A), C224.1, L204.2
- net SA868.PTT: now also U204.3 (INB)
- net SA868.PWR: now also R203.1
- net SA868.RX: now also U204.2 (OUTA)
- net SA868_RF_OUT: now also C221.1, L202.1
- net S_3V3: now also C?.1, U204.1 (VCC1), U205.1 (VCC1)
- net S_5V: now also R221.1
- net S_GND: now also C203.1, C204.1, C205.1, C208.2, C209.2, C210.2, C211.2, C212.2, C214.2, C215.2, C219.2, C220.2, J201.14 (GND), J201.20 (GND), J201.25 (GND), J201.30 (GND), J201.34 (GND), J201.39 (GND), J201.6 (GND), J201.9 (GND), TX201.10 (GND), TX201.9 (GND), U206.11 (AGNDC), U206.18 (AGNDP), U206.22 (AGNDX), U206.26 (DGND), U206.4 (DGNDU), Y201.2, Y201.3, AE201.2 (Shield), C221.2, C222.2, C223.2, C224.2, C?.2, C?.2, C?.2, C?.2, D201.1 (K), J202.2 (Pin_2), Q201.3 (E), Q202.3 (E), R206.2, R209.2, R210.2, R213.1, R217.1, RV201.1, RV202.1, SW201.1 (A), U201.2, U202.3 (MODE), U202.6 (GND), U203.2 (GND), U204.4 (GND1), U204.5 (GND2), U205.4 (GND1), U205.5 (GND2)
- net UART.RXD: now also U205.2 (OUTA)
- net UART.TXD: now also U205.3 (INB)
- net at R219.1: now also R218.2, J203.2 (Pin_2)
- net at R219.2: now also U206.1 (D+)
- net at R26.1: now also Q3.1 (B)
- net SAM-M8Q.RST: now reaches R26.2
- net at U8.18 (~{RESET}): now also Q3.2 (C), R23.1; no longer Q3.1 (C)
- net Battery Polarized: now reaches C?.1, L?.1, Q1.3 (S), Q2.5 (E2), R14.1, U1.1 (VIN), U1.2 (EN)
- net S_4V: now reaches C204.2
- net S_4V: now also C203.2, C205.2, R214.1, TX201.8 (VBAT), C?.1, R201.2, R205.1, R208.1, R211.1, R215.2, U203.4 (IN-), U204.8 (VCC2), U205.8 (VCC2)
- net at TX201.7 (H/L): now also SW201.2 (B)
- net at R222.1: now also C215.1, U206.20 (XTO), Y201.1
- net at R222.2: now also C211.1, U206.21 (XTI), Y201.4
- net VBUS: now reaches C209.1, U206.3 (VBUS)
- net VBUS: now also R221.2
- net at U206.16 (VOUTL): now also C218.1
- net at C208.1, U206.27 (VDDI), U206.8 (SEL0)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: now also R218.1
- net at R220.1: now also J203.1 (Pin_1)
- net at R220.2: now also U206.2 (D-)
- net A_IN Filtered renamed SA868_AUDIO_IN
- net SA868_AUDIO_IN: now also RV202.3
- net Audio In Left renamed PCM_AUDIO.IN_L
- net PCM_AUDIO.IN_L: now also RV201.3
- net Audio In Right renamed PCM_AUDIO.IN_R
- net PCM_AUDIO.IN_R: now also J204.1 (Pin_1)
- net Audio Out Right renamed PCM_AUDIO.OUT_R
- net PCM_AUDIO.OUT_R: now also J204.2 (Pin_2)
- removed net BMI088.INT: J1.29 (GCLK1/GPIO5), J1.31 (GCLK2/GPIO6)
- removed net GND: 1W1.1 (Pin_1), 1W2.1 (Pin_1), C208.2, C209.2, C210.2, C211.2, C212.2, C214.2, C215.2, C219.2, C220.2, I2C1.1 (Pin_1), TX201.10 (GND), TX201.9 (GND), U206.11 (AGNDC), U206.18 (AGNDP), U206.22 (AGNDX), U206.26 (DGND), U206.4 (DGNDU), Y201.2, Y201.4
- net PTT: no longer names the net of TX201.5 (PTT)
- net PTT: now also Q202.2 (C), R215.1
- net RXD 5V: no longer names the net of TX201.16 (RXD)
- net RXD 5V: now also U205.6 (OUTB)
- net Radio Audio Output renamed SA868_AUDIO_OUT
- net SA868_AUDIO_OUT: now also RV201.2
- net SAM_M8Q.TX_RDY renamed SAM-M8Q.TX_RDY
- net SQ: no longer names the net of TX201.1 (SQ)
- net SQ: now also R212.2
- net TXD 5V: no longer names the net of TX201.17 (TXD)
- net TXD 5V: now also U205.7 (INA)
- new net: C223.1, L203.2, L204.1
- new net: R204.2, R206.1, U202.5 (FB)
- new net: C222.1, L202.2, L203.1
- new net: Q201.1 (B), R212.1, R213.2
- new net: Q201.2 (C), R211.2, U204.7 (INA)
- new net: L?.2, TP201.1, U202.7 (SW)
- new net: TP202.1, U202.4 (PG)
- new net: R203.2, U201.1
- new net: C?.1, L?.1, U201.3 (5), U202.1 (VIN), U202.2 (EN)
- new net: J202.1 (Pin_1), U201.4
- new net: R202.2, R204.1
- new net: R207.1, U203.1 (OUT)
- new net: C?.1, R201.1, R202.1, U202.8 (VOUT), U203.3 (IN+)
- new net: Q202.1 (B), R216.1, R217.2
- new net: R216.2, U204.6 (OUTB)
- new net: C14.2, J3.1 (Pin_1), U3.9 (AIN4)
- new net: C15.2, J3.2 (Pin_2), U3.10 (AIN5)
- new net: C16.2, J3.3 (Pin_3), U3.11 (AIN6)
- new net: C17.2, J3.4 (Pin_4), U3.12 (AIN7)
- new net: R51.2, R53.1, U7.5 (SDO)
- new net: D201.2 (A), R205.2
- new net 2.5V Reference Voltage: C?.1, U3.1 (REF), U5.1 (V_Out)
- new net ADC CH0: C10.2, R14.2, R18.1, U3.5 (AIN0)
- new net ADC CH4: R207.2, R209.1
- new net ADC CH5: R208.2, R210.1
- new net PCM_AUDIO.OUT_L: C218.2, RV202.2
- no-connect marks 38 -> 43
Other:
- note added: "1-Wire Expansion Bus"
- note added: "2.5V Voltage Reference Circuit"
- note added: "DS18B20 Temperature Sensor (On Board)"
- note added: "I2C Expansion Bus"
- note added: "MAX11615 12-Bit 8-Channel I2C ADC"
- note added: "PCM2902C USB PCM Audio Interface"
- note added: "PCM2902C/SA868 Audio Connection"
- note added: "SA868 VHF Radio Module"
- note added: "SAM-M8Q GPS Module"
- note removed: "I2C Expansion"
- moved on the sheet: 1W1, 1W2, C203, C204, C205, C208, C209, C210, C211, C212, C213, C214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

Commit message: schematic rev A initial design
Parts:
- removed AE201: Antenna, giraffe_flight_computer_footprints:LINX_CONSMA001-G, symbol Device:Antenna_Shield
- removed C? (x2): 0.1µF, Capacitor_SMD:C_0603_1608Metric, symbol Device:C_Small
- removed C?: 1μF, Resistor_SMD:R_0805_2012Metric, symbol Device:C_Small
- removed J202: BAT, giraffe_flight_computer_footprints:OSTVN02A150 2x1 Terminal Block, symbol Connector:Screw_Terminal_01x02
- removed R203: ?Ω, Resistor_SMD:R_0603_1608Metric, symbol Device:R_Small
- removed SW1: ~, symbol Switch:SW_SPST
- removed TP2: GND REF, symbol Connector:TestPoint_Alt
- removed U201: ?, Package_DIP:DIP-4_W8.89mm_SMDSocket_LongPads, symbol giraffe_symbols:Optical_Relay
- removed U5: AD1582B, Package_TO_SOT_SMD:SOT-23-3, symbol giraffe_symbols:AD1582
- added AE1: SMA, giraffe_flight_computer_footprints:MolexSmaConnector, symbol giraffe_symbols:Molex SMA 0732511150
- added C?: 1μF, Resistor_SMD:R_0805_2012Metric, symbol Device:C_Small
- added C? (x2): 0.1µF, Capacitor_SMD:C_0603_1608Metric, symbol Device:C_Small
- added J10: HAT ADC CONNECT, Connector_PinSocket_1.27mm:PinSocket_2x02_P1.27mm_Vertical, symbol Connector_Generic:Conn_02x02_Counter_Clockwise
- added J12, J2: BAT-, Connector_Wire:SolderWirePad_1x01_SMD_1x2mm, symbol Connector_Generic:Conn_01x01
- added J3: PCM Interface, Connector_PinHeader_1.00mm:PinHeader_1x04_P1.00mm_Vertical, symbol Connector_Generic:Conn_01x04
- added J6: BAT+, Connector_Wire:SolderWirePad_1x01_SMD_1x2mm, symbol Connector_Generic:Conn_01x01
- added R28: ?Ω, Resistor_SMD:R_0603_1608Metric, symbol Device:R_Small
- added TP1, TP10, TP11, TP12, TP13, TP16, TP17, TP18, TP19, TP2, TP20, TP21, TP22, TP5, TP6, TP7, TP8, TP9: ~, TestPoint:TestPoint_Keystone_5000-5004_Miniature, symbol Connector:TestPoint
- added U9: AD1582B, Package_TO_SOT_SMD:SOT-23-3, symbol giraffe_symbols:AD1582
- C10: renamed from C1; footprint (none) -> Capacitor_Tantalum_SMD:CP_EIA-7343-31_Kemet-D
- D1: footprint (none) -> giraffe_flight_computer_footprints:B36S3RGB LED
- D2: footprint (none) -> LED_SMD:LED_0603_1608Metric
- D3: renamed from D201; footprint (none) -> LED_SMD:LED_0603_1608Metric
- J1: renamed from J2; value BAT -> BAT+; footprint (none) -> Connector_Wire:SolderWirePad_1x01_SMD_1x2mm; symbol Connector:Screw_Terminal_01x02 -> Connector_Generic:Conn_01x01
- J4: footprint (none) -> Connector_PinHeader_1.00mm:PinHeader_1x04_P1.00mm_Vertical
- J5: renamed from J1; footprint Connector_PinSocket_2.54mm:PinSocket_2x20_P2.54mm_Vertical -> giraffe_flight_computer_footprints:pi_zero
- J7: renamed from J201; footprint Connector_PinSocket_2.54mm:PinSocket_2x20_P2.54mm_Vertical -> giraffe_flight_computer_footprints:pi_zero
- J8: renamed from J204; footprint (none) -> Connector_PinHeader_1.00mm:PinHeader_1x02_P1.00mm_Vertical
- J9: renamed from J203; footprint (none) -> Connector_PinHeader_1.00mm:PinHeader_1x03_P1.00mm_Vertical; symbol Connector_Generic:Conn_01x02 -> Connector_Generic:Conn_01x03
- Q3: footprint (none) -> Package_TO_SOT_SMD:SOT-23
- Q4: renamed from Q202; value Q_NPN_BCE -> NPN; footprint (none) -> Package_TO_SOT_SMD:SOT-23
- Q5: renamed from Q201; footprint (none) -> Package_TO_SOT_SMD:SOT-23
- TP14: renamed from TP202; footprint TestPoint:TestPoint_Pad_D1.5mm -> TestPoint:TestPoint_Keystone_5000-5004_Miniature
- TP15: renamed from TP201; footprint TestPoint:TestPoint_Pad_D1.5mm -> TestPoint:TestPoint_Keystone_5000-5004_Miniature
- TP3: footprint TestPoint:TestPoint_Pad_D1.5mm -> TestPoint:TestPoint_Keystone_5000-5004_Miniature
- TP4: renamed from TP1; footprint TestPoint:TestPoint_Pad_D1.5mm -> TestPoint:TestPoint_Keystone_5000-5004_Miniature
- Y1: renamed from Y201; symbol Device:Crystal_GND23 -> Device:Crystal
- renumbered 1W2 to 1W1, 1W1 to 1W2, C24 to C1, C8 to C11, C15 to C12, C9 to C13, C16 to C14, C10 to C15, C17 to C16, C2 to C17, C3 to C18, C29 to C2, C26 to C21, C27 to C22, C22 to C23, C28 to C25, C19 to C26, C23 to C27, C25 to C3, C221 to C30, C222 to C31, C223 to C32, C224 to C33, C203 to C36, C204 to C37, C209 to C38, C205 to C41, C213 to C42, C216 to C43, C212 to C44, C219 to C45, C217 to C46, C214 to C47, C208 to C48, C218 to C49, C20 to C5, C210 to C50, C211 to C51, C215 to C52, C220 to C53, C21 to C7, C7 to C8, C14 to C9, J3 to J11, L202 to L2, L203 to L3, L204 to L4, R51 to R1, R24 to R10, R25 to R11, R10 to R12, R12 to R13, R16 to R14, R23 to R15, R26 to R16, R1 to R17, R2 to R18, R6 to R19, R53 to R2, R7 to R20, R9 to R21, R17 to R22, R21 to R23, R11 to R24, R15 to R25, R8 to R26, R13 to R27, R221 to R29, R19 to R3, R202 to R30, R204 to R31, R206 to R32, R218 to R33, R219 to R34, R220 to R35, R214 to R36, R201 to R37, R207 to R38, R209 to R39, R20 to R4, R222 to R40, R208 to R41, R210 to R42, R212 to R43, R217 to R44, R215 to R45, R211 to R46, R213 to R47, R216 to R48, R205 to R49, R3 to R5, R4 to R6, R5 to R7, R14 to R8, R18 to R9, RV201 to RV1, RV202 to RV2, SW201 to SW2, TX201 to TX1, U4 to U1, U202 to U11, U205 to U12, U206 to U13, U203 to U14, U204 to U15, U9 to U2, U6 to U3, U7 to U4, U1 to U5, U3 to U6, U2 to U7
Connections:
- net ADC CH4: now also J10.1 (Pin_1)
- net ADC CH5: now also J10.2 (Pin_2)
- net Battery Polarized: now also TP2.1
- net H_5V_HAT: now also C?.1, C?.1, TP8.1, U9.3 (V_In); no longer U14.5 (VS)
- net H_GND: now also C?.2, C?.2, C?.2, J2.1 (Pin_1), U9.2 (GND); no longer J1.2 (Pin_2)
- net PCM.CLK: now also J3.4 (Pin_4)
- net PCM.DIN: now also J3.2 (Pin_2)
- net PCM.DOUT: now also J3.1 (Pin_1)
- net PCM.FS: now also J3.3 (Pin_3)
- net RF_OUT_FILTERED: now also AE1.1, TP12.1
- net SA868.PWR: now also U11.2 (EN), R28.1
- net SA868_AUDIO_IN: now also TP11.1
- net SA868_AUDIO_OUT: now also TP10.1
- net SA868_RF_OUT: now also TP9.1
- net SAM-M8Q.TX_RDY: now also TP7.1
- net S_4V: now also TP17.1, TP20.1
- net S_5V: now also U14.5 (VS)
- net S_GND: now also J9.3 (Pin_3), AE1.2 (MNT_1), AE1.3 (MNT_2), AE1.4 (MNT_3), AE1.5 (MNT_4), J12.1 (Pin_1), R28.2; no longer Y1.2, Y1.3
- net at R33.2, R34.1: now also J9.1 (Pin_1); no longer J9.2 (Pin_2)
- net at Q3.2 (C), R15.1, U8.18 (~{RESET}): now also TP6.1
- net at C?.1, R12.1, R21.1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: now also TP5.1
- net at J1.1 (Pin_1): now also Q1.1 (D), Q2.6 (E1), TP1.1
- net at Q5.2 (C), R46.2, U15.7 (INA): now also TP21.1
- net at R43.2, TX1.1 (SQ): now also TP19.1
- net at Q4.2 (C), R45.1, TX1.5 (PTT): now also TP18.1
- net at R35.1: now also J9.2 (Pin_2); no longer J9.1 (Pin_1)
- net at C51.1, R40.2, U13.21 (XTI): now also Y1.2; no longer Y1.4
- net at C?.1, L?.1, U11.1 (VIN): now also J6.1 (Pin_1), TP13.1; no longer U11.2 (EN)
- net at C?.1, R30.1, R37.1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: now also TP16.1
- net at R48.2, U15.6 (OUTB): now also TP22.1
- net 2.5V Reference Voltage: no longer names the net of U6.1 (REF)
- net 2.5V Reference Voltage: now also C?.1, U9.1 (V_Out)
- net LED.B renamed Status LED Blue
- net LED.G renamed Status LED Green
- net LED.R renamed Status LED Red
- no-connect marks 43 -> 45
Other:
- note added: "MAX11615 12-Bit 8-Channel I2C ADC With External 2.5V Reference Voltage"
- note added: "Optional"
- note removed: "2.5V Voltage Reference Circuit"
- note removed: "MAX11615 12-Bit 8-Channel I2C ADC"
- company: (none) -> Joshua Jerred
- title: (none) -> Giraffe Flight Computer
- moved on the sheet: C10, C11, C12, C13, C14, C15, C16, C17, C18, C50, C8, C9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

Commit message: More schematic changes
Parts:
- removed 1W1, 1W2: 1-Wire, giraffe_flight_computer_footprints:Molex-52745-0497, symbol Connector_Generic:Conn_01x03
- removed AE1: SMA, giraffe_flight_computer_footprints:MolexSmaConnector, symbol giraffe_symbols:Molex SMA 0732511150
- removed C1, C18, C2, C21, C22, C23, C25, C26, C27, C3, C36, C5, C7, C? (x6): 0.1µF, Capacitor_SMD:C_0603_1608Metric, symbol Device:C_Small
- removed C10: 100µF, Capacitor_Tantalum_SMD:CP_EIA-7343-31_Kemet-D, symbol Device:C_Small
- removed C11, C12, C13, C14, C15, C16, C8, C9: 100pF, Capacitor_SMD:C_0603_1608Metric, symbol Device:C_Small
- removed C17, C? (x4): 10μF, Resistor_SMD:R_1210_3225Metric, symbol Device:C_Small
- removed C30, C33: 20pF, Capacitor_SMD:C_0603_1608Metric, symbol Device:C_Small
- removed C31, C32: 36pF, Capacitor_SMD:C_0603_1608Metric, symbol Device:C_Small
- removed C37: 10kpF, Capacitor_SMD:C_0603_1608Metric, symbol Device:C_Small
- removed C38, C47, C48, C50, C53, C?: 1μF, Resistor_SMD:R_0805_2012Metric, symbol Device:C_Small
- removed C41: 1kpF, Capacitor_SMD:C_0603_1608Metric, symbol Device:C_Small
- removed C42, C43, C46, C49: 1μF, Resistor_SMD:R_0805_2012Metric, symbol Device:C_Polarized_Small
- removed C44, C45: 10μF, Resistor_SMD:R_1210_3225Metric, symbol Device:C_Polarized_Small
- removed C51, C52: ?pF, Capacitor_SMD:C_0603_1608Metric, symbol Device:C_Small
- removed D1: STATUS, giraffe_flight_computer_footprints:B36S3RGB LED, symbol Device:LED_ARGB
- removed D2: HAT PWR LED, LED_SMD:LED_0603_1608Metric, symbol Device:LED
- removed D3: SHOE PWR LED, LED_SMD:LED_0603_1608Metric, symbol Device:LED
- removed I2C1: I²C, giraffe_flight_computer_footprints:Molex-52745-0497, symbol Connector_Generic:Conn_01x04
- removed J1, J6: BAT+, Connector_Wire:SolderWirePad_1x01_SMD_1x2mm, symbol Connector_Generic:Conn_01x01
- removed J10: HAT ADC CONNECT, Connector_PinSocket_1.27mm:PinSocket_2x02_P1.27mm_Vertical, symbol Connector_Generic:Conn_02x02_Counter_Clockwise
- removed J11: SHOE ADC, Connector_PinSocket_1.27mm:PinSocket_2x02_P1.27mm_Vertical, symbol Connector_Generic:Conn_02x02_Counter_Clockwise
- removed J12, J2: BAT-, Connector_Wire:SolderWirePad_1x01_SMD_1x2mm, symbol Connector_Generic:Conn_01x01
- removed J3: PCM Interface, Connector_PinHeader_1.00mm:PinHeader_1x04_P1.00mm_Vertical, symbol Connector_Generic:Conn_01x04
- removed J4: EEPROM PROG, Connector_PinHeader_1.00mm:PinHeader_1x04_P1.00mm_Vertical, symbol Connector_Generic:Conn_01x04
- removed J5: PI_HEADER_HAT, giraffe_flight_computer_footprints:pi_zero, symbol giraffe_symbols:Raspberry_Pi_2_3
- removed J7: PI_HEADER_SHOE, giraffe_flight_computer_footprints:pi_zero, symbol giraffe_symbols:Raspberry_Pi_2_3
- removed J8: Extra Audio, Connector_PinHeader_1.00mm:PinHeader_1x02_P1.00mm_Vertical, symbol Connector_Generic:Conn_01x02
- removed J9: USB, Connector_PinHeader_1.00mm:PinHeader_1x03_P1.00mm_Vertical, symbol Connector_Generic:Conn_01x03
- removed L2, L4: 56nH, giraffe_flight_computer_footprints:IND_AIAC-1812-33NK-T, symbol Device:L
- removed L3: 68nH, giraffe_flight_computer_footprints:IND_AIAC-1812-33NK-T, symbol Device:L
- removed L? (x2): 0.47uH, Inductor_SMD:L_Coilcraft_XAL4020-XXX, symbol Device:L
- removed Q1: DMG2305UX, Package_TO_SOT_SMD:SOT-23-3, symbol Simulation_SPICE:PMOS
- removed Q2: DMMT5401, Package_TO_SOT_SMD:SOT-23-6, symbol giraffe_symbols:DMMT5401
- removed Q3, Q4, Q5: NPN, Package_TO_SOT_SMD:SOT-23, symbol Device:Q_NPN_BCE
- removed R1, R2: 0Ω, Resistor_SMD:R_0603_1608Metric, symbol Device:R_Small
- removed R10, R11: 3.9kΩ, Resistor_SMD:R_0603_1608Metric, symbol Device:R_Small
- removed R12: 21.5KΩ, Resistor_SMD:R_0603_1608Metric, symbol Device:R_Small
- removed R13: 1kΩ, Potentiometer_SMD:Potentiometer_Bourns_TC33X_Vertical, symbol Device:R_Trim
- removed R14: 3kΩ, Resistor_SMD:R_0603_1608Metric, symbol Device:R_Small
- removed R15, R16, R17, R18, R21, R22, R23, R24, R25, R27, R28, R3, R30, R32, R37, R38, R39, R4, R41, R42, R43, R45, R46, R48, R49, R5, R6, R7, R8, R9: ?Ω, Resistor_SMD:R_0603_1608Metric, symbol Device:R_Small
- removed R19, R20: *, Resistor_SMD:R_0603_1608Metric, symbol Device:R_Small
- removed R26: 4.7kΩ, Resistor_SMD:R_0603_1608Metric, symbol Device:R_Small
- removed R29: 2.2Ω, Resistor_SMD:R_0603_1608Metric, symbol Device:R_Small
- removed R31: ?Ω, Potentiometer_SMD:Potentiometer_Bourns_TC33X_Vertical, symbol Device:R_Trim
- removed R33: 1.5kΩ, Resistor_SMD:R_0603_1608Metric, symbol Device:R_Small
- removed R34, R35: 22Ω, Resistor_SMD:R_0603_1608Metric, symbol Device:R_Small
- removed R36: 10kΩ, Resistor_SMD:R_0603_1608Metric, symbol Device:R_Small
- removed R40: 1MΩ, Resistor_SMD:R_0603_1608Metric, symbol Device:R_Small
- removed R44, R47: ?kΩ, Resistor_SMD:R_0603_1608Metric, symbol Device:R_Small
- removed RV1, RV2: 100kΩ, Potentiometer_SMD:Potentiometer_Bourns_TC33X_Vertical, symbol Device:R_Potentiometer
- removed SW2: ~, symbol Switch:SW_SPST
- removed TP1, TP10, TP11, TP12, TP13, TP14, TP15, TP16, TP17, TP18, TP19, TP2, TP20, TP21, TP22, TP3, TP4, TP5, TP6, TP7, TP8, TP9: ~, TestPoint:TestPoint_Keystone_5000-5004_Miniature, symbol Connector:TestPoint
- removed TX1: SA868, giraffe_flight_computer_footprints:DORJI_DRA818V, symbol giraffe_symbols:SA868
- removed U1: DS18B20, Package_SO:MSOP-8_3x3mm_P0.65mm, symbol Sensor_Temperature:DS18B20Z
- removed U11, U5: TPS61033, Package_TO_SOT_SMD:SOT-583-8, symbol giraffe_symbols:TPS61033
- removed U12, U15: ISO6720B, Package_SO:SOIC-8_3.9x4.9mm_P1.27mm, symbol giraffe_symbols:ISO6721B
- removed U13: PCM2902C, Package_SO:SSOP-28_5.3x10.2mm_P0.65mm, symbol giraffe_symbols:PCM2902
- removed U14, U7: INA180A1, Package_TO_SOT_SMD:SOT-23-5, symbol giraffe_symbols:INA180A
- removed U2: CAT24C32, giraffe_flight_computer_footprints:CAT24C32WI_GT3, symbol giraffe_symbols:CAT24C32WI-GT3
- removed U3: BMI088, giraffe_flight_computer_footprints:BMI088, symbol giraffe_symbols:BMI088
- removed U4: BME280, giraffe_flight_computer_footprints:BME280, symbol giraffe_symbols:BME280
- removed U6: MAX11615, Package_SO:QSOP-16_3.9x4.9mm_P0.635mm, symbol giraffe_symbols:MAX1161x
- removed U8: SAM-M8Q, RF_GPS:ublox_SAM-M8Q, symbol giraffe_symbols:SAM-M8Q
- removed U9: AD1582B, Package_TO_SOT_SMD:SOT-23-3, symbol giraffe_symbols:AD1582
- removed Y1: 12MHz, Crystal:Crystal_SMD_0603-2Pin_6.0x3.5mm, symbol Device:Crystal
- added J16, J4: ADC, Connector_PinSocket_1.27mm:PinSocket_2x02_P1.27mm_Vertical, symbol Connector_Generic:Conn_02x02_Counter_Clockwise
- added J2, J8: PI, giraffe_flight_computer_footprints:pi_zero, symbol giraffe_symbols:pi_zero
- added J5, J6: BAT, symbol Connector_Generic:Conn_01x02
Connections:
- new net hat/+BATT: J5.2 (Pin_2)
- new net hat/-BATT: J2.14 (GND), J2.20 (GND), J2.25 (GND), J2.30 (GND), J2.34 (GND), J2.39 (GND), J2.6 (GND), J2.9 (GND), J5.1 (Pin_1)
- new net hat/1_WIRE: J2.7 (GCLK0/GPIO4)
- new net hat/3V3: J2.1 (3V3), J2.17 (3V3)
- new net hat/5V: J2.2 (5V), J2.4 (5V)
- new net hat/ADC.CH4: J4.1 (Pin_1)
- new net hat/ADC.CH5: J4.2 (Pin_2)
- new net hat/ADC.CH6: J4.3 (Pin_3)
- new net hat/ADC.CH7: J4.4 (Pin_4)
- new net hat/BMI088.INT1: J2.29 (GCLK1/GPIO5)
- new net hat/BMI088.INT3: J2.31 (GCLK2/GPIO6)
- new net hat/EEPROM.SCL: J2.28 (ID_SC/GPIO1)
- new net hat/EEPROM.SDA: J2.27 (ID_SD/GPIO0)
- new net hat/I2C0.SCL: J2.5 (SCL/GPIO3)
- new net hat/I2C0.SDA: J2.3 (SDA/GPIO2)
- new net hat/PCM.CLK: J2.12 (GPIO18/PWM0)
- new net hat/PCM.DIN: J2.38 (GPIO20/MOSI1)
- new net hat/PCM.DOUT: J2.40 (GPIO21/SCLK1)
- new net hat/PCM.FS: J2.35 (GPIO19/MISO1)
- new net hat/SAM_M8Q.RST: J2.33 (PWM1/GPIO13)
- new net hat/SAM_M8Q.TX_RDY: J2.32 (PWM0/GPIO12)
- new net hat/SPI0.CE0: J2.24 (~{CE0}/GPIO8)
- new net hat/SPI0.CE1: J2.26 (~{CE1}/GPIO7)
- new net hat/SPI0.MISO: J2.21 (MISO0/GPIO9)
- new net hat/SPI0.MOSI: J2.19 (MOSI0/GPIO10)
- new net hat/SPI0.SCLK: J2.23 (SCLK0/GPIO11)
- new net hat/STATUS_LED.BLUE: J2.15 (GPIO22)
- new net hat/STATUS_LED.GREEN: J2.13 (GPIO27)
- new net hat/STATUS_LED.RED: J2.11 (GPIO17)
- new net shoe/+BATT: J6.2 (Pin_2)
- new net shoe/-BATT: J6.1 (Pin_1), J8.14 (GND), J8.20 (GND), J8.25 (GND), J8.30 (GND), J8.34 (GND), J8.39 (GND), J8.6 (GND), J8.9 (GND)
- new net shoe/3V3: J8.1 (3V3), J8.17 (3V3)
- new net shoe/5V: J8.2 (5V), J8.4 (5V)
- new net shoe/SA868.PTT: J8.18 (GPIO24)
- new net shoe/SA868.PWR: J8.16 (GPIO23)
- new net shoe/SA868.RX: J8.22 (GPIO25)
- new net shoe/UART.RX: J8.10 (GPIO15/RXD)
- new net shoe/UART.TX: J8.8 (GPIO14/TXD)
- no-connect marks 45 -> 30
Other:
- added sheet hat (hat.kicad_sch)
- added sheet shoe (shoe.kicad_sch)
- note removed: "1-Wire Expansion Bus"
- note removed: "BME280 Temperature/Pressure/Humidity Sensor"
- note removed: "BMI088 IMU/GYRO"
- note removed: "Boost Converter"
- note removed: "Current Sensor"
- note removed: "DS18B20 Temperature Sensor (On Board)"
- note removed: "GPIO Configuration EEPROM / EEPROM I2C Bus"
- note removed: "HAT"
- note removed: "I2C Expansion Bus"
- note removed: "MAX11615 12-Bit 8-Channel I2C ADC With External 2.5V Reference Voltage"
- note removed: "Optional"
- note removed: "Optional Pull-Up Resistors May not be needed due to internal pull-ups depending on device/wires added to the I2C header."
- note removed: "PCM2902C USB PCM Audio Interface"
- note removed: "PCM2902C/SA868 Audio Connection"
- note removed: "Reverse Polarity Protection"
- note removed: "SA868 RF Low Pass Filter"
- note removed: "SA868 VHF Radio Module"
- note removed: "SAM-M8Q GPS Module"
- note removed: "SHOE"
- note removed: "Status LED"
- note removed: "eevblog.com/forum/projects /how-does-the-zvd-circuit-work/"
