File: hardware/giraffe_flight_computer/giraffe_flight_computer.kicad_sch (KiCad schematic)
At the start: 6 parts, among them J1 PI, J2 BAT, J3 ADC, J4 BAT, J5 ADC, J6 PI

Commit message: [pre-commit.ci] auto fixes from pre-commit.com hooks
for more information, see https://pre-commit.ci
Connections:
- net hat/PCM.DOUT renamed hat/PCM.DOUBT
Other:
- sheet hat ports: added PCM.DOUBT; removed PCM.DOUT
Changed lines of the file:
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@@
       (effects (font (size 1.27 1.27)) (justify right))
     )
-    (pin "PCM.DOUT" input (at 50.8 96.52 0)
+    (pin "PCM.DOUBT" input (at 50.8 96.52 0)
       (effects (font (size 1.27 1.27)) (justify right))
     )
