File: hardware/giraffe_flight_computer/giraffe_flight_computer.kicad_pcb (KiCad board)
At the start: 4 copper layers, 65 x 30 mm, 135 parts, among them J1 PI, J10 BATT_C, J2 BAT, J3 ADC, J4 BAT, J5 ADC, J6 PI, J8 USB, J9 EXT_AUDIO, Q3 NPN, U1 CAT24C32, U10 PCM2902C, U11 TPS61033, U12 ISO6720B, U14 74LVC1G04, U15 TLP185, U16 TLP185, U2 BMI088, U3 DS18B20, U4 TPS61033, U5 BME280, U7 MAX11615, U8 SAM-M8Q, U9 AD1582B, Y1 12MHz

Commit message: More hardware updates
Routing:
- net H_GND: vias 32 -> 51
Other:
- board text removed: "BMI088"
Changed lines of the file:
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@@
         (effects (font (size 1 1) (thickness 0.15)) (justify right mirror))
     )
-    (fp_text value "~" (at 0 0) (layer "B.SilkS")
+    (fp_text value "~" (at 2.75 0.05) (layer "B.SilkS")
         (effects (font (size 1.27 1.27) (thickness 0.15)) (justify mirror))
     )
@@
     )
   )
-  (gr_rect (start 57.25 28.25) (end 61.25 33.75)
-    (stroke (width 0.15) (type default)) (fill none) (layer "F.SilkS"))
   (gr_rect (start 49.35 34.65) (end 51.15 38)
     (stroke (width 0.15) (type default)) (fill none) (layer "F.SilkS"))
@@
     (effects (font (size 0.6 0.6) (thickness 0.125) bold) (justify left bottom))
   )
-  (gr_text "BMI088" (at 59.25 28) (layer "F.SilkS" knockout)
-    (effects (font (size 0.7 0.7) (thickness 0.125) bold) (justify bottom))
-  )
   (gr_text "OT" (at 83.5 28 270) (layer "F.SilkS")
     (effects (font (size 0.5 0.5) (thickness 0.125) bold) (justify left bottom))
@@
   (via (at 29.485 33.9) (size 0.6) (drill 0.3) (layers "F.Cu" "B.Cu") (net 1))
   (via (at 77.75 33) (size 0.8) (drill 0.4) (layers "F.Cu" "B.Cu") (free) (net 1))
+  (via (at 66.6 27.25) (size 0.8) (drill 0.4) (layers "F.Cu" "B.Cu") (free) (net 1))
   (via (at 32.5 24.25) (size 0.6) (drill 0.3) (layers "F.Cu" "B.Cu") (free) (net 1))
   (via (at 29.25 22) (size 0.6) (drill 0.3) (layers "F.Cu" "B.Cu") (free) (net 1))
+  (via (at 27.6 44.65) (size 0.8) (drill 0.4) (layers "F.Cu" "B.Cu") (free) (net 1))
   (via (at 30.75 22) (size 0.6) (drill 0.3) (layers "F.Cu" "B.Cu") (free) (net 1))
+  (via (at 54.45 45.55) (size 0.8) (drill 0.4) (layers "F.Cu" "B.Cu") (free) (net 1))
+  (via (at 87.05 47.35) (size 0.8) (drill 0.4) (layers "F.Cu" "B.Cu") (free) (net 1))
   (via (at 68.5 44.25) (size 0.8) (drill 0.4) (layers "F.Cu" "B.Cu") (free) (net 1))
   (via (at 69.25 41.5) (size 0.8) (drill 0.4) (layers "F.Cu" "B.Cu") (free) (net 1))
+  (via (at 28.3 46.35) (size 0.8) (drill 0.4) (layers "F.Cu" "B.Cu") (free) (net 1))
   (via (at 31.5 24.25) (size 0.6) (drill 0.3) (layers "F.Cu" "B.Cu") (free) (net 1))
   (via (at 90.3 43.1) (size 0.9) (drill 0.5) (layers "F.Cu" "B.Cu") (net 1))
   (via (at 82.75 33.75) (size 0.8) (drill 0.4) (layers "F.Cu" "B.Cu") (free) (net 1))
+  (via (at 84.9 43.05) (size 0.8) (drill 0.4) (layers "F.Cu" "B.Cu") (free) (net 1))
+  (via (at 30.4 47.05) (size 0.8) (drill 0.4) (layers "F.Cu" "B.Cu") (free) (net 1))
   (via (at 32.5 23.5) (size 0.6) (drill 0.3) (layers "F.Cu" "B.Cu") (free) (net 1))
+  (via (at 77.65 38.7) (size 0.8) (drill 0.4) (layers "F.Cu" "B.Cu") (free) (net 1))
   (via (at 79 28.75) (size 0.8) (drill 0.4) (layers "F.Cu" "B.Cu") (free) (net 1))
+  (via (at 64.55 28.25) (size 0.8) (drill 0.4) (layers "F.Cu" "B.Cu") (free) (net 1))
   (via (at 30 22) (size 0.6) (drill 0.3) (layers "F.Cu" "B.Cu") (free) (net 1))
+  (via (at 53.25 39.35) (size 0.8) (drill 0.4) (layers "F.Cu" "B.Cu") (free) (net 1))
+  (via (at 89.45 46.65) (size 0.8) (drill 0.4) (layers "F.Cu" "B.Cu") (free) (net 1))
   (via (at 67.5 43) (size 0.8) (drill 0.4) (layers "F.Cu" "B.Cu") (free) (net 1))
+  (via (at 71.1 38.4) (size 0.8) (drill 0.4) (layers "F.Cu" "B.Cu") (free) (net 1))
   (via (at 34.6 33.5) (size 0.6) (drill 0.3) (layers "F.Cu" "B.Cu") (free) (net 1))
   (via (at 67.5 32) (size 0.8) (drill 0.4) (layers "F.Cu" "B.Cu") (free) (net 1))
@@
   (via (at 80.75 32) (size 0.8) (drill 0.4) (layers "F.Cu" "B.Cu") (free) (net 1))
   (via (at 78.75 33.75) (size 0.8) (drill 0.4) (layers "F.Cu" "B.Cu") (free) (net 1))
+  (via (at 45.5 45.45) (size 0.8) (drill 0.4) (layers "F.Cu" "B.Cu") (free) (net 1))
+  (via (at 90.5 44.85) (size 0.8) (drill 0.4) (layers "F.Cu" "B.Cu") (free) (net 1))
   (via (at 70.25 29.25) (size 0.8) (drill 0.4) (layers "F.Cu" "B.Cu") (free) (net 1))
+  (via (at 55.6 25.9) (size 0.8) (drill 0.4) (layers "F.Cu" "B.Cu") (free) (net 1))
   (via (at 79.75 44.25) (size 0.8) (drill 0.4) (layers "F.Cu" "B.Cu") (free) (net 1))
+  (via (at 73.75 41.1) (size 0.8) (drill 0.4) (layers "F.Cu" "B.Cu") (free) (net 1))
+  (via (at 63.65 29.95) (size 0.8) (drill 0.4) (layers "F.Cu" "B.Cu") (free) (net 1))
   (via (at 78 42) (size 0.8) (drill 0.4) (layers "F.Cu" "B.Cu") (free) (net 1))
   (via (at 79.75 31) (size 0.8) (drill 0.4) (layers "F.Cu" "B.Cu") (free) (net 1))
@@
   (via (at 31.5 23.5) (size 0.6) (drill 0.3) (layers "F.Cu" "B.Cu") (free) (net 1))
   (via (at 80.75 43.25) (size 0.8) (drill 0.4) (layers "F.Cu" "B.Cu") (free) (net 1))
+  (via (at 83.9 31.05) (size 0.8) (drill 0.4) (layers "F.Cu" "B.Cu") (free) (net 1))
   (via (at 35.3 33.5) (size 0.6) (drill 0.3) (layers "F.Cu" "B.Cu") (free) (net 1))
+  (via (at 69.3 27.3) (size 0.8) (drill 0.4) (layers "F.Cu" "B.Cu") (free) (net 1))
   (via (at 78.5 41.25) (size 0.8) (drill 0.4) (layers "F.Cu" "B.Cu") (free) (net 1))
   (via (at 65.25 40.5) (size 0.8) (drill 0.4) (layers "F.Cu" "B.Cu") (free) (net 1))
@@
   (segment (start 38.75 29.75) (end 40.75 29.75) (width 0.1524) (layer "In1.Cu") (net 30))
   (segment (start 40.75 29.75) (end 41.25 29.25) (width 0.1524) (layer "In1.Cu") (net 30))
-  (segment (start 56.053115 36.553115) (end 56.25 36.75) (width 0.1524) (layer "In1.Cu") (net 30))
   (segment (start 41.25 29.25) (end 41.25 27) (width 0.1524) (layer "In1.Cu") (net 30))
   (segment (start 82 46) (end 66 46) (width 0.1524) (layer "In2.Cu") (net 30))
@@
   (segment (start 47.498 23.044) (end 48.75 24.296) (width 0.1524) (layer "F.Cu") (net 37))
   (segment (start 57.658 29.1705) (end 57.658 23.044) (width 0.1524) (layer "B.Cu") (net 40))
-  (segment (start 58 23.386) (end 57.658 23.044) (width 0.1524) (layer "B.Cu") (net 40))
   (segment (start 57.9875 29.5) (end 57.658 29.1705) (width 0.1524) (layer "B.Cu") (net 40))
   (via (at 58.5 28) (size 0.8) (drill 0.4) (layers "F.Cu" "B.Cu") (net 41))

Commit message: Giraffe Flight Computer Hat REV A complete
Parts:
- moved TP3 4.81 mm to (50.9, 46.9)
- moved PWR 0.75 mm to (141.0, 46.5)
- moved RX 0.75 mm to (148.0, 46.5)
- moved TX 0.75 mm to (144.5, 46.5)
- moved R44 0.51 mm to (141.0, 45.0)
- moved R45 0.50 mm to (148.0, 45.0)
- moved R47 0.50 mm to (144.5, 45.0)
- renumbered LED3 to PWR, LED4 to RX, LED5 to TX
Routing:
- net /hat/+BATT: track 23.7 -> 20.1 mm
- net /shoe/+BATT: track 19.7 -> 22.9 mm, vias 0 -> 3
- net Net-(C47-Pad1): track 1.45 -> 4.47 mm
- net H_GND: track 13.6 -> 16.0 mm, vias 51 -> 67
- net Net-(LED5-A): track 0.00 -> 1.52 mm
- net Net-(LED4-A): track 0.00 -> 1.52 mm
- net unconnected-(U4-PG-Pad4): track 0.97 -> 0.00 mm, vias 1 -> 0
- net /shoe/SA868_RX: track 34.4 -> 33.6 mm
- net /shoe/SA868_PTT: track 36.4 -> 35.9 mm
- net S_GND: vias 3 -> 20
- added copper zone on B.Cu, net /hat/+BATT
Other:
- board text added: "5V A G"
- board text added: "GIRAFFE FLIGHT COMPUTER"
- board text added: "V1 Rev A"
- board text added: "github.com/joshua-jerred/giraffe"
- board text removed: "5V ADC GND"

Commit message: lower flight computer board schematic complete
Parts:
- removed C47: 36pF, Capacitor_SMD:C_0603_1608Metric
- removed C48: 20pF, Capacitor_SMD:C_0603_1608Metric
- removed J4: BAT, giraffe_flight_computer_footprints:battery_connection
- removed J5: ADC, Connector_PinHeader_1.27mm:PinHeader_1x01_P1.27mm_Vertical
- removed L5: 56uH, giraffe_flight_computer_footprints:Murata-LQH3NPH_ME-0-0-MFG
- removed PWR (x2): PWR, LED_SMD:LED_0603_1608Metric
- removed R40, R41: ?, Resistor_SMD:R_0603_1608Metric
- removed R42: ?k, Resistor_SMD:R_0603_1608Metric
- removed R43, R44, R45, R46, R47: ?Ω, Resistor_SMD:R_0603_1608Metric
- removed R48: 0Ω, Resistor_SMD:R_0603_1608Metric
- removed RV2: 100k, Potentiometer_SMD:Potentiometer_Bourns_TC33X_Vertical
- removed RX: RX, LED_SMD:LED_0603_1608Metric
- removed TX: PTT, LED_SMD:LED_0603_1608Metric
- removed U14: 74LVC1G04, Package_TO_SOT_SMD:SOT-353_SC-70-5
- removed U15, U16: TLP185, Package_SO:SOIC-4_4.55x3.7mm_P2.54mm
- added C12: 100μF, Capacitor_Tantalum_SMD:CP_EIA-7343-31_Kemet-D, F.Cu at (108.7, -0.87)
- added C23: 10μF, Capacitor_Tantalum_SMD:CP_EIA-3216-18_Kemet-A, F.Cu at (119.8, 8.38)
- added K1: TLP241A, Package_DIP:DIP-4_W8.89mm_SMDSocket_LongPads, F.Cu at (123.7, 27.9)
- added LED1: SML-D12M8WT86, LED_SMD:LED_0603_1608Metric, F.Cu at (51.8, 33.0)
- added LED3: PWR, LED_SMD:LED_0603_1608Metric, F.Cu at (114.9, 3.35)
- added LED4: RX, LED_SMD:LED_0603_1608Metric, F.Cu at (114.9, 5.94)
- added LED5: PTT, LED_SMD:LED_0603_1608Metric, F.Cu at (114.9, 8.53)
- added R21: 0Ω, Resistor_SMD:R_0603_1608Metric, F.Cu at (101.7, -9.29)
- added R31: ?Ω, Resistor_SMD:R_0603_1608Metric, F.Cu at (101.7, -6.78)
- added R34: ?Ω, Resistor_SMD:R_0603_1608Metric, F.Cu at (101.7, -4.27)
- added R36: 0Ω, Resistor_SMD:R_0603_1608Metric, F.Cu at (101.7, -1.76)
- added R37: 0Ω, Resistor_SMD:R_0603_1608Metric, F.Cu at (101.7, 0.75)
- added R38: 0Ω, Resistor_SMD:R_0603_1608Metric, F.Cu at (101.7, 3.26)
- added RV3: 100k, Potentiometer_SMD:Potentiometer_Bourns_TC33X_Vertical, F.Cu at (144.6, 14.0)
- added TP1: 3v3, TestPoint:TestPoint_Pad_D1.0mm, F.Cu at (105.3, 3.58)
- added TP4: TestPoint, TestPoint:TestPoint_Pad_D1.0mm, F.Cu at (105.3, 6.63)
- added TP5: TestPoint, TestPoint:TestPoint_Pad_D1.0mm, F.Cu at (108.3, 3.58)
- added TP6: TestPoint, TestPoint:TestPoint_Pad_D1.0mm, F.Cu at (108.3, 6.63)
- added TP7: TestPoint, TestPoint:TestPoint_Pad_D1.0mm, F.Cu at (111.4, 3.58)
- added TP8: TestPoint, TestPoint:TestPoint_Pad_D1.0mm, F.Cu at (111.4, 6.63)
- added U13: 74LVC1G04, Package_TO_SOT_SMD:SOT-353_SC-70-5, F.Cu at (119.5, -8.54)
- added U6: TLP185, Package_SO:SOIC-4_4.55x3.7mm_P2.54mm, F.Cu at (132.8, 2.54)
- AE1: value ~ -> ANT
- C38: value 10μF -> 20pF; footprint Capacitor_Tantalum_SMD:CP_EIA-3216-18_Kemet-A -> Capacitor_SMD:C_0603_1608Metric; moved to B.Cu
- C44: value 20pF -> 36pF
- C45: value 100μF -> 36pF; footprint Capacitor_Tantalum_SMD:CP_EIA-7343-31_Kemet-D -> Capacitor_SMD:C_0603_1608Metric; moved to B.Cu
- C46: value 36pF -> 20pF
- L2: value 0.47uH -> 56uH; footprint Inductor_SMD:L_Coilcraft_XAL4020-XXX -> giraffe_flight_computer_footprints:Murata-LQH3NPH_ME-0-0-MFG; moved to B.Cu
- L3: value 56uH -> 68uH
- L4: value 68uH -> 56uH
- LED2: value STATUS -> B36S3RGB-F6C0001HOU1930
- R1: value ?Ω -> 56Ω
- R10: value ? -> 2.2k
- R19: value ?k -> ?Ω; footprint Potentiometer_SMD:Potentiometer_Bourns_TC33X_Vertical -> Resistor_SMD:R_0603_1608Metric
- R33: value ?k -> ?Ω
- R35: value ?k -> 0Ω
- R39: value 10kΩ -> 0Ω
- R6: value ?Ω -> 270Ω
- R7, R8: value ?Ω -> 360Ω
- R9: value ? -> 6.8k
- TP9: value ~ -> TestPoint; footprint TestPoint:TestPoint_Pad_1.0x1.0mm -> TestPoint:TestPoint_Pad_D1.0mm
- U11: value TPS61033 -> TLP185; footprint Package_TO_SOT_SMD:SOT-583-8 -> Package_SO:SOIC-4_4.55x3.7mm_P2.54mm
- moved C45 15.6 mm to (128.5, 40.1)
- moved C44 11.1 mm to (130.6, 33.0), turned to 90 degrees
- moved L2 11.0 mm to (132.8, 41.4), turned to 90 degrees
- moved C38 8.33 mm to (136.1, 42.7), turned to 0 degrees
- moved L3 5.88 mm to (129.5, 36.6), turned to 180 degrees
- moved C46 5.03 mm to (125.5, 33.0)
- moved L4 3.77 mm to (125.7, 36.6)
Connections:
- net Net-(TX1-MIC_IN) renamed /shoe/SA868 MIC_IN
- net Net-(TX1-RXD) renamed /shoe/SA868 UART RXD
- net Net-(TX1-TXD) renamed /shoe/SA868 UART TXD
- net Net-(U7-REF) renamed /hat/ADC_V_REF
- C25 pad 1: /shoe/+BATT -> S_5V
- C32 pad 1: S_4V -> S_5V
- C38 pad 1: S_4V -> /shoe/SA868 RF
- C41 pad 2: S_4V -> S_5V
- C42 pad 2: S_4V -> S_5V
- C43 pad 2: S_4V -> S_5V
- C44 pad 1: Net-(TX1-ANT) -> Net-(C44-Pad1)
- C45 pad 1: S_4V -> Net-(C45-Pad1)
- C46 pad 1: Net-(C46-Pad1) -> Net-(AE1-A)
- J6 pad 2: S_5V -> /shoe/S_5V_IN
- J6 pad 22: /shoe/SA868_RX -> /shoe/RX_DETECT
- J6 pad 4: S_5V -> /shoe/S_5V_IN
- L2 pad 1: /shoe/+BATT -> /shoe/SA868 RF
- L2 pad 2: Net-(U11-SW) -> Net-(C44-Pad1)
- L3 pad 1: Net-(TX1-ANT) -> Net-(C44-Pad1)
- L3 pad 2: Net-(C46-Pad1) -> Net-(C45-Pad1)
- L4 pad 1: Net-(C46-Pad1) -> Net-(C45-Pad1)
- L4 pad 2: Net-(C47-Pad1) -> Net-(AE1-A)
- R19 pad 1: Net-(U11-FB) -> /shoe/SA868_PWR_CTRL
- R19 pad 2: Net-(R19-Pad2) -> Net-(K1-Anode)
- R20 pad 1: Net-(U11-EN) -> S_5V
- R20 pad 2: /shoe/SA868_PWR_CTRL -> Net-(LED3-A)
- R33 pad 1: S_4V -> Net-(R33-Pad1)
- R33 pad 2: Net-(R19-Pad2) -> Net-(LED5-A)
- R35 pad 1: Net-(U11-FB) -> Net-(R35-Pad1)
- R35 pad 2: S_GND -> /shoe/SA868 PTT
- R39 pad 1: Net-(TX1-PD) -> /shoe/SA868 AUDIO_OUT
- R39 pad 2: S_4V -> Net-(C48-Pad1)
- RV1 pad 3: /shoe/AUDIO_OUT_LEFT -> Net-(C47-Pad1)
- TP9 pad 1: S_4V -> /shoe/SA868 AUDIO_OUT
- TX1 pad 1: Net-(TX1-SQ) -> /shoe/SA868 RX
- TX1 pad 12: Net-(TX1-ANT) -> /shoe/SA868 RF
- TX1 pad 3: Net-(TX1-AF_OUT) -> /shoe/SA868 AUDIO_OUT
- TX1 pad 5: Net-(TX1-PTT) -> /shoe/SA868 PTT
- TX1 pad 8: S_4V -> S_5V
- U11 pad 1: /shoe/+BATT -> Net-(R34-Pad1)
- U11 pad 4: unconnected-(U11-PG-Pad4) -> Net-(R33-Pad1)
- U11 pad 6: S_GND -> S_5V
- U12 pad 8: S_4V -> S_5V
Routing:
- net S_4V: track 71.0 -> 0.00 mm, vias 9 -> 0
- net (no net): track 0.00 -> 44.8 mm
- net S_5V: track 81.8 -> 123.6 mm, vias 0 -> 10
- net /shoe/SA868_RX: track 33.6 -> 0.00 mm, vias 1 -> 0
- net /shoe/RX_DETECT: track 0.00 -> 33.6 mm, vias 0 -> 1
- net Net-(TX1-AF_OUT): track 32.0 -> 0.00 mm, vias 2 -> 0
- net /shoe/SA868 AUDIO_OUT: track 0.00 -> 32.0 mm, vias 0 -> 2
- net /shoe/+BATT: track 22.9 -> 0.00 mm, vias 3 -> 0
- net Net-(U11-EN): track 18.2 -> 0.00 mm, vias 2 -> 0
- net Net-(TX1-ANT): track 16.6 -> 0.00 mm
- net /shoe/SA868 RF: track 0.00 -> 16.6 mm
- net Net-(TX1-SQ): track 11.9 -> 0.00 mm, vias 1 -> 0
- net /shoe/SA868 RX: track 0.00 -> 11.9 mm, vias 0 -> 1
- net Net-(R33-Pad1): track 0.00 -> 11.9 mm, vias 0 -> 1
- net /shoe/ADC_CH4: track 11.0 -> 0.00 mm
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- added copper zone on F.Cu, net Net-(C44-Pad1)
- added copper zone on B.Cu, net S_5V
- added copper zone on F.Cu, net S_5V
- removed copper zone on F.Cu, net /shoe/+BATT
- removed copper zone on F.Cu, net Net-(U11-SW)
- removed copper zone on B.Cu, net S_4V
- removed copper zone on F.Cu, net S_4V

Commit message: sync pcb work
Parts:
- removed LED4: RX, LED_SMD:LED_0603_1608Metric
- removed R31: ?Ω, Resistor_SMD:R_0603_1608Metric
- removed U13: 74LVC1G04, Package_TO_SOT_SMD:SOT-353_SC-70-5
- added C47: ?, Resistor_SMD:R_0805_2012Metric, F.Cu at (170.5, -51.8)
- added C48: ?, Resistor_SMD:R_0805_2012Metric, F.Cu at (170.5, -48.8)
- added J11: 3V3, giraffe_flight_computer_footprints:battery_connection, F.Cu at (78.7, 12.2)
- added J12: 3V3, giraffe_flight_computer_footprints:battery_connection, F.Cu at (88.9, 10.7)
- added J4: USB, Connector_PinHeader_1.00mm:PinHeader_1x03_P1.00mm_Vertical, F.Cu at (145.1, 2.46)
- added J5: EXT_AUDIO, Connector_PinHeader_1.00mm:PinHeader_1x03_P1.00mm_Vertical, F.Cu at (148.5, 2.46)
- added LED6: ~, LED_SMD:LED_0603_1608Metric, F.Cu at (175.5, -28.6)
- added Q1: BC847CT, Package_TO_SOT_SMD:SOT-23, F.Cu at (131.8, 32.7)
- added Q2: BC847CT, Package_TO_SOT_SMD:SOT-23, F.Cu at (143.9, 38.4)
- added Q4: BC847CT, Package_TO_SOT_SMD:SOT-23, F.Cu at (171.0, -23.4)
- added R40: ?kΩ, Resistor_SMD:R_0603_1608Metric, F.Cu at (139.0, -28.0)
- added R41: 470Ω, Resistor_SMD:R_0603_1608Metric, F.Cu at (130.8, 36.6)
- added R42: 5kΩ, Resistor_SMD:R_0603_1608Metric, F.Cu at (144.0, 29.7)
- added R43: 50kΩ, Resistor_SMD:R_0603_1608Metric, F.Cu at (146.7, 38.5)
- added R44: 10kΩ, Resistor_SMD:R_0603_1608Metric, F.Cu at (143.0, -33.1)
- added R45: 1kΩ, Resistor_SMD:R_0603_1608Metric, F.Cu at (143.0, -30.5)
- added R46: 390Ω, Resistor_SMD:R_0603_1608Metric, F.Cu at (143.0, -28.0)
- C12: moved to B.Cu
- C28, C32, C39, C40: footprint Resistor_SMD:R_0805_2012Metric -> Resistor_SMD:R_0603_1608Metric
- C36, C37, RV1: moved to F.Cu
- J8: value USB -> 3V3; footprint Connector_PinHeader_1.00mm:PinHeader_1x03_P1.00mm_Vertical -> giraffe_flight_computer_footprints:battery_connection
- J9: value EXT_AUDIO -> 3V3; footprint Connector_PinHeader_1.00mm:PinHeader_1x03_P1.00mm_Vertical -> giraffe_flight_computer_footprints:battery_connection
- L2, L4: value 56uH -> 56nH; footprint giraffe_flight_computer_footprints:Murata-LQH3NPH_ME-0-0-MFG -> Inductor_SMD:L_0603_1608Metric_Pad1.05x0.95mm_HandSolder
- L3: value 68uH -> 68nH; footprint giraffe_flight_computer_footprints:Murata-LQH3NPH_ME-0-0-MFG -> Inductor_SMD:L_0603_1608Metric_Pad1.05x0.95mm_HandSolder
- LED5: value PTT -> ~
- R19: value ?Ω -> 50kΩ
- R20, R33: value ?Ω -> 150Ω
- R21: value 0Ω -> 5kΩ
- R34: value ?Ω -> 390Ω
- moved TP2 101.9 mm to (171.0, -45.5)
- moved TP9 80.2 mm to (167.1, -27.5)
- moved LED3 71.1 mm to (175.5, -33.8)
- moved C24 70.7 mm to (131.2, -15.2)
- moved TP1 69.5 mm to (164.0, -33.6)
- moved TP4 69.5 mm to (164.0, -30.5)
- moved U6 68.2 mm to (191.8, -31.8)
- moved TP7 66.9 mm to (167.1, -33.6)
- moved TP8 66.9 mm to (167.1, -30.5)
- moved C26 66.0 mm to (139.8, -15.4)
- moved R28 66.0 mm to (139.8, -12.9), turned to 0 degrees
- moved TP5 63.8 mm to (164.0, -27.5)
- moved TP6 63.8 mm to (164.0, -24.4)
- moved R29 62.7 mm to (139.8, -10.4), turned to 0 degrees
- moved R20 61.6 mm to (135.0, -35.6)
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Connections:
- net /shoe/AUDIO_OUT_LEFT renamed /shoe/USB Audio Codec/audio_codec_out_left
- net /shoe/SA868_PWR_CTRL renamed /shoe/PI_GPIO_SHOE_POWER_CONTROL
- C12 pad 1: S_5V -> /shoe/S_5V_IN
- C23 pad 1: S_5V -> /shoe/S_5V_IN
- C25 pad 1: S_5V -> /shoe/S_5V_IN
- C34 pad 2: /shoe/AUDIO_IN_RIGHT -> /shoe/USB Audio Codec/AUDIO_IN_RIGHT
- C35 pad 2: /shoe/AUDIO_OUT_RIGHT -> /shoe/USB Audio Codec/AUDIO_OUT_RIGHT
- J1 pad 1: H_3V3 -> unconnected-(J1-3V3-Pad1)
- J1 pad 17: H_3V3 -> unconnected-(J1-3V3-Pad17)
- J6 pad 1: S_3V3 -> unconnected-(J6-3V3-Pad1)
- J6 pad 17: S_3V3 -> unconnected-(J6-3V3-Pad17)
- J6 pad 18: /shoe/SA868_PTT -> /shoe/PI_GPIO_SA868_PTT
- J6 pad 22: /shoe/RX_DETECT -> /shoe/PI_GPIO_SA868_RX
- J8 pad 1: S_GND -> S_3V3
- J8 pad 2: Net-(J8-Pin_2) -> (no net)
- J9 pad 1: S_GND -> S_3V3
- J9 pad 2: /shoe/AUDIO_OUT_RIGHT -> (no net)
- K1 pad 1: Net-(K1-Anode) -> /shoe/S_5V_IN
- K1 pad 2: S_GND -> Net-(K1-Cathode)
- LED5 pad 1: S_GND -> Net-(LED5-K)
- R19 pad 2: Net-(K1-Anode) -> Net-(Q1-C)
- R21 pad 1: Net-(R21-Pad1) -> Net-(Q4-C)
- R28 pad 1: Net-(J8-Pin_3) -> Net-(J4-Pin_3)
- R29 pad 1: Net-(J8-Pin_2) -> Net-(J4-Pin_2)
- R33 pad 1: Net-(R33-Pad1) -> Net-(LED5-A)
- R33 pad 2: Net-(LED5-A) -> S_5V
- R34 pad 2: /shoe/SA868_PTT -> Net-(Q2-C)
- R35 pad 1: Net-(R35-Pad1) -> Net-(LED5-K)
- R36 pad 1: S_GND -> Net-(TX1-PD)
- R36 pad 2: Net-(TX1-H/L) -> S_5V
- R37 pad 1: Net-(TX1-PD) -> S_GND
- R37 pad 2: S_5V -> Net-(TX1-H/L)
- U11 pad 1: Net-(R34-Pad1) -> S_5V
- U11 pad 3: S_GND -> Net-(R34-Pad1)
- U11 pad 4: Net-(R33-Pad1) -> S_GND
- U11 pad 6: S_5V -> Net-(LED5-K)
- U6 pad 1: Net-(R21-Pad1) -> Net-(R46-Pad2)
- U6 pad 3: S_GND -> Net-(LED6-K)
- U6 pad 4: /shoe/RX_DETECT -> S_GND
- U6 pad 6: S_3V3 -> Net-(R44-Pad2)
Routing:
- net S_5V: track 123.6 -> 0.00 mm, vias 10 -> 5
- net S_3V3: track 53.2 -> 0.00 mm, vias 2 -> 0
- net (no net): track 44.8 -> 0.00 mm
- net /shoe/UART.TX: track 41.5 -> 0.00 mm, vias 1 -> 0
- net /shoe/UART.RX: track 37.2 -> 0.00 mm, vias 1 -> 0
- net /shoe/SA868_PTT: track 35.9 -> 0.00 mm, vias 1 -> 0
- net /shoe/RX_DETECT: track 33.6 -> 0.00 mm, vias 1 -> 0
- net /shoe/SA868 AUDIO_OUT: track 32.0 -> 0.00 mm, vias 2 -> 0
- net /shoe/S_5V_IN: track 0.00 -> 27.0 mm
- net /shoe/SA868 MIC_IN: track 26.8 -> 0.00 mm, vias 2 -> 0
- net Net-(U10-SEL0): track 18.9 -> 0.00 mm
- net Net-(U10-VINR): track 15.3 -> 0.00 mm, vias 2 -> 0
- net /shoe/PI_GPIO_SHOE_POWER_CONTROL: track 5.92 -> 21.1 mm
- net Net-(U10-VOUTR): track 14.3 -> 0.00 mm, vias 2 -> 0
- net Net-(U10-VOUTL): track 13.8 -> 0.00 mm, vias 2 -> 0
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- removed copper zone on F.Cu, net Net-(C44-Pad1)
- removed copper zone on F.Cu, net S_GND
- removed copper zone on In1.Cu, net S_GND
