File: hardware/legacy/GFC Hat/GFC-Hat.kicad_pcb (KiCad board)
At the start: 4 copper layers, 65 x 30 mm, 45 parts, among them J1 BAT, U1 MCP3021, U2 BME280, U3 CAT24C32, U4 SAM-M8Q, U5 BMI088

Commit message: [pre-commit.ci] auto fixes from pre-commit.com hooks
for more information, see https://pre-commit.ci
Parts:
- TP1: footprint TestPoint:TestPoint_Keystone_5019_Minature -> TestPoint:TestPoint_Keystone_5019_Miniature
Changed lines of the file:
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@@
     )
   )
-  (footprint "TestPoint:TestPoint_Keystone_5019_Minature" (layer "B.Cu")
+  (footprint "TestPoint:TestPoint_Keystone_5019_Miniature" (layer "B.Cu")
     (at 22.54 42.606)
     (descr "SMT Test Point- Micro Miniature 5019, http://www.keyelco.com/product-pdf.cfm?p=1357")
