File: hardware/legacy/GFC Hat/power_supply.kicad_sch (KiCad schematic)
At the start: 17 parts, among them J1 BAT, SW1 Sliding Power Switch, U1 MCP3021, U6 MT3608

Commit message: [pre-commit.ci] auto fixes from pre-commit.com hooks
for more information, see https://pre-commit.ci
Parts:
- TP1: footprint TestPoint:TestPoint_Keystone_5019_Minature -> TestPoint:TestPoint_Keystone_5019_Miniature
Changed lines of the file:
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@@
       (effects (font (size 1.27 1.27)) (justify left))
     )
-    (property "Footprint" "TestPoint:TestPoint_Keystone_5019_Minature" (at 63.5 81.28 0)
+    (property "Footprint" "TestPoint:TestPoint_Keystone_5019_Miniature" (at 63.5 81.28 0)
       (effects (font (size 1.27 1.27)) hide)
     )
