File: hardware/legacy/GFC Shoe/GFC_SHOE.kicad_sch (KiCad schematic)
At the start: 15 parts

Commit message: [pre-commit.ci] auto fixes from pre-commit.com hooks
for more information, see https://pre-commit.ci
Other:
- sheet DAC ports: added DAC{BCLK LRC DIN DOUBT}; removed DAC{BCLK LRC DIN DOUT}
Changed lines of the file:
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@@
     (effects (font (size 1.27 1.27)) (justify left bottom))
   )
-  (global_label "DAC{BCLK LRC DIN DOUT}" (shape input) (at 190.5 82.55 0) (fields_autoplaced)
+  (global_label "DAC{BCLK LRC DIN DOUBT}" (shape input) (at 190.5 82.55 0) (fields_autoplaced)
     (effects (font (size 1.27 1.27)) (justify left))
     (property "Intersheet References" "${INTERSHEET_REFS}" (id 0) (at 217.6479 82.4706 0)
@@
       (effects (font (size 1.27 1.27)) (justify right))
     )
-    (pin "DAC{BCLK LRC DIN DOUT}" input (at 187.96 82.55 0)
+    (pin "DAC{BCLK LRC DIN DOUBT}" input (at 187.96 82.55 0)
       (effects (font (size 1.27 1.27)) (justify right))
     )
