File: hardware/legacy/GFC Shoe/dac.kicad_sch (KiCad schematic)
At the start: 27 parts, among them J1 USB, U1 PCM2902C, Y1 12MHz

Commit message: [pre-commit.ci] auto fixes from pre-commit.com hooks
for more information, see https://pre-commit.ci
Changed lines of the file:
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@@
     (effects (font (size 1.27 1.27)) (justify left bottom))
   )
-  (label "DAC.DOUT" (at 177.8 54.61 0)
+  (label "DAC.DOUBT" (at 177.8 54.61 0)
     (effects (font (size 1.27 1.27)) (justify left bottom))
   )
@@
     (effects (font (size 1.27 1.27)) (justify left))
   )
-  (hierarchical_label "DAC{BCLK LRC DIN DOUT}" (shape input) (at 214.63 64.77 0)
+  (hierarchical_label "DAC{BCLK LRC DIN DOUBT}" (shape input) (at 214.63 64.77 0)
     (effects (font (size 1.27 1.27)) (justify left))
   )
