File: hardware/Prototype Boards/5v Buck Supply/5v Buck Supply.kicad_pcb (KiCad board)
At the start: 2 copper layers, 36.6 x 31.8 mm, 55 parts, among them J1 BATT, J2 PRIMARY, J3 EXTERNAL, J4 IO, Q1 NPN, U1 TPS54302DDCR, U2 INA2180Ax, U3 AP2112K-3.3

Commit message: buck BOM
Parts:
- C6, C7: value C -> DNS
- R15, R17, R19, R21: value R -> 0
