File: hardware/power_board/external_interface.kicad_sch (KiCad schematic)
At the start: 9 parts, among them J5 XT30 Female

Commit message: power board work
Parts:
- removed BC6: N/A, symbol Connector:Conn_01x03_Socket
- removed BT5, BT6: INR18650-35E, symbol Device:Battery_Cell
- removed TH1: Thermistor, symbol Device:Thermistor
- added BC2: ?, symbol Connector_Generic:Conn_01x01
- added BC3, J2: 5019390400, symbol Connector:Conn_01x04_Socket
- added J1: XT30-PW, symbol Connector_Generic:Conn_01x02
- BC1: renamed from J5; value XT30 Female -> XT30-F
Connections:
- net GND: now also BC1.1 (Pin_1), BC3.1 (Pin_1), J1.1 (Pin_1); no longer BC1.2 (Pin_2)
- net at BT1.1 (+), BT3.1 (+): now also BC1.2 (Pin_2); no longer BC1.1 (Pin_1)
- net BATT_BALLANCE: now reaches BT1.2 (-), BT2.1 (+), BT3.2 (-), BT4.1 (+)
- net BATT_BALLANCE: now also BC2.1 (Pin_1)
- new net BATT_EXT_3V3: BC3.2 (Pin_2)
- new net BATT_EXT_I2C_SCL: BC3.4 (Pin_4)
- new net BATT_EXT_I2C_SDA: BC3.3 (Pin_3)
- no-connect marks 0 -> 3
Other:
- note added: "Battery Pack"
- note added: "Upload to pico via debug connection and interface via UART?"
- moved on the sheet: BT1, BT2, BT3, BT4
