File: hardware/power_board/5V_buck_converter.kicad_sch (KiCad schematic)
At the start: 23 parts, among them U1 TPS54302DDCR

Commit message: power board work
Parts:
- added R12: 0Ω, symbol Device:R
- renumbered C11 to C?, C16 to C?, C7 to C?, C8 to C?, C4 to C?, C17 to C?, C1 to C?, C2 to C?, C15 to C?, C3 to C?, C9 to C?, L1 to L?, R15 to R?, R2 to R?, R16 to R?, R14 to R?, R1 to R?, TP2 to TP?, TP1 to TP?, TP5 to TP?, TP3 to TP?, TP4 to TP?, U1 to U?
Connections:
- net +5V is gone; now on net 5.1V_BUCK_OUTPUT: C?.1, C?.1, L?.1, R?.1, TP?.1
- net +BATT_FILTERED: now also C?.1, C?.1
- net BUCK_CONVERTER_DISABLE: now also R12.2; no longer R?.1, R?.2, TP?.1, U?.5 (EN)
- net 5.1V_BUCK_OUTPUT: now reaches C?.1, C?.1, C?.1
- new net buck_enable: R12.1, R?.1, R?.2, TP?.1, U?.5 (EN)
Other:
- note added: "5.1 V OUTPUT https://datasheets.raspberrypi.com/hat/hat-plus-specification.pdf"
- note added: "Optional 5V side bulk capacitance"
- note added: "Optional battery side bulk capacitance"
- moved on the sheet: C?, R?, TP?, U?

Commit message: sync
Parts:
- U?: Unit Price (none) -> 1.06
Changed lines of the file:
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@@
 	(text_box "TODO: 3V3 LDO or Buck?\n\nhttps://www.adafruit.com/product/2745"
 		(exclude_from_sim no)
-		(at 189.23 128.27 0)
+		(at 170.18 143.51 0)
 		(size 35.56 12.7)
 		(margins 0.9525 0.9525 0.9525 0.9525)
@@
 			)
 		)
+		(property "BOARD" ""
+			(at 195.58 69.85 0)
+			(effects
+				(font
+					(size 1.27 1.27)
+				)
+			)
+		)
 		(pin "2"
 		)
@@
 			)
 		)
+		(property "BOARD" ""
+			(at 186.69 69.85 0)
+			(effects
+				(font
+					(size 1.27 1.27)
+				)
+			)
+		)
 		(pin "1"
 		)
@@
 			)
 		)
+		(property "BOARD" ""
+			(at 233.68 62.23 0)
+			(effects
+				(font
+					(size 1.27 1.27)
+				)
+			)
+		)
 		(pin "1"
 		)
@@
 			)
 		)
+		(property "BOARD" ""
+			(at 81.28 60.96 0)
+			(effects
+				(font
+					(size 1.27 1.27)
+				)
+			)
+		)
 		(pin "1"
 		)
@@
 			)
 		)
+		(property "BOARD" ""
+			(at 66.04 78.74 0)
+			(effects
+				(font
+					(size 1.27 1.27)
+				)
+			)
+		)
 		(pin "2"
 		)
@@
 			)
 		)
+		(property "BOARD" ""
+			(at 139.7 41.91 0)
+			(effects
+				(font
+					(size 1.27 1.27)
+				)
+			)
+		)
 		(pin "1"
 		)
@@
 			)
 		)
+		(property "BOARD" ""
+			(at 195.58 80.01 0)
+			(effects
+				(font
+					(size 1.27 1.27)
+				)
+			)
+		)
 		(pin "2"
 		)
@@
 			)
 		)
+		(property "BOARD" ""
+			(at 167.64 50.8 0)
+			(effects
+				(font
+					(size 1.27 1.27)
+				)
+			)
+		)
 		(pin "1"
 		)
@@
 			)
 		)
+		(property "BOARD" ""
+			(at 76.2 46.99 0)
+			(effects
+				(font
+					(size 1.27 1.27)
+				)
+			)
+		)
 		(pin "1"
 		)
@@
 			)
 		)
+		(property "BOARD" ""
+			(at 242.57 62.23 0)
+			(effects
+				(font
+					(size 1.27 1.27)
+				)
+			)
+		)
 		(pin "1"
 		)
@@
 			)
 		)
+		(property "BOARD" ""
+			(at 34.29 55.88 0)
+			(effects
+				(font
+					(size 1.27 1.27)
+				)
+			)
+		)
 		(pin "1"
 		)
@@
 			)
 		)
+		(property "BOARD" ""
+			(at 195.58 59.69 0)
+			(effects
+				(font
+					(size 1.27 1.27)
+				)
+			)
+		)
 		(pin "2"
 		)
@@
 			)
 		)
+		(property "BOARD" ""
+			(at 88.9 41.91 0)
+			(effects
+				(font
+					(size 1.27 1.27)
+				)
+			)
+		)
 		(pin "1"
 		)
@@
 			)
 		)
-		(property "Unit Price" ""
+		(property "Unit Price" "1.06"
 			(at 107.95 49.53 0)
 			(effects
@@
 			)
 		)
+		(property "BOARD" ""
+			(at 107.95 49.53 0)
+			(effects
+				(font
+					(size 1.27 1.27)
+				)
+			)
+		)
 		(pin "6"
 		)
@@
 			)
 		)
+		(property "BOARD" ""
+			(at 43.18 55.88 0)
+			(effects
+				(font
+					(size 1.27 1.27)
+				)
+			)
+		)
 		(pin "1"
 		)
@@
 			)
 		)
+		(property "BOARD" ""
+			(at 251.46 62.23 0)
+			(effects
+				(font
+					(size 1.27 1.27)
+				)
+			)
+		)
 		(pin "1"
 		)
@@
 			)
 		)
+		(property "BOARD" ""
+			(at 74.93 66.04 0)
+			(effects
+				(font
+					(size 1.27 1.27)
+				)
+			)
+		)
 		(pin "1"
 		)
@@
 			)
 		)
+		(property "BOARD" ""
+			(at 162.56 46.99 0)
+			(effects
+				(font
+					(size 1.27 1.27)
+				)
+			)
+		)
 		(pin "1"
 		)
@@
 			)
 		)
+		(property "BOARD" ""
+			(at 149.86 46.99 0)
+			(effects
+				(font
+					(size 1.27 1.27)
+				)
+			)
+		)
 		(pin "1"
 		)
@@
 			)
 		)
+		(property "BOARD" ""
+			(at 64.77 46.99 0)
+			(effects
+				(font
+					(size 1.27 1.27)
+				)
+			)
+		)
 		(pin "1"
 		)
@@
 			)
 		)
+		(property "BOARD" ""
+			(at 81.28 71.12 0)
+			(effects
+				(font
+					(size 1.27 1.27)
+				)
+			)
+		)
 		(pin "1"
 		)
@@
 			)
 		)
+		(property "BOARD" ""
+			(at 160.02 74.93 0)
+			(effects
+				(font
+					(size 1.27 1.27)
+				)
+			)
+		)
 		(pin "1"
 		)
@@
 			)
 		)
+		(property "BOARD" ""
+			(at 156.21 46.99 0)
+			(effects
+				(font
+					(size 1.27 1.27)
+				)
+			)
+		)
 		(pin "1"
 		)
@@
 			)
 		)
+		(property "BOARD" ""
+			(at 179.07 50.8 0)
+			(effects
+				(font
+					(size 1.27 1.27)
+				)
+			)
+		)

Commit message: sync
Parts:
- added C18, C20: 1uf, Capacitor_SMD:C_0805_2012Metric, symbol Device:C
- added Q2: MMBT3904LT1G, Package_TO_SOT_SMD:SOT-23, symbol Simulation_SPICE:NPN
- added R17: 10k, Capacitor_SMD:C_0603_1608Metric_Pad1.08x0.95mm_HandSolder, symbol Device:R
- added R18: 1k, Capacitor_SMD:C_0603_1608Metric_Pad1.08x0.95mm_HandSolder, symbol Device:R
- added R19: 0, Resistor_SMD:R_0805_2012Metric_Pad1.20x1.40mm_HandSolder, symbol Device:R
- added TP3: TestPoint, TestPoint:TestPoint_Pad_D1.0mm, symbol Connector:TestPoint_Small
- added TP7, TP8: TestPoint ks, footprints:KEYSTONE_5015, symbol Connector:TestPoint
- added U2: AP2112K-3.3, Package_TO_SOT_SMD:SOT-23-5, symbol Regulator_Linear:AP2112K-3.3
Connections:
- net GND: now also C18.2, C20.2, Q2.3 (E), U2.2 (GND)
- net 5.1V_BUCK_OUTPUT renamed 5.1V_PRIMARY_OUTPUT
- new net: Q2.2 (B), R18.1
- new net 3V3 Primary: R19.2, TP8.1
- new net 3V3_DISABLE: R18.2
- new net 3v3_en: Q2.1 (C), R17.1, TP3.1, U2.3 (EN)
- new net 3v3_out: C20.1, R19.1, TP7.1, U2.5 (VOUT)
- new net 5V Primary: C18.1, R17.2, U2.1 (VIN)
Other:
- note added: "3V3 LDO"

Commit message: sync
Parts:
- gave numbers to parts that had none: 23
