File: hardware/power_board/power_board.kicad_pcb (KiCad board)
At the start: 4 copper layers, 65 x 30 mm, 148 parts, among them J1 PI, J10 BATT_C, J11 3V3, J12 3V3, J2 BAT, J3 ADC, J4 USB, J5 EXT_AUDIO, J6 PI, J8 3V3, J9 3V3, K1 TLP241A, Q1 BC847CT, Q2 BC847CT, Q3 NPN, Q4 BC847CT, Q5 BC847CT, U1 CAT24C32, U10 PCM2902C, U11 TLP185, U12 ISO6720B, U2 BMI088, U3 DS18B20, U4 TPS61033, U5 BME280, U7 MAX11615, U8 SAM-M8Q, U9 AD1582B, Y1 12MHz

Commit message: sync
Parts:
- removed 1W1: 1W1, giraffe_flight_computer_footprints:Molex-52745-0497
- removed 1W2: 1W2, giraffe_flight_computer_footprints:Molex-52745-0497
- removed C19: 10μF, Capacitor_Tantalum_SMD:CP_EIA-3216-18_Kemet-A
- removed C47, C48: ?, Resistor_SMD:R_0805_2012Metric
- removed I2C1: I²C, giraffe_flight_computer_footprints:Molex-52745-0497
- removed J1, J6: PI, giraffe_flight_computer_footprints:pi_zero
- removed J10: BATT_C, Connector_PinHeader_1.00mm:PinHeader_1x03_P1.00mm_Vertical
- removed J11, J12, J8, J9: 3V3, giraffe_flight_computer_footprints:battery_connection
- removed J2: BAT, giraffe_flight_computer_footprints:battery_connection
- removed J3: ADC, Connector_PinSocket_1.27mm:PinSocket_2x02_P1.27mm_Vertical
- removed J4: USB, Connector_PinHeader_1.00mm:PinHeader_1x03_P1.00mm_Vertical
- removed J7: ~, Connector_PinHeader_1.00mm:PinHeader_1x04_P1.00mm_Vertical
- removed K1: TLP241A, Package_DIP:DIP-4_W8.89mm_SMDSocket_LongPads
- removed L1: 0.47uH, Inductor_SMD:L_Coilcraft_XAL4020-XXX
- removed L2, L4: 56nH, Inductor_SMD:L_0603_1608Metric_Pad1.05x0.95mm_HandSolder
- removed L3: 68nH, Inductor_SMD:L_0603_1608Metric_Pad1.05x0.95mm_HandSolder
- removed LED1: SML-D12M8WT86, LED_SMD:LED_0603_1608Metric
- removed LED2: B36S3RGB-F6C0001HOU1930, giraffe_flight_computer_footprints:B36S3RGB LED
- removed LED3: PWR, LED_SMD:LED_0603_1608Metric
- removed LED5, LED6: ~, LED_SMD:LED_0603_1608Metric
- removed PCM1: PCM, Connector_PinHeader_1.27mm:PinHeader_1x04_P1.27mm_Vertical
- removed Q1, Q4, Q5: BC847CT, Package_TO_SOT_SMD:SOT-23
- removed R1: 56Ω, Resistor_SMD:R_0603_1608Metric
- removed R10: 2.2k, Resistor_SMD:R_0603_1608Metric
- removed R11: 4.7kΩ, Resistor_SMD:R_0603_1608Metric
- removed R12, R13, R2, R3: ?, Resistor_SMD:R_0603_1608Metric
- removed R14, R35, R36, R37, R38, R39: 0Ω, Resistor_SMD:R_0603_1608Metric
- removed R15: 21.5k, Resistor_SMD:R_0603_1608Metric
- removed R16: 1k, Potentiometer_SMD:Potentiometer_Bourns_TC33X_Vertical
- removed R20, R33: 150Ω, Resistor_SMD:R_0603_1608Metric
- removed R26, R27: ?Ω, Resistor_SMD:R_0603_1608Metric
- removed R28, R29: 22Ω, Resistor_SMD:R_0603_1608Metric
- removed R30: 1.5kΩ, Resistor_SMD:R_0603_1608Metric
- removed R31, R42, R46: 5kΩ, Resistor_SMD:R_0603_1608Metric
- removed R32: 1MΩ, Resistor_SMD:R_0603_1608Metric
- removed R34: 390Ω, Resistor_SMD:R_0603_1608Metric
- removed R4, R5: 3.9kΩ, Resistor_SMD:R_0603_1608Metric
- removed R40: ?kΩ, Resistor_SMD:R_0603_1608Metric
- removed R41: 470Ω, Resistor_SMD:R_0603_1608Metric
- removed R43: 50kΩ, Resistor_SMD:R_0603_1608Metric
- removed R6: 270Ω, Resistor_SMD:R_0603_1608Metric
- removed R7, R8: 360Ω, Resistor_SMD:R_0603_1608Metric
- removed R9: 6.8k, Resistor_SMD:R_0603_1608Metric
- removed RV1, RV3: 100k, Potentiometer_SMD:Potentiometer_Bourns_TC33X_Vertical
- removed TP1: 3v3, TestPoint:TestPoint_Pad_D1.0mm
- removed TP2: GND, TestPoint:TestPoint_Keystone_5015_Micro-Minature
- removed TP4, TP5, TP6, TP7, TP8, TP9: TestPoint, TestPoint:TestPoint_Pad_D1.0mm
- removed TX1: SA868, giraffe_flight_computer_footprints:DORJI_DRA818V
- removed U10: PCM2902C, Package_SO:SSOP-28_5.3x10.2mm_P0.65mm
- removed U11: TLP185, Package_SO:SOIC-4_4.55x3.7mm_P2.54mm
- removed U12: ISO6720B, Package_SO:SOIC-8_3.9x4.9mm_P1.27mm
- removed U4: TPS61033, Package_TO_SOT_SMD:SOT-583-8
- removed U8: SAM-M8Q, RF_GPS:ublox_SAM-M8Q
- removed U9: AD1582B, Package_TO_SOT_SMD:SOT-23-3
- removed Y1: 12MHz, Crystal:Crystal_SMD_0603-2Pin_6.0x3.5mm
- added TP12: TestPoint, TestPoint:TestPoint_Pad_D1.0mm, F.Cu at (39.4, 62.4)
- added U6: Si5351A-B-GT, Package_SO:MSOP-10_3x3mm_P0.5mm, F.Cu at (80.3, 69.0)
- AE1: value ANT -> ~; footprint giraffe_flight_computer_footprints:MolexSmaConnector -> giraffe_flight_computer_footprints:LINX_CONSMA001-G; moved to F.Cu
- C1, C3: value 0.1µF -> 15pf; footprint Capacitor_SMD:C_0603_1608Metric -> Capacitor_SMD:C_0603_1608Metric_Pad1.08x0.95mm_HandSolder; moved to F.Cu
- C10, C2, C9: value 0.1µF -> 0.1uf; footprint Capacitor_SMD:C_0603_1608Metric -> Capacitor_SMD:C_0603_1608Metric_Pad1.08x0.95mm_HandSolder; moved to F.Cu
- C11, C25, C6: value 10μF -> 0.1uf; footprint Capacitor_Tantalum_SMD:CP_EIA-3216-18_Kemet-A -> Capacitor_SMD:C_0603_1608Metric_Pad1.08x0.95mm_HandSolder
- C12: value 100μF -> 1uf; footprint Capacitor_Tantalum_SMD:CP_EIA-7343-31_Kemet-D -> Capacitor_SMD:C_0603_1608Metric_Pad1.08x0.95mm_HandSolder; moved to F.Cu
- C13: value 0.1µF -> 1uf; footprint Capacitor_SMD:C_0603_1608Metric -> Capacitor_SMD:C_0603_1608Metric_Pad1.08x0.95mm_HandSolder
- C14, C15, C7, C8: value 0.1µF -> 0.1uf; footprint Capacitor_SMD:C_0603_1608Metric -> Capacitor_SMD:C_0603_1608Metric_Pad1.08x0.95mm_HandSolder
- C16: value 0.1µF -> DNS; footprint Capacitor_SMD:C_0603_1608Metric -> Capacitor_SMD:C_0603_1608Metric_Pad1.08x0.95mm_HandSolder; moved to F.Cu
- C17: value 1μF -> DNS; footprint Resistor_SMD:R_0805_2012Metric -> Capacitor_SMD:C_0603_1608Metric_Pad1.08x0.95mm_HandSolder
- C18: value 100μF -> 1uf; footprint Capacitor_Tantalum_SMD:CP_EIA-7343-31_Kemet-D -> Capacitor_SMD:C_0805_2012Metric; moved to F.Cu
- C20: value 0.1µF -> 1uf; footprint Capacitor_SMD:C_0603_1608Metric -> Capacitor_SMD:C_0805_2012Metric
- C21, C5: value 0.1µF -> ?; footprint Capacitor_SMD:C_0603_1608Metric -> Capacitor_SMD:C_0603_1608Metric_Pad1.08x0.95mm_HandSolder
- C22: value 0.1µF -> DNS; footprint Capacitor_SMD:C_0603_1608Metric -> Capacitor_SMD:C_1210_3225Metric_Pad1.33x2.70mm_HandSolder
- C23: value 10μF -> DNS; footprint Capacitor_Tantalum_SMD:CP_EIA-3216-18_Kemet-A -> Capacitor_SMD:C_1210_3225Metric_Pad1.33x2.70mm_HandSolder
- C24: value 1μF -> 10uf; footprint Resistor_SMD:R_0805_2012Metric -> Capacitor_SMD:C_1210_3225Metric
- C26: value 1μF -> 0.1uf; footprint Capacitor_SMD:C_0603_1608Metric -> Capacitor_SMD:C_0603_1608Metric_Pad1.08x0.95mm_HandSolder
- C27: value 10μF -> 22uf; footprint Resistor_SMD:R_1210_3225Metric -> Capacitor_SMD:C_1210_3225Metric
- C28: value 0.1μF -> 22uf; footprint Resistor_SMD:R_0603_1608Metric -> Capacitor_SMD:C_1210_3225Metric
- C29: value 10μF -> 75pf; footprint Resistor_SMD:R_1210_3225Metric -> Capacitor_SMD:C_0603_1608Metric_Pad1.08x0.95mm_HandSolder
- C30: value 1uF -> DNS; footprint Resistor_SMD:R_0805_2012Metric -> Capacitor_SMD:C_1210_3225Metric_Pad1.33x2.70mm_HandSolder
- C31: value 1μF -> DNS; footprint Resistor_SMD:R_0805_2012Metric -> Capacitor_SMD:C_1210_3225Metric_Pad1.33x2.70mm_HandSolder
- C32: value 0.1μF -> DNS; footprint Resistor_SMD:R_0603_1608Metric -> Capacitor_SMD:C_1210_3225Metric_Pad1.33x2.70mm_HandSolder
- C33: value 1μF -> 1uf; footprint Resistor_SMD:R_0805_2012Metric -> Capacitor_SMD:C_0603_1608Metric_Pad1.08x0.95mm_HandSolder
- C34: value 1μF -> 10uf; footprint Resistor_SMD:R_0805_2012Metric -> Capacitor_SMD:C_0603_1608Metric_Pad1.08x0.95mm_HandSolder
- C35, C36, C37: value 1μF -> 0.1uf; footprint Resistor_SMD:R_0805_2012Metric -> Capacitor_SMD:C_0603_1608Metric_Pad1.08x0.95mm_HandSolder
- C38: value 20pF -> ?pf; footprint Capacitor_SMD:C_0603_1608Metric -> Capacitor_SMD:C_0603_1608Metric_Pad1.08x0.95mm_HandSolder; moved to F.Cu
- C39: value 0.1μF -> ?pf; footprint Resistor_SMD:R_0603_1608Metric -> Capacitor_SMD:C_0603_1608Metric_Pad1.08x0.95mm_HandSolder
- C4: value 0.1µF -> ?; footprint Capacitor_SMD:C_0603_1608Metric -> Capacitor_SMD:C_0603_1608Metric_Pad1.08x0.95mm_HandSolder; moved to F.Cu
- C40: value 0.1μF -> ?; footprint Resistor_SMD:R_0603_1608Metric -> Capacitor_SMD:C_0603_1608Metric_Pad1.08x0.95mm_HandSolder
- C41: value 0.1µF -> 1uf; footprint Capacitor_SMD:C_0603_1608Metric -> Capacitor_SMD:C_0603_1608Metric_Pad1.08x0.95mm_HandSolder; moved to F.Cu
- C42: value 10kpF -> ?; footprint Capacitor_SMD:C_0603_1608Metric -> Capacitor_SMD:C_0603_1608Metric_Pad1.08x0.95mm_HandSolder; moved to F.Cu
- C43: value 1kpF -> ?; footprint Capacitor_SMD:C_0603_1608Metric -> Capacitor_SMD:C_0603_1608Metric_Pad1.08x0.95mm_HandSolder; moved to F.Cu
- C44, C45: value 36pF -> ?; footprint Capacitor_SMD:C_0603_1608Metric -> Capacitor_SMD:C_0603_1608Metric_Pad1.08x0.95mm_HandSolder; moved to F.Cu
- C46: value 20pF -> 1uf; footprint Capacitor_SMD:C_0603_1608Metric -> Capacitor_SMD:C_0603_1608Metric_Pad1.08x0.95mm_HandSolder; moved to F.Cu
- J5: value EXT_AUDIO -> PI; footprint Connector_PinHeader_1.00mm:PinHeader_1x03_P1.00mm_Vertical -> giraffe_flight_computer_footprints:pi_zero
- Q2: value BC847CT -> MMBT3904LT1G
- Q3: value NPN -> BC847CT; moved to F.Cu
- R17: value 3k -> 10k; footprint Resistor_SMD:R_0603_1608Metric -> Capacitor_SMD:C_0603_1608Metric_Pad1.08x0.95mm_HandSolder
- R18: value 0Ω -> 1k; footprint Resistor_SMD:R_0603_1608Metric -> Capacitor_SMD:C_0603_1608Metric_Pad1.08x0.95mm_HandSolder
- R19: value 50kΩ -> 0; footprint Resistor_SMD:R_0603_1608Metric -> Resistor_SMD:R_0805_2012Metric_Pad1.20x1.40mm_HandSolder
- R21: value 5kΩ -> DNS; footprint Resistor_SMD:R_0603_1608Metric -> Resistor_SMD:R_0603_1608Metric_Pad0.98x0.95mm_HandSolder
- R22: value ? -> DNS; footprint Resistor_SMD:R_0603_1608Metric -> Resistor_SMD:R_0603_1608Metric_Pad0.98x0.95mm_HandSolder
- R23: value ? -> 49; footprint Resistor_SMD:R_0603_1608Metric -> Resistor_SMD:R_0603_1608Metric_Pad0.98x0.95mm_HandSolder
- R24: value * -> 100k; footprint Resistor_SMD:R_0603_1608Metric -> Resistor_SMD:R_0603_1608Metric_Pad0.98x0.95mm_HandSolder; moved to F.Cu
- R25: value * -> 13.3k; footprint Resistor_SMD:R_0603_1608Metric -> Resistor_SMD:R_0603_1608Metric_Pad0.98x0.95mm_HandSolder; moved to F.Cu
- TP3: value GND -> TestPoint; footprint TestPoint:TestPoint_Keystone_5015_Micro-Minature -> TestPoint:TestPoint_Pad_D1.0mm
- U1: value CAT24C32 -> INA180A; footprint giraffe_flight_computer_footprints:CAT24C32WI_GT3 -> Package_TO_SOT_SMD:SOT-23-5; moved to F.Cu
- U2: value BMI088 -> AP2112K-3.3; footprint giraffe_flight_computer_footprints:BMI088 -> Package_TO_SOT_SMD:SOT-23-5; moved to F.Cu
- U3: value DS18B20 -> W25Q128JVS; footprint Package_SO:MSOP-8_3x3mm_P0.65mm -> Package_SO:SOIC-8_5.3x5.3mm_P1.27mm
- U5: value BME280 -> RP2040; footprint giraffe_flight_computer_footprints:BME280 -> Package_DFN_QFN:QFN-56-1EP_7x7mm_P0.4mm_EP3.2x3.2mm
- U7: value MAX11615 -> MIC2091-2YM5; footprint Package_SO:QSOP-16_3.9x4.9mm_P0.635mm -> Package_TO_SOT_SMD:SOT-23-5; moved to F.Cu
- moved R21 209.4 mm to (24.0, 71.6)
- moved C26 139.1 mm to (24.0, 61.6)
- moved C29 132.0 mm to (24.0, 64.1)
- moved C31 130.9 mm to (29.2, 72.7)
- moved C30 130.1 mm to (29.2, 68.4)
- moved C27 124.7 mm to (35.0, 64.2)
- moved C24 122.1 mm to (35.0, 59.9)
- moved Q2 121.5 mm to (39.1, 73.0), turned to 0 degrees
- moved C35 117.1 mm to (54.4, 69.1)
- moved C32 111.9 mm to (29.2, 76.9), turned to 0 degrees
- moved R19 106.6 mm to (28.5, 80.5), turned to 0 degrees
- moved C28 106.2 mm to (35.0, 68.4), turned to 0 degrees
- moved C33 104.2 mm to (54.4, 64.1)
- moved C34 103.9 mm to (54.4, 66.6)
- moved C25 98.8 mm to (24.0, 59.1), turned to 0 degrees
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Connections:
- C1 pad 1: H_3V3 -> Net-(U5-XIN)
- C1 pad 2: H_GND -> GND
- C10 pad 1: H_GND -> GND
- C10 pad 2: H_3V3 -> 3V3_PICO
- C11 pad 1: H_5V -> GND
- C11 pad 2: H_GND -> 3V3_PICO
- C12 pad 1: /shoe/S_5V_IN -> GND
- C12 pad 2: S_GND -> 3V3_PICO
- C13 pad 1: H_3V3 -> GND
- C13 pad 2: H_GND -> /RP2040/+1V1_PICO_ADC_REF
- C14 pad 1: H_3V3 -> GND
- C14 pad 2: H_GND -> /RP2040/+1V1_PICO_ADC_REF
- C15 pad 1: H_3V3 -> GND
- C15 pad 2: H_GND -> /RP2040/+1V1_PICO_ADC_REF
- C16 pad 1: H_3V3 -> GND
- C16 pad 2: H_GND -> /Power Input/battery_voltage_signal
- C17 pad 1: /hat/ADC_V_REF -> GND
- C17 pad 2: H_GND -> /Power Input/input_current_sense_signal
- C18 pad 1: H_5V -> 5V Primary
- C18 pad 2: H_GND -> GND
- C2 pad 1: H_GND -> +3V3_RP2040
- C2 pad 2: H_3V3 -> GND
- C20 pad 1: H_GND -> /Voltage Converters/3v3_out
- C20 pad 2: H_5V -> GND
- C21 pad 1: H_5V -> unconnected-(C21-Pad1)
- C21 pad 2: H_GND -> unconnected-(C21-Pad2)
- C22 pad 1: H_5V -> /Power Input/power_input_processed
- C22 pad 2: H_GND -> GND
- C23 pad 1: /shoe/S_5V_IN -> /Power Input/power_input_processed
- C23 pad 2: S_GND -> GND
- C24 pad 1: S_5V -> /Power Input/power_input_processed
- C24 pad 2: S_GND -> GND
- C25 pad 1: /shoe/S_5V_IN -> /Power Input/power_input_processed
- C25 pad 2: S_GND -> GND
- C26 pad 1: S_GND -> /Voltage Converters/buck_boot
- C26 pad 2: Net-(U10-SEL0) -> /Voltage Converters/buck_sw
- C27 pad 1: Net-(U10-VCCCI) -> 5V_PRIMARY
- C27 pad 2: S_GND -> GND
- C28 pad 1: S_GND -> 5V_PRIMARY
- C28 pad 2: S_3V3 -> GND
- C29 pad 1: Net-(U10-VCOM) -> Net-(C29-Pad1)
- C29 pad 2: S_GND -> /Voltage Converters/buck_feedback
- C3 pad 1: H_GND -> Net-(C3-Pad1)
- C3 pad 2: H_3V3 -> GND
- C30 pad 1: S_GND -> 5V_PRIMARY
- C30 pad 2: Net-(U10-VCCP1I) -> GND
- C31 pad 1: S_GND -> 5V_PRIMARY
- C31 pad 2: Net-(U10-VCCP2I) -> GND
- C32 pad 1: S_5V -> 5V_PRIMARY
- C32 pad 2: S_GND -> GND
- C33 pad 1: S_GND -> GND
- C33 pad 2: Net-(U10-VCCXI) -> 3V3_PICO
- C34 pad 1: Net-(U10-VOUTR) -> GND
- C34 pad 2: /shoe/USB Audio Codec/AUDIO_IN_RIGHT -> 3V3_PICO
- C35 pad 1: Net-(U10-VINR) -> GND
- C35 pad 2: /shoe/USB Audio Codec/AUDIO_OUT_RIGHT -> 3V3_PICO
- C36 pad 1: Net-(U10-VOUTL) -> GND
- C36 pad 2: /shoe/USB Audio Codec/audio_codec_out_left -> /RP2040/WSPR Transmitter/Si5351_3V3
- C37 pad 1: Net-(U10-VINL) -> GND
- C37 pad 2: /shoe/AUDIO_IN_LEFT -> /RP2040/WSPR Transmitter/Si5351_3V3
- C38 pad 1: /shoe/SA868 RF -> GND
- C38 pad 2: S_GND -> Net-(U6-XA)
- C39 pad 1: Net-(U10-XTI) -> GND
- C39 pad 2: S_GND -> Net-(U6-XB)
- C4 pad 1: H_GND -> unconnected-(C4-Pad1)
- C4 pad 2: H_3V3 -> unconnected-(C4-Pad2)
- C40 pad 1: Net-(U10-XTO) -> Net-(C40-Pad1)
- C40 pad 2: S_GND -> Net-(U6-CLK0)
- C41 pad 1: S_GND -> GND
- C41 pad 2: S_5V -> 3V3_PICO
- C42 pad 1: S_GND -> GND
- C42 pad 2: S_5V -> Net-(C40-Pad1)
- C43 pad 1: S_GND -> GND
- C43 pad 2: S_5V -> Net-(C43-Pad2)
- C44 pad 1: Net-(C44-Pad1) -> GND
- C44 pad 2: S_GND -> Net-(C44-Pad2)
- C45 pad 1: Net-(C45-Pad1) -> GND
- C45 pad 2: S_GND -> Net-(AE1-A)
- C46 pad 1: Net-(AE1-A) -> GND
- C46 pad 2: S_GND -> 3V3_PICO
- C5 pad 1: H_GND -> Net-(U1-IN-)
- C5 pad 2: H_3V3 -> Net-(U1-IN+)
- C6 pad 1: /hat/+BATT -> GND
- C6 pad 2: H_GND -> 3V3_PICO
- C7 pad 1: H_GND -> GND
- C7 pad 2: H_3V3 -> 3V3_PICO
- C8 pad 1: H_GND -> GND
- C8 pad 2: H_3V3 -> 3V3_PICO
- C9 pad 1: H_GND -> GND
- C9 pad 2: H_3V3 -> 3V3_PICO
- J5 pad 1: S_GND -> unconnected-(J5-3V3-Pad1)
- J5 pad 2: /shoe/USB Audio Codec/AUDIO_OUT_RIGHT -> +5V
- J5 pad 3: /shoe/USB Audio Codec/AUDIO_IN_RIGHT -> I2C0.SDA
- Q2 pad 1: Net-(Q2-B) -> /Voltage Converters/3v3_en
- Q2 pad 2: S_GND -> Net-(Q2-B)
- Q2 pad 3: Net-(Q2-C) -> GND
- Q3 pad 2: Net-(Q3-C) -> GND
- Q3 pad 3: H_GND -> Net-(Q3-C)
- R17 pad 1: Net-(U4-FB) -> /Voltage Converters/3v3_en
- R17 pad 2: H_GND -> 5V Primary
- R18 pad 1: Net-(U5-SDO) -> Net-(Q2-B)
- R18 pad 2: H_3V3 -> 3V3_DISABLE
- R19 pad 1: /shoe/PI_GPIO_SHOE_POWER_CONTROL -> /Voltage Converters/3v3_out
- R19 pad 2: Net-(Q1-B) -> 3V3 Primary
- R21 pad 1: Net-(Q4-B) -> /Voltage Converters/buck_enable
- R21 pad 2: /shoe/SA868 RX -> /Power Input/power_input_processed
- R22 pad 1: H_5V -> GND
- R22 pad 2: /hat/ADC.CH2 -> /Voltage Converters/buck_enable
- R23 pad 1: /hat/ADC.CH2 -> 5V_PRIMARY
- R23 pad 2: H_GND -> Net-(C29-Pad1)
- R24 pad 1: /hat/I2C0.SDA -> Net-(C29-Pad1)
- R24 pad 2: H_3V3 -> /Voltage Converters/buck_feedback
- R25 pad 1: H_3V3 -> /Voltage Converters/buck_feedback
- R25 pad 2: /hat/I2C0.SCL -> GND
- TP3 pad 1: H_GND -> /Voltage Converters/3v3_en
- U1 pad 1: H_GND -> /Power Input/input_current_sense_signal
- U1 pad 2: H_GND -> GND
- U1 pad 3: H_GND -> Net-(U1-IN+)
- U1 pad 4: H_GND -> Net-(U1-IN-)
- U1 pad 5: /hat/EEPROM.SDA -> +3V3_RP2040
- U2 pad 1: unconnected-(U2-INT2-Pad1) -> 5V Primary
- U2 pad 2: H_GND -> GND
- U2 pad 3: H_3V3 -> /Voltage Converters/3v3_en
- U2 pad 4: H_GND -> unconnected-(U2-NC-Pad4)
- U2 pad 5: /hat/SPI0.CE1 -> /Voltage Converters/3v3_out
- U3 pad 1: unconnected-(U3-NC-Pad1) -> /RP2040/QSPI_SS
- U3 pad 2: unconnected-(U3-NC-Pad2) -> /RP2040/QSPI_SD1
- U3 pad 3: H_3V3 -> /RP2040/QSPI_SD2
- U3 pad 4: /hat/1_WIRE -> GND
- U3 pad 5: H_GND -> /RP2040/QSPI_SD0
- U3 pad 6: unconnected-(U3-NC-Pad6) -> /RP2040/QSPI_SCLK
- U3 pad 7: unconnected-(U3-NC-Pad7) -> /RP2040/QSPI_SD3
- U3 pad 8: unconnected-(U3-NC-Pad8) -> 3V3_PICO
- U5 pad 1: H_GND -> 3V3_PICO
- U5 pad 2: H_3V3 -> /RP2040/2040_UART0.TX
- U5 pad 3: /hat/I2C0.SDA -> /RP2040/2040_UART0.RX
- U5 pad 4: /hat/I2C0.SCL -> /RP2040/2040_I2C1.SDA
- U5 pad 5: Net-(U5-SDO) -> /RP2040/2040_I2C1.SCL
- U5 pad 6: H_3V3 -> /RP2040/2040_UART1.TX
- U5 pad 7: H_GND -> /RP2040/2040_UART1.RX
- U5 pad 8: H_3V3 -> unconnected-(U5-GPIO6-Pad8)
- U7 pad 1: /hat/ADC_V_REF -> 3V3_PICO
- U7 pad 2: unconnected-(U7-NC-Pad2) -> GND
- U7 pad 3: unconnected-(U7-NC-Pad3) -> /RP2040/WSPR Transmitter/WSPR_POWER_ENABLE
- U7 pad 4: unconnected-(U7-NC-Pad4) -> /RP2040/WSPR Transmitter/WSPR_POWER_FAULT
- U7 pad 5: /hat/ADC.CH0 -> /RP2040/WSPR Transmitter/Si5351_3V3
Routing:
- net /hat/I2C0.SCL: track 86.2 -> 0.00 mm, vias 5 -> 0
- net /hat/I2C0.SDA: track 85.2 -> 0.00 mm, vias 4 -> 0
- net H_5V: track 83.9 -> 0.00 mm, vias 4 -> 0
- net H_3V3: track 58.0 -> 0.00 mm, vias 19 -> 0
- net /hat/ADC.CH5: track 41.7 -> 0.00 mm, vias 2 -> 0
- net /hat/ADC.CH4: track 40.8 -> 0.00 mm, vias 1 -> 0
- net /hat/ADC.CH7: track 40.7 -> 0.00 mm, vias 1 -> 0
- net /hat/ADC.CH6: track 39.3 -> 0.00 mm, vias 1 -> 0
- net /hat/EEPROM.SDA: track 38.8 -> 0.00 mm, vias 1 -> 0
- net /hat/PCM.CLK: track 38.5 -> 0.00 mm
- net /hat/1_WIRE: track 34.7 -> 0.00 mm, vias 3 -> 0
- net /hat/EEPROM.SCL: track 33.0 -> 0.00 mm, vias 1 -> 0
- net /shoe/S_5V_IN: track 27.0 -> 0.00 mm
- net /hat/BMI088.INT1: track 24.3 -> 0.00 mm, vias 2 -> 0
- net /hat/SAM_M8Q.RST: track 21.5 -> 0.00 mm, vias 1 -> 0
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- removed copper zone on B.Cu, net /hat/+BATT
- removed copper zone on F.Cu, net /hat/+BATT
- removed copper zone on F.Cu, net /hat/BOOST_SW
- removed copper zone on In1.Cu, net H_3V3
- removed copper zone on F.Cu, net H_5V
- removed copper zone on B.Cu, net H_GND
- removed copper zone on F.Cu, net H_GND
- removed copper zone on In2.Cu, net H_GND
- removed copper zone on B.Cu, net S_5V
- removed copper zone on F.Cu, net S_5V
- removed copper zone on B.Cu, net S_GND
- removed copper zone on In2.Cu, net S_GND
Other:
- outline, holes or cut-outs redrawn
- board text removed: "0x76"
- board text removed: "0x77"
- board text removed: "1-W EXT0"
- board text removed: "1-W EXT1"
- board text removed: "3v3"
- board text removed: "5V A G"
- board text removed: "ADC"
- board text removed: "CH6 CH4"
- board text removed: "CH7 CH5"
- board text removed: "CK"
- board text removed: "EEPROM PROG"
- board text removed: "EXT ADC"
- board text removed: "FS"
- board text removed: "GIRAFFE FLIGHT COMPUTER"
- board text removed: "GND"
- board text removed: "I2C EXT"
- board text removed: "IN"
- board text removed: "OT"
- board text removed: "SCL"
- board text removed: "SDA"
- board text removed: "V1 Rev A"
- board text removed: "github.com/joshua-jerred/giraffe"

Commit message: sync
Parts:
- removed J5: PI, giraffe_flight_computer_footprints:pi_zero
- removed U3: W25Q128JVS, Package_SO:SOIC-8_5.3x5.3mm_P1.27mm
- added C19: 0.1uf, Capacitor_SMD:C_0603_1608Metric_Pad1.08x0.95mm_HandSolder, F.Cu at (85.1, 73.5)
- added C47: 2.2uf, Capacitor_SMD:C_0603_1608Metric_Pad1.08x0.95mm_HandSolder, F.Cu at (85.1, 76.0)
Connections:
- net /Power Input/power_input_processed renamed /Main Power Supply/+BATT_FILTERED
- net /RP2040/PRIMARY_POWER_SUPPLY_DISABLE renamed /Main Power Supply/BUCK_CONVERTER_DISABLE
- net /Voltage Converters/3v3_en renamed /Main Power Supply/3v3_en
- net /Voltage Converters/3v3_out renamed /Main Power Supply/3v3_out
- net /Voltage Converters/buck_boot renamed /Main Power Supply/buck_boot
- net /Voltage Converters/buck_enable renamed /Main Power Supply/buck_enable
- net /Voltage Converters/buck_feedback renamed /Main Power Supply/buck_feedback
- net /Voltage Converters/buck_sw renamed /Main Power Supply/buck_sw
