File: hardware/power_board/power_board.kicad_sch (KiCad schematic)
At the start: 44 parts, among them J1 Screw_Terminal_01x02, J12 PI, J4 IO, J7 PRIMARY, J8 EXTERNAL, Q1 MMBT3904LT1G, Q2 Q_PMOS_GDS, U2 RP2040, U3 AP2112K-3.3, U4 CAT24C32, U6 INA180A

Commit message: power board work
Parts:
- removed BC1: n/a, symbol Connector_Generic:Conn_02x03_Counter_Clockwise
- removed BC2: ?, symbol Connector_Generic:Conn_01x02
- removed C18, C19: ~, symbol Device:C_Small
- removed C5: DNS, Capacitor_SMD:C_0603_1608Metric_Pad1.08x0.95mm_HandSolder, symbol Device:C_Small
- removed C6: 0.1uf, Capacitor_SMD:C_0603_1608Metric_Pad1.08x0.95mm_HandSolder, symbol Device:C
- removed D1: D_Zener, symbol Device:D_Zener
- removed J1: Screw_Terminal_01x02, symbol Connector:Screw_Terminal_01x02
- removed J4: IO, Connector_PinHeader_2.54mm:PinHeader_1x06_P2.54mm_Vertical, symbol Connector:Conn_01x06_Socket
- removed J7: PRIMARY, TerminalBlock_TE-Connectivity:TerminalBlock_TE_282834-3_1x03_P2.54mm_Horizontal, symbol Connector:Screw_Terminal_01x03
- removed J8: EXTERNAL, TerminalBlock_TE-Connectivity:TerminalBlock_TE_282834-2_1x02_P2.54mm_Horizontal, symbol Connector:Screw_Terminal_01x02
- removed Q2: Q_PMOS_GDS, symbol Device:Q_PMOS_GDS
- removed R10, R9: DNS, Capacitor_SMD:C_0603_1608Metric_Pad1.08x0.95mm_HandSolder, symbol Device:R_Small
- removed R11, R13, R7, R8: 0, Capacitor_SMD:C_0603_1608Metric_Pad1.08x0.95mm_HandSolder, symbol Device:R_Small
- removed R12: 0.05, Resistor_SMD:R_0805_2012Metric_Pad1.20x1.40mm_HandSolder, symbol Device:R
- removed R17: 0, Resistor_SMD:R_0805_2012Metric_Pad1.20x1.40mm_HandSolder, symbol Device:R
- removed R18: 0, symbol Device:R_Small
- removed R25: 100R, symbol Device:R
- removed R3: 18k, Capacitor_SMD:C_0603_1608Metric_Pad1.08x0.95mm_HandSolder, symbol Device:R_Small
- removed R4: 3.3k, Capacitor_SMD:C_0603_1608Metric_Pad1.08x0.95mm_HandSolder, symbol Device:R_Small
- removed R5, R6: 10k, Capacitor_SMD:C_0603_1608Metric_Pad1.08x0.95mm_HandSolder, symbol Device:R_Small
- removed TP6, TP7: TestPoint, symbol Connector:TestPoint
- removed U2: RP2040, Package_DFN_QFN:QFN-56-1EP_7x7mm_P0.4mm_EP3.2x3.2mm, symbol MCU_RaspberryPi:RP2040
- removed U4: CAT24C32, SOIC127P600X175-8N, symbol a_giraffe_symbols:CAT24C32WI-GT3
- removed U6: INA180A, symbol a_giraffe_symbols:INA180A
- added C?: ?, Capacitor_SMD:C_0603_1608Metric_Pad1.08x0.95mm_HandSolder, symbol Device:C_Small
- added JP?: 0603 0Ω, Resistor_SMD:R_1210_3225Metric, symbol Jumper:SolderJumper_2_Open
- added R5, R?: ?Ω, symbol Device:R
- added TP?: ~, symbol Connector:TestPoint
- renumbered C10 to C?, C13 to C?, D2 to D?, J12 to J?, Q1 to Q?, R24 to R?, R22 to R?, R21 to R?, R19 to R?, TP10 to TP?, TP11 to TP?, TP9 to TP?, U3 to U?
Other:
- sheet 18650 Pack renamed Power Input
- sheet 5V Buck Converter renamed Voltage Converters
- added sheet RP2040 (rp2040.kicad_sch)
- sheet Power Input: file 18650_pack.kicad_sch -> power_input.kicad_sch
- sheet Power Input ports: added batt_ext_3V3, batt_ext_I2C_SCL, batt_ext_I2C_SDA, battery_voltage_signal, input_current_sense_signal, power_input_processed; removed +BATT, -BATT, BATTERY_PACK_BALLANCE
- sheet Voltage Converters ports: added 3V3_PRIMARY_OUTPUT, 3V3_RP2040_OUTPUT; removed none
- note removed: "5.1 V OUTPUT https://datasheets.raspberrypi.com/hat/hat-plus-specification.pdf"
- note removed: "Battery Pack"
- note removed: "Current Sense"
- note removed: "https://components101.com/articles /design-guide-pmos-mosfet-for- reverse-voltage-polarity-protection"
- moved on the sheet: C?, D?, Q?, R?, TP?, U?

Commit message: sync
Parts:
- removed D?: LED, symbol Device:LED
- removed R?: ~, symbol Device:R_Small
- added C4: ?, Capacitor_SMD:C_0603_1608Metric_Pad1.08x0.95mm_HandSolder, symbol Device:C_Small
- added R15, R8: 5.1kΩ, symbol Device:R
- added SB1, SB2, SB3: ~, symbol Jumper:SolderJumper_2_Open
- added TP4, TP5, TP6: ~, symbol Connector:TestPoint
- added USB: USB_C_Receptacle_USB2.0_14P, symbol a_giraffe_symbols:USB_C_Receptacle_USB2.0_14P
- U?: Unit Price (none) -> 0.56
Connections:
- net GND: now also R15.2, R8.2, SB3.1 (A), USB.A1 (GND), USB.A12 (GND), USB.B1 (GND), USB.B12 (GND)
- new net: R15.1, TP6.1, USB.A5 (CC1)
- new net: R8.1, TP5.1, USB.B5 (CC2)
- new net: SB3.2 (B), USB.S1 (SHIELD)
- new net USB_C.D+: USB.A6 (D+), USB.B6 (D+)
- new net USB_C.D-: USB.A7 (D-), USB.B7 (D-)
- new net USB_C_VBUS: USB.A4 (VBUS), USB.A9 (VBUS), USB.B4 (VBUS), USB.B9 (VBUS)
Other:
- sheet RP2040 ports: added EX_BATT_I2C_SCL, EX_BATT_I2C_SDA; removed none
- moved on the sheet: C?, JP?, R5, R?, TP?

Commit message: sync
Parts:
- removed C? (x2): 1uf, Capacitor_SMD:C_0805_2012Metric, symbol Device:C
- removed Q?: MMBT3904LT1G, Package_TO_SOT_SMD:SOT-23, symbol Simulation_SPICE:NPN
- removed R?: 0, Resistor_SMD:R_0805_2012Metric_Pad1.20x1.40mm_HandSolder, symbol Device:R
- removed R?: 1k, Capacitor_SMD:C_0603_1608Metric_Pad1.08x0.95mm_HandSolder, symbol Device:R
- removed R?: 10k, Capacitor_SMD:C_0603_1608Metric_Pad1.08x0.95mm_HandSolder, symbol Device:R
- removed TP? (x2): TestPoint ks, footprints:KEYSTONE_5015, symbol Connector:TestPoint
- removed TP?: TestPoint, TestPoint:TestPoint_Pad_D1.0mm, symbol Connector:TestPoint_Small
- removed U?: AP2112K-3.3, Package_TO_SOT_SMD:SOT-23-5, symbol Regulator_Linear:AP2112K-3.3
- added TP10, TP9: ~, symbol Connector:TestPoint
Connections:
- net USB_C.D+: now also TP9.1
- net USB_C.D-: now also TP10.1
- net USB_C_VBUS renamed USB_C_VBUS_5V
Other:
- sheet RP2040 ports: added PRIMARY_POWER_SUPPLY_DISABLE, USB_C{D- D+}; removed PRIMARY_POWER_SUPPLY_ENABLE
- sheet Voltage Converters ports: added 5.1V_PRIMARY_OUTPUT; removed 5.1V_BUCK_OUTPUT
- note removed: "3V3 LDO"
- moved on the sheet: R15, R8, SB3, TP4, TP5, TP6, USB

Commit message: sync
Parts:
- gave numbers to parts that had none: 5
- renumbered USB to USB1
Other:
- added sheet WSPR Transmitter (wspr_transmitter.kicad_sch)
- sheet Power Input ports: added none; removed batt_ext_3V3
- sheet RP2040 ports: added none; removed RP2080_3V3_VCC

Commit message: sync
Other:
- removed sheet WSPR Transmitter
- sheet RP2040 ports: added 2040_I2C0_WSPR{SDA SCL}; removed none
Changed lines of the file:
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@@
+		)
+	)
+	(bus
+		(pts
+			(xy 186.69 86.36) (xy 198.12 86.36)
+		)
+		(stroke
+			(width 0)
+			(type default)
 		)
 	)
@@
 			)
 		)
+		(pin "2040_I2C0_WSPR{SDA SCL}" bidirectional
+			(at 186.69 86.36 0)
+			(effects
+				(font
+					(size 1.27 1.27)
+				)
+				(justify right)
+			)
+		)
 		(instances
 			(project "power_board"
@@
 				)
 			)
-		)
-	)
-	(sheet
-		(at 218.44 83.82)
-		(size 31.75 21.59)
-		(exclude_from_sim no)
-		(in_bom yes)
-		(on_board yes)
-		(dnp no)
-		(fields_autoplaced yes)
-		(stroke
-			(width 0.1524)
-			(type solid)
-		)
-		(fill
-			(color 0 0 0 0.0000)
-		)
-		(property "Sheetname" "WSPR Transmitter"
-			(at 218.44 83.1084 0)
-			(effects
-				(font
-					(size 1.27 1.27)
-				)
-				(justify left bottom)
-			)
-		)
-		(property "Sheetfile" "wspr_transmitter.kicad_sch"
-			(at 218.44 105.9946 0)
-			(effects
-				(font
-					(size 1.27 1.27)
-				)
-				(justify left top)
-			)
-		)
-		(instances
-			(project "power_board"
-				(path "/8b6d32d3-7736-4ef0-bfd7-9f676eec710d"
-					(page "5")
-				)
-			)

Commit message: sync
Other:
- sheet Voltage Converters renamed Main Power Supply
- sheet Main Power Supply: file 5V_buck_converter.kicad_sch -> main_power_supply.kicad_sch
Changed lines of the file:
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@@
 			(color 0 0 0 0.0000)
 		)
-		(property "Sheetname" "Voltage Converters"
+		(property "Sheetname" "Main Power Supply"
 			(at 143.51 26.035 0)
 			(effects
@@
 			)
 		)
-		(property "Sheetfile" "5V_buck_converter.kicad_sch"
+		(property "Sheetfile" "main_power_supply.kicad_sch"
 			(at 142.875 29.845 0)
 			(effects

Commit message: sync
Parts:
- removed J5: PI, giraffe_flight_computer_footprints:pi_zero, symbol giraffe_symbols:pi_zero
- added J8: ~, symbol keystone_symbols:Backplane Connector
Connections:
- net GND: now also J8.1 (GND)
- new net +3V3_KS: J8. (IO4)
- new net +5V_KS: J8. (IO4)
- new net KS_BACKPLANE.I2C_SCL: J8. (IO4)
- new net KS_BACKPLANE.I2C_SDA: J8. (IO4)
- new net KS_BACKPLANE.IO3: J8. (IO4)
- new net KS_BACKPLANE.IO4: J8. (IO4)
- no-connect marks 26 -> 0
Other:
- added sheet External IO (external_io.kicad_sch)
- sheet RP2040 ports: added KS_BACKPLANE_IO{I2C_SCL I2C_SDA IO3 IO4}; removed none
- note added: "Board Stack Connector"
- note added: "This board is responsible for controling and providing reliable power to this connector. The FC also talks to the RP2040 through this connector. Extra IO was provided to support future boards."
- note removed: "LED"
- note removed: "Raspberry Pi Zero 2"
- moved on the sheet: C21, C4, JP3, R20, R5, SB1, SB2, TP11, TP4

Commit message: sync
Parts:
- removed R15, R8: 5.1kΩ, symbol Device:R
- removed SB3: ~, symbol Jumper:SolderJumper_2_Open
- removed TP10, TP5, TP6, TP9: ~, symbol Connector:TestPoint
- removed USB1: USB_C_Receptacle_USB2.0_14P, symbol a_giraffe_symbols:USB_C_Receptacle_USB2.0_14P
Other:
- sheet Main Power Supply ports: added 5V_KS_ENABLE_GPIO; removed 3V3_PRIMARY_OUTPUT, BUCK_CONVERTER_DISABLE
