File: hardware/power_board/external_io.kicad_sch (KiCad schematic)
At the start: 0 parts

Commit message: sync
Parts:
- added JP4: ~, Connector_PinHeader_2.54mm:PinHeader_1x02_P2.54mm_Vertical, symbol Jumper:Jumper_2_Open
- added R15, R8: 5.1kΩ, symbol Device:R
- added SB3: ~, symbol Jumper:SolderJumper_2_Open
- added TP10, TP5, TP6, TP9: ~, symbol Connector:TestPoint
- added USB1: USB_C_Receptacle_USB2.0_14P, symbol a_giraffe_symbols:USB_C_Receptacle_USB2.0_14P
Connections:
- new net: R15.1, TP6.1, USB1.A5 (CC1)
- new net: R8.1, TP5.1, USB1.B5 (CC2)
- new net: SB3.2 (B), USB1.S1 (SHIELD)
- new net GND: R15.2, R8.2, SB3.1 (A), USB1.A1 (GND), USB1.A12 (GND), USB1.B1 (GND), USB1.B12 (GND)
- new net USB_C.D+: TP9.1, USB1.A6 (D+), USB1.B6 (D+)
- new net USB_C.D-: TP10.1, USB1.A7 (D-), USB1.B7 (D-)
- new net USB_C_VBUS_5V: JP4.1 (A), USB1.A4 (VBUS), USB1.A9 (VBUS), USB1.B4 (VBUS), USB1.B9 (VBUS)

Commit message: sync complete hardware
Connections:
- net +5V_KS: now reaches JP4.2 (B)
Changed lines of the file:
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@@
 	(generator_version "9.0")
 	(paper "A")
-	(text_box "There is no USB isolation, this port is\nmainly for development."
+	(text_box "There is no USB isolation, this port is mainly for development. JP4 can only be bridged if other components are missing.\n"
 		(exclude_from_sim no)
-		(at 96.52 38.1 0)
-		(size 24.13 8.89)
+		(at 115.57 15.24 0)
+		(size 24.13 13.97)
 		(margins 0.9525 0.9525 0.9525 0.9525)
 		(stroke
@@
 	(wire
 		(pts
+			(xy 110.49 21.59) (xy 110.49 24.13)
+		)
+		(stroke
+			(width 0)
+			(type default)
+		)
+	)
+	(wire
+		(pts
 			(xy 63.5 36.83) (xy 64.77 36.83)
 		)
@@
 		(pts
 			(xy 64.77 39.37) (xy 63.5 39.37)
+		)
+		(stroke
+			(width 0)
+			(type default)
+		)
+	)
+	(wire
+		(pts
+			(xy 110.49 24.13) (xy 102.87 24.13)
 		)
 		(stroke
@@
 					(unit 1)
 				)
+			)
+		)
+	)
+	(symbol
+		(lib_id "keystone_symbols:+5V_KS")
+		(at 110.49 21.59 0)
+		(unit 1)
+		(exclude_from_sim no)
+		(in_bom yes)
+		(on_board yes)
+		(dnp no)
+		(property "Reference" "#PWR074"
+			(at 110.49 25.4 0)
+			(effects
+				(font
+					(size 1.27 1.27)
+				)
+				(hide yes)
+			)
+		)
+		(property "Value" "+5V_KS"
+			(at 110.49 17.78 0)
+			(effects
+				(font
+					(size 1.27 1.27)
+				)
+			)
+		)
+		(property "Footprint" ""
+			(at 110.49 21.59 0)
+			(effects
+				(font
+					(size 1.27 1.27)
+				)
+				(hide yes)
+			)
+		)
+		(property "Datasheet" ""
+			(at 110.49 21.59 0)
+			(effects
+				(font
+					(size 1.27 1.27)
+				)
+				(hide yes)
+			)
+		)
+		(property "Description" "Power symbol creates a global label with name {dblquote}+5V_KS{dblquote}. This is the 5V supply that is controlled by the power supply board."
+			(at 110.49 21.59 0)
+			(effects
+				(font
+					(size 1.27 1.27)
+				)
+				(hide yes)
+			)
+		)
+		(pin "1"
+		)
+		(instances
+			(project "power_board"
+				(path "/8b6d32d3-7736-4ef0-bfd7-9f676eec710d/bb6c7426-de14-407d-8e70-f65bc2207c4b"
+					(reference "#PWR074")
+					(unit 1)
+				)
