File: hardware/power_board/main_power_supply.kicad_sch (KiCad schematic)
At the start: 34 parts, among them Q2 MMBT3904LT1G, U2 AP2112K-3.3, U4 TPS54302DDCR

Commit message: sync
Changed lines of the file:
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@@
 		)
 	)
-	(text_box "TODO: Some kind of voltage output protection?"
+	(text_box "TODO: Some kind of voltage output protection? Bleed resistor for USB-C backpower noise?"
 		(exclude_from_sim no)
-		(at 223.52 31.75 0)
-		(size 16.51 8.89)
+		(at 201.93 21.59 0)
+		(size 27.94 8.89)
 		(margins 0.9525 0.9525 0.9525 0.9525)
 		(stroke
 			(width 0)
-			(type default)
+			(type solid)
 		)
 		(fill
@@
 			)
 			(justify left bottom)
+		)
+	)
+	(text_box "The main power supply is currently fairly simple, future versions should\ninvestigate redundancy options.\n\nMain details:\n+Protected battery input\n+5V & 3V control IO (High = disable power supply)\n- 3V3 @ 1A Continuous Output for the RP2040\n- 5V @ 3A and 3V3 @ 1A Controlled Outputs (Default On)"
+		(exclude_from_sim no)
+		(at 12.7 12.7 0)
+		(size 50.8 25.4)
+		(margins 0.9525 0.9525 0.9525 0.9525)
+		(stroke
+			(width 0)
+			(type solid)
+		)
+		(fill
+			(type none)
+		)
+		(effects
+			(font
+				(size 1.27 1.27)
+			)
+			(justify left top)
 		)
 	)
@@
 		(property "Netclass" "POWER:3V3"
 			(at 132.588 142.24 0)
+			(effects
+				(font
+					(size 1.27 1.27)
+					(italic yes)
+				)
+				(justify left)
+			)
+		)
+	)
+	(netclass_flag ""
+		(length 2.54)
+		(shape round)
+		(at 210.82 152.4 0)
+		(fields_autoplaced yes)
+		(effects
+			(font
+				(size 1.27 1.27)
+				(color 194 0 0 1)
+			)
+			(justify left bottom)
+		)
+		(property "Netclass" "POWER:3V3"
+			(at 211.328 149.86 0)
 			(effects
 				(font
@@
 			(effects
 				(font
-					(size 1.27 1.27)
-					(italic yes)
-				)
-				(justify left)
-			)
-		)
-	)
-	(netclass_flag ""
-		(length 2.54)
-		(shape round)
-		(at 210.82 152.4 0)
-		(fields_autoplaced yes)
-		(effects
-			(font
-				(size 1.27 1.27)
-				(color 194 0 0 1)
-			)
-			(justify left bottom)
-		)
-		(property "Netclass" "POWER:3V3_2040"
-			(at 211.328 149.86 0)
-			(effects
-				(font

Commit message: sync
Parts:
- removed C18, C20: 1uf, Capacitor_SMD:C_0805_2012Metric, symbol Device:C
- removed Q2: MMBT3904LT1G, Package_TO_SOT_SMD:SOT-23, symbol Simulation_SPICE:NPN
- removed R12: 0Ω, symbol Device:R
- removed R17: 10k, Capacitor_SMD:C_0603_1608Metric_Pad1.08x0.95mm_HandSolder, symbol Device:R
- removed R18: 1k, Capacitor_SMD:C_0603_1608Metric_Pad1.08x0.95mm_HandSolder, symbol Device:R
- removed R19: 0, Resistor_SMD:R_0805_2012Metric_Pad1.20x1.40mm_HandSolder, symbol Device:R
- removed TP3: TestPoint, TestPoint:TestPoint_Pad_D1.0mm, symbol Connector:TestPoint_Small
- removed TP7, TP8: TestPoint ks, footprints:KEYSTONE_5015, symbol Connector:TestPoint
- removed U2: AP2112K-3.3, Package_TO_SOT_SMD:SOT-23-5, symbol Regulator_Linear:AP2112K-3.3
- added C48: 10uf, Capacitor_SMD:C_1206_3216Metric, symbol Device:C_Small
- added C49, C50, C51: 1uf, symbol Device:C_Small
- added C52: 0.1uf, symbol Device:C_Small
- added R29: 10kΩ, Resistor_SMD:R_0603_1608Metric, symbol Device:R
- added TP17, TP18, TP19, TP20, TP21: TestPoint, TestPoint:TestPoint_Pad_D1.0mm, symbol Connector:TestPoint
- added U2: AP22814AW5, Package_TO_SOT_SMD:SOT-23-5, symbol Power_Management:AP22814AW5
- added U3: TLV75533PDBV, Package_TO_SOT_SMD:SOT-23-5, symbol Regulator_Linear:TLV75533PDBV
Connections:
- net 3V3_RP2040_OUTPUT: now also C50.2, TP17.1, U3.5 (OUT)
- net GND: now also C48.1, C49.1, C50.1, C51.1, C52.1, U2.2 (GND), U3.2 (GND)
- net buck_boot: now also TP21.1
- net 5.1V_PRIMARY_OUTPUT renamed 5V_BUS_CONSTANT
- net 5V_BUS_CONSTANT: now also C48.2, C49.2, C51.2, U2.5 (IN), U3.1 (IN), U3.3 (EN)
- new net 3V3_RP2040: R29.1
- new net 5.1V_CONTROLLED_OUTPUT: C52.2, TP18.1, U2.1 (OUT)
- new net 5V_CONTROLED_FAULT_FLAG: R29.2, TP19.1, U2.3 (~{FLG})
- new net 5V_KS_ENABLE_GPIO: TP20.1, U2.4 (EN)
Other:
- note added: "5.1V (Pi Zero Hat Spec)"
- note added: "5.1V Controlled Output"
- note added: "RP2040 3V3 LDO"
- note added: "https://datasheets.raspberrypi.com/hat/hat-plus-specification.pdf"
- note removed: "3V3 LDO"
- note removed: "5.1 V OUTPUT https://datasheets.raspberrypi.com/hat/hat-plus-specification.pdf"
- moved on the sheet: C30, C31, C32, TP12

Commit message: sync complete hardware
Connections:
- net 5V_CONTROLED_FAULT_FLAG renamed 5V_CONTROLED_FAULT_GPIO
Changed lines of the file:
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@@
 		)
 	)
-	(hierarchical_label "5V_CONTROLED_FAULT_FLAG"
+	(hierarchical_label "5V_CONTROLED_FAULT_GPIO"
 		(shape output)
 		(at 129.54 148.59 0)
