File: hardware/power_board/power_input.kicad_sch (KiCad schematic)
At the start: 23 parts, among them J1 XT30-PW, J2 5019390400, Q1 ?, U1 INA180A

Commit message: sync
Parts:
- BC1: Unit Price (none) -> 0.60; now not fitted
- BT1, BT2, BT3, BT4: Unit Price (none) -> 5.99
- J2: value 5019390400 -> 5019530405
- U1: footprint (none) -> Package_TO_SOT_SMD:SOT-23-5; Unit Price (none) -> 0.90
Changed lines of the file:
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@@
 	)
 	(hierarchical_label "batt_ext_I2C_SCL"
-		(shape bidirectional)
+		(shape input)
 		(at 242.57 44.45 0)
 		(effects
@@
 		(in_bom yes)
 		(on_board no)
-		(dnp no)
+		(dnp yes)
 		(property "Reference" "BC1"
 			(at 68.58 33.02 0)
@@
 			)
 		)
+		(property "BOARD" ""
+			(at 66.04 35.56 0)
+			(effects
+				(font
+					(size 1.27 1.27)
+				)
+			)
+		)
+		(property "Unit Price" "0.60"
+			(at 66.04 35.56 0)
+			(effects
+				(font
+					(size 1.27 1.27)
+				)
+			)
+		)
 		(pin "2"
 		)
@@
 				)
 				(hide yes)
+			)
+		)
+		(property "BOARD" ""
+			(at 175.26 49.53 0)
+			(effects
+				(font
+					(size 1.27 1.27)
+				)
 			)
 		)
@@
 			)
 		)
-		(property "Description" "Single-cell battery"
+		(property "Description" "3500 mAh 18650 w/o protection"
 			(at 43.18 53.34 0)
 			(effects
@@
 			)
 		)
-		(property "Unit Price" ""
+		(property "Unit Price" "5.99"
 			(at 43.18 53.34 0)
 			(effects
@@
 				)
 				(hide yes)
+			)
+		)
+		(property "BOARD" ""
+			(at 43.18 53.34 0)
+			(effects
+				(font
+					(size 1.27 1.27)
+				)
 			)
 		)
@@
 			)
 		)
+		(property "BOARD" ""
+			(at 208.28 69.85 0)
+			(effects
+				(font
+					(size 1.27 1.27)
+				)
+			)
+		)
 		(pin "2"
 		)
@@
 			)
 		)
+		(property "BOARD" ""
+			(at 156.21 52.07 0)
+			(effects
+				(font
+					(size 1.27 1.27)
+				)
+			)
+		)
 		(pin "2"
 		)
@@
 				)
 				(hide yes)
+			)
+		)
+		(property "BOARD" ""
+			(at 142.24 49.53 0)
+			(effects
+				(font
+					(size 1.27 1.27)
+				)
 			)
 		)
@@
 			)
 		)
+		(property "BOARD" ""
+			(at 208.28 80.01 0)
+			(effects
+				(font
+					(size 1.27 1.27)
+				)
+			)
+		)
 		(pin "2"
 		)
@@
 			)
 		)
+		(property "BOARD" ""
+			(at 38.1 157.48 0)
+			(effects
+				(font
+					(size 1.27 1.27)
+				)
+			)
+		)
 		(pin "1"
 		)
@@
 			)
 		)
+		(property "BOARD" ""
+			(at 156.21 39.37 0)
+			(effects
+				(font
+					(size 1.27 1.27)
+				)
+			)
+		)
 		(pin "2"
 		)
@@
 				)
 				(justify left)
+			)
+		)
+		(property "BOARD" ""
+			(at 156.21 68.58 0)
+			(effects
+				(font
+					(size 1.27 1.27)
+				)
 			)
 		)
@@
 			)
 		)
+		(property "BOARD" ""
+			(at 57.15 139.7 0)
+			(effects
+				(font
+					(size 1.27 1.27)
+				)
+			)
+		)
 		(pin "1"
 		)
@@
 			)
 		)
-		(property "Description" "Molex Pico-Clasp"
+		(property "Description" "Molex Pico-Clasp Connector"
 			(at 70.485 80.645 0)
 			(effects
@@
 				)
 				(justify left)
+			)
+		)
+		(property "BOARD" ""
+			(at 68.58 78.74 0)
+			(effects
+				(font
+					(size 1.27 1.27)
+				)
 			)
 		)
@@
 			)
 		)
-		(property "Description" "Single-cell battery"
+		(property "Description" "3500 mAh 18650 w/o protection"
 			(at 43.18 40.64 0)
 			(effects
@@
 			)
 		)
-		(property "Unit Price" ""
+		(property "Unit Price" "5.99"
 			(at 43.18 40.64 0)
 			(effects
@@
 				)
 				(hide yes)
+			)
+		)
+		(property "BOARD" ""
+			(at 43.18 40.64 0)
+			(effects
+				(font
+					(size 1.27 1.27)
+				)
 			)
 		)
@@
 			)
 		)
+		(property "BOARD" ""
+			(at 119.38 52.07 0)
+			(effects
+				(font
+					(size 1.27 1.27)
+				)
+			)
+		)
 		(pin "2"
 		)
@@
 				)
 				(justify left)
+			)
+		)
+		(property "BOARD" ""
+			(at 52.07 125.73 0)
+			(effects
+				(font
+					(size 1.27 1.27)
+				)
 			)
 		)
@@
 			)
 		)
+		(property "BOARD" ""
+			(at 66.04 58.42 0)
+			(effects
+				(font
+					(size 1.27 1.27)
+				)
+			)
+		)
 		(pin "1"
 		)
@@
 			)
 		)
-		(property "Description" "Generic 18650"
+		(property "Description" "3500 mAh 18650"
 			(at 29.845 41.275 0)
 			(effects
@@
 			)
 		)
-		(property "Unit Price" ""
+		(property "Unit Price" "5.99"
 			(at 33.02 40.64 0)
 			(effects
@@
 				)
 				(hide yes)
+			)
+		)
+		(property "BOARD" ""
+			(at 33.02 40.64 0)
+			(effects
+				(font
+					(size 1.27 1.27)
+				)
 			)
 		)
@@
 			)
 		)
-		(property "Description" "Single-cell battery"
+		(property "Description" "3500 mAh 18650 w/o protection"
 			(at 33.02 53.34 0)
 			(effects
@@
 			)
 		)
-		(property "Unit Price" ""
+		(property "Unit Price" "5.99"
 			(at 33.02 53.34 0)
 			(effects
@@
 				)
 				(hide yes)
+			)
+		)
+		(property "BOARD" ""
+			(at 33.02 53.34 0)
+			(effects
+				(font
+					(size 1.27 1.27)
+				)
 			)
 		)
@@
 				)
 				(justify left)
+			)
+		)
+		(property "BOARD" ""
+			(at 62.23 125.73 0)
+			(effects
+				(font
+					(size 1.27 1.27)
+				)
 			)
 		)
@@
 			)
 		)
-		(property "Footprint" ""
+		(property "Footprint" "Package_TO_SOT_SMD:SOT-23-5"
 			(at 38.735 152.4 0)
 			(effects
@@
 			)
 		)
+		(property "BOARD" ""
+			(at 57.15 154.94 0)
+			(effects
+				(font
+					(size 1.27 1.27)
+				)
+			)
+		)
+		(property "Unit Price" "0.90"
+			(at 57.15 154.94 0)
+			(effects
+				(font
+					(size 1.27 1.27)
+				)
+			)
+		)
 		(pin "2"
 		)
@@
 				)
 				(justify right)
+			)
+		)
+		(property "BOARD" ""
+			(at 57.15 114.3 0)
+			(effects
+				(font
+					(size 1.27 1.27)
+				)
 			)
 		)
@@
 			)
 		)
-		(property "Value" "5019390400"
+		(property "Value" "5019530405"
 			(at 215.265 46.355 0)
 			(effects
@@
 				)
 				(justify left)
+			)
+		)
+		(property "BOARD" ""
+			(at 217.17 49.53 0)
+			(effects
+				(font
+					(size 1.27 1.27)
+				)
 			)
 		)
@@
 			)
 		)
+		(property "BOARD" ""
+			(at 168.91 55.88 0)
+			(effects
+				(font
+					(size 1.27 1.27)
+				)
+			)
+		)

Commit message: sync
Connections:
- net batt_ext_3V3 renamed 3V3_RP2040
Changed lines of the file:
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@@
+	)
+	(junction
+		(at 34.29 58.42)
+		(diameter 0)
+		(color 0 0 0 0)
 	)
 	(junction
@@
 	(wire
 		(pts
-			(xy 33.02 58.42) (xy 38.1 58.42)
+			(xy 33.02 58.42) (xy 34.29 58.42)
 		)
 		(stroke
@@
 	(wire
 		(pts
+			(xy 22.86 62.23) (xy 34.29 62.23)
+		)
+		(stroke
+			(width 0)
+			(type default)
+		)
+	)
+	(wire
+		(pts
 			(xy 43.18 33.02) (xy 54.61 33.02)
 		)
@@
 	(wire
 		(pts
+			(xy 229.87 59.69) (xy 238.76 59.69)
+		)
+		(stroke
+			(width 0)
+			(type default)
+		)
+	)
+	(wire
+		(pts
 			(xy 224.79 54.61) (xy 224.79 52.07)
 		)
@@
 	(wire
 		(pts
-			(xy 222.25 49.53) (xy 242.57 49.53)
-		)
-		(stroke
-			(width 0)
-			(type default)
-		)
-	)
-	(wire
-		(pts
 			(xy 208.28 63.5) (xy 177.8 63.5)
 		)
@@
 	(wire
 		(pts
+			(xy 34.29 62.23) (xy 34.29 58.42)
+		)
+		(stroke
+			(width 0)
+			(type default)
+		)
+	)
+	(wire
+		(pts
 			(xy 43.18 45.72) (xy 48.26 45.72)
 		)
@@
 	(wire
 		(pts
-			(xy 222.25 44.45) (xy 242.57 44.45)
+			(xy 222.25 44.45) (xy 240.03 44.45)
 		)
 		(stroke
@@
 	(wire
 		(pts
+			(xy 229.87 49.53) (xy 229.87 59.69)
+		)
+		(stroke
+			(width 0)
+			(type default)
+		)
+	)
+	(wire
+		(pts
+			(xy 222.25 49.53) (xy 229.87 49.53)
+		)
+		(stroke
+			(width 0)
+			(type default)
+		)
+	)
+	(wire
+		(pts
 			(xy 48.26 58.42) (xy 60.96 58.42)
 		)
@@
 	(wire
 		(pts
+			(xy 238.76 59.69) (xy 238.76 57.15)
+		)
+		(stroke
+			(width 0)
+			(type default)
+		)
+	)
+	(wire
+		(pts
 			(xy 177.8 49.53) (xy 181.61 49.53)
 		)
@@
 	(wire
 		(pts
+			(xy 22.86 60.96) (xy 22.86 62.23)
+		)
+		(stroke
+			(width 0)
+			(type default)
+		)
+	)
+	(wire
+		(pts
 			(xy 163.83 39.37) (xy 163.83 49.53)
 		)
@@
 	(wire
 		(pts
-			(xy 222.25 46.99) (xy 242.57 46.99)
+			(xy 222.25 46.99) (xy 240.03 46.99)
+		)
+		(stroke
+			(width 0)
+			(type default)
+		)
+	)
+	(wire
+		(pts
+			(xy 34.29 58.42) (xy 38.1 58.42)
 		)
 		(stroke
@@
 	(hierarchical_label "batt_ext_I2C_SCL"
 		(shape input)
-		(at 242.57 44.45 0)
+		(at 240.03 44.45 0)
 		(effects
 			(font
@@
 		)
 	)
-	(hierarchical_label "batt_ext_3V3"
-		(shape input)
-		(at 242.57 49.53 0)
-		(effects
-			(font
-				(size 1.27 1.27)
-			)
-			(justify left)
-		)
-	)
 	(hierarchical_label "batt_ext_I2C_SDA"
 		(shape bidirectional)
-		(at 242.57 46.99 0)
+		(at 240.03 46.99 0)
 		(effects
 			(font
@@
 	)
 	(symbol
+		(lib_id "power:PWR_FLAG")
+		(at 22.86 60.96 0)
+		(unit 1)
+		(exclude_from_sim no)
+		(in_bom yes)
+		(on_board yes)
+		(dnp no)
+		(property "Reference" "#FLG05"
+			(at 22.86 59.055 0)
+			(effects
+				(font
+					(size 1.27 1.27)
+				)
+				(hide yes)
+			)
+		)
+		(property "Value" "PWR_FLAG"
+			(at 22.86 57.15 0)
+			(effects
+				(font
+					(size 1.27 1.27)
+				)
+			)
+		)
+		(property "Footprint" ""
+			(at 22.86 60.96 0)
+			(effects
+				(font
+					(size 1.27 1.27)
+				)
+				(hide yes)
+			)
+		)
+		(property "Datasheet" "~"
+			(at 22.86 60.96 0)
+			(effects
+				(font
+					(size 1.27 1.27)
+				)
+				(hide yes)
+			)
+		)
+		(property "Description" "Special symbol for telling ERC where power comes from"
+			(at 22.86 60.96 0)
+			(effects
+				(font
+					(size 1.27 1.27)
+				)
+				(hide yes)
+			)
+		)
+		(pin "1"
+		)
+		(instances
+			(project "power_board"
+				(path "/8b6d32d3-7736-4ef0-bfd7-9f676eec710d/37a25529-547a-4c46-9309-80d1f4ca78d2"
+					(reference "#FLG05")
+					(unit 1)
+				)
+			)
+		)
+	)
+	(symbol
 		(lib_id "Jumper:SolderJumper_2_Open")
 		(at 156.21 39.37 0)
@@
 					(unit 1)
 				)
+			)
+		)
+	)
+	(symbol
+		(lib_id "power:+3V3")
+		(at 238.76 57.15 0)
+		(unit 1)
+		(exclude_from_sim no)
+		(in_bom yes)
+		(on_board yes)
+		(dnp no)
+		(property "Reference" "#PWR047"
+			(at 238.76 60.96 0)
+			(effects
+				(font
+					(size 1.27 1.27)
+				)
+				(hide yes)
+			)
+		)
+		(property "Value" "3V3_RP2040"
+			(at 238.76 53.34 0)
+			(effects
+				(font
+					(size 1.27 1.27)
+				)
+			)
+		)
+		(property "Footprint" ""
+			(at 238.76 57.15 0)
+			(effects
+				(font
+					(size 1.27 1.27)
+				)
+				(hide yes)
+			)
+		)
+		(property "Datasheet" ""
+			(at 238.76 57.15 0)
+			(effects
+				(font
+					(size 1.27 1.27)
+				)
+				(hide yes)
+			)
+		)
+		(property "Description" "3V3_RP2040"
+			(at 238.76 57.15 0)
+			(effects
+				(font
+					(size 1.27 1.27)
+				)
+				(hide yes)
+			)
+		)
+		(pin "1"
+		)
+		(instances
+			(project "power_board"
+				(path "/8b6d32d3-7736-4ef0-bfd7-9f676eec710d/37a25529-547a-4c46-9309-80d1f4ca78d2"
+					(reference "#PWR047")
+					(unit 1)
+				)

Commit message: sync
Other:
- note removed: "Upload to pico via debug connection and interface via UART?"
- moved on the sheet: C2, C5, R2, R3, R6, U1

Commit message: sync complete hardware
Parts:
- BC1: now fitted
Connections:
- net 3V3_RP2040 renamed +5V_KS
- net batt_ext_I2C_SCL renamed BATT_EXT_I2C_SCL
- net BATT_EXT_I2C_SCL: no longer J2.4 (Pin_4)
- net batt_ext_I2C_SDA renamed BATT_EXT_I2C_SDA
- net BATT_EXT_I2C_SDA: no longer J2.3 (Pin_3)
- new net KS_BACKPLANE_IO.I2C_SCL: J2.4 (Pin_4)
- new net KS_BACKPLANE_IO.I2C_SDA: J2.3 (Pin_3)
- no-connect marks 3 -> 2
Other:
- moved on the sheet: J2
