File: hardware/power_board/rp2040.kicad_sch (KiCad schematic)
At the start: 11 parts, among them Y1 Crystal_GND24

Commit message: sync
Parts:
- removed C?: 2.2uf, symbol Device:C_Small
- removed C?: 0.1uf, symbol Device:C_Small
- removed J?: Conn_01x03_Socket, symbol Connector:Conn_01x03_Socket
- removed R8: 1KΩ, symbol Device:R
- removed U?: W25Q16JVUXIQ TR, USON-8_UX_2x3x0p6_WIN, symbol a_giraffe_symbols:W25Q16JVUXIQ_TR
- added C10, C11, C14, C15, C6, C7, C8, C9, C?: 0.1uf, Capacitor_SMD:C_0603_1608Metric_Pad1.08x0.95mm_HandSolder, symbol Device:C_Small
- added C12, C13: 1uf, Capacitor_SMD:C_0603_1608Metric_Pad1.08x0.95mm_HandSolder, symbol Device:C_Small
- added C16, C17: DNS, Capacitor_SMD:C_0603_1608Metric_Pad1.08x0.95mm_HandSolder, symbol Device:C_Small
- added C19: 0.1uf, symbol Device:C_Small
- added J3: SD_Card_Device, symbol Connector:SD_Card_Device
- added J4: TC2030, Connector:Tag-Connect_TC2030-IDC-NL_2x03_P1.27mm_Vertical, symbol Connector:TC2030
- added LED1: ~, symbol Device:LED
- added R10: 1kΩ, symbol Device:R
- added R11: 10kΩ, symbol Device:R
- added R13, R14: 27.4Ω, symbol Device:R
- added R16: ?Ω, symbol Device:R
- added U3: W25Q128JVS, Package_SO:SOIC-8_5.3x5.3mm_P1.27mm, symbol Memory_Flash:W25Q128JVS
- U?: Unit Price (none) -> 1.0
- Y1: value Crystal_GND24 -> ABM8-272-T3
Connections:
- net 3V3_PICO: now also U?.1 (IOVDD), U?.10 (IOVDD), U?.22 (IOVDD), U?.33 (IOVDD), U?.42 (IOVDD), U?.43 (ADC_AVDD), U?.44 (VREG_IN), U?.48 (USB_VDD), U?.49 (IOVDD), C10.2, C11.2, C12.2, C19.1, C6.2, C7.2, C8.2, C9.2, C?.2, R11.1, U3.8 (VCC)
- net ADC0_INPUT_VOLTAGE_SIGNAL: now also U?.38 (GPIO26_ADC0), C16.2
- net ADC1_INPUT_CURRENT_SENSE_SIGNAL: now also U?.39 (GPIO27_ADC1), C17.2
- net GND: now also C10.1, C11.1, C12.1, C13.1, C14.1, C15.1, C16.1, C17.1, C19.2, C6.1, C7.1, C8.1, C9.1, C?.1, LED1.1 (K), U3.4 (GND)
- net QSPI_SCLK: now also U3.6 (CLK)
- net QSPI_SD0: now also U3.5 (DI/IO_{0})
- net QSPI_SD1: now also U3.2 (DO/IO_{1})
- net QSPI_SD2: now also U3.3 (~{WP}/IO_{2})
- net QSPI_SD3: now also U3.7 (~{HOLD}/~{RESET}/IO_{3})
- net QSPI_SS: now also R10.2, R11.2, U3.1 (~{CS})
- net at C3.1, R9.1: now also Y1.3; no longer Y1.1
- net at C1.1, U?.20 (XIN): now also Y1.1; no longer Y1.3
- net RP2040_UART_0_TX: now reaches U?.2 (GPIO0)
- net +1V1_PICO_ADC_REF: now reaches U?.23 (DVDD), U?.45 (VREG_VOUT), U?.50 (DVDD)
- net +1V1_PICO_ADC_REF: now also C13.2, C14.2, C15.2
- net RP2040_UART_0_RX: now reaches U?.3 (GPIO1)
- net RP2040_STATUS_LED: now reaches U?.37 (GPIO25)
- net RP2040_STATUS_LED: now also R16.1
- net at U?.46 (USB_DM): now also R14.2
- net at U?.47 (USB_DP): now also R13.2
- net at JP2.2 (B): now also R10.1
- new net: LED1.2 (A), R16.2
- new net: J3.3 (VSS), J3.6 (VSS)
- new net 2040_USB_D+: R13.1
- new net 2040_USB_D-: R14.1
- no-connect marks 1 -> 0
Other:
- note added: "One 0.1uf cap per power input"
- note added: "Place C12 by pin 44"
- note added: "Place C13 by pin 45"
- note added: "https://datasheets.raspberrypi.com/rp2040/hardware-design-with-rp2040.pdf"
- moved on the sheet: C1, C3, JP2, R9, Y1

Commit message: sync
Parts:
- removed J3: SD_Card_Device, symbol Connector:SD_Card_Device
- removed J4: TC2030, Connector:Tag-Connect_TC2030-IDC-NL_2x03_P1.27mm_Vertical, symbol Connector:TC2030
- added J4: Micro_SD_Card, symbol a_giraffe_symbols:Micro_SD_Card
- added SW1: SW_MEC_5G, symbol Switch:SW_MEC_5G
Connections:
- net 3V3_PICO: now also J4.4 (VDD)
- net ADC0_INPUT_VOLTAGE_SIGNAL: now also U?.39 (GPIO27_ADC1); no longer U?.38 (GPIO26_ADC0)
- net ADC1_INPUT_CURRENT_SENSE_SIGNAL: now also U?.40 (GPIO28_ADC2); no longer U?.39 (GPIO27_ADC1)
- net GND: now also J4.6 (VSS), J4.9 (SHIELD), SW1.3 (B), SW1.4 (B)
- net RP2040_RESET_PIN: now reaches U?.26 (RUN)
- net RP2040_RESET_PIN: now also SW1.1 (A), SW1.2 (A)
- net RP2040_SPI0_RX: now reaches U?.27 (GPIO16)
- net RP2040_SPI0_~{CS}: now reaches U?.28 (GPIO17)
- net RP2040_SPI0_SCK: now reaches U?.29 (GPIO18)
- net RP2040_SPI0_TX: now reaches U?.30 (GPIO19)
- net RP2040_I2C_1_SDA: now reaches U?.4 (GPIO2)
- net RP2040_I2C_1_SCL: now reaches U?.5 (GPIO3)
- net RP2040_I2C_0_SDA: now reaches U?.6 (GPIO4)
- net RP2040_I2C_0_SCL: now reaches U?.7 (GPIO5)
- net 2040_USB_D+ renamed USB_C.D+
- net 2040_USB_D- renamed USB_C.D-
- new net SD_CS: J4.2 (DAT3/CD)
- new net SD_DI: J4.3 (CMD)
- no-connect marks 0 -> 2
Other:
- note added: "https://www.electroniccircuitsdesign.com/pinout/sd-microsd-card-pinout.html"
- moved on the sheet: C16, C17

Commit message: sync
Parts:
- added C33: 1uf, Capacitor_SMD:C_0603_1608Metric_Pad1.08x0.95mm_HandSolder, symbol Device:C_Small
- added C34: 10uf, Capacitor_SMD:C_0603_1608Metric_Pad1.08x0.95mm_HandSolder, symbol Device:C_Small
- added J3: 5019530305, symbol Connector_Generic:Conn_01x03
Connections:
- net 3V3_PICO: now also C33.2, C34.2
- net GND: now also U?.19 (TESTEN), C33.1, C34.1, J3.1 (Pin_1)
- net RP2040_I2C_0_SCL: now also U?.16 (GPIO13); no longer U?.7 (GPIO5)
- net RP2040_I2C_0_SDA: now also U?.15 (GPIO12); no longer U?.6 (GPIO4)
- net RP2040_SPI1_RX: now reaches U?.11 (GPIO8)
- net RP2040_SPI1_~{CS}: now reaches U?.12 (GPIO9)
- net RP2040_SPI1_SCK: now reaches U?.13 (GPIO10)
- net RP2040_SPI1_TX: now reaches U?.14 (GPIO11)
- net RP2040_SWCLK: now reaches U?.24 (SWCLK)
- net RP2040_SWCLK: now also J3.3 (Pin_3)
- net RP2040_SWDIO: now reaches U?.25 (SWD)
- net RP2040_SWDIO: now also J3.2 (Pin_2)
- net RP2040_UART_0_RX renamed 2040_UART0.RX
- net RP2040_UART_0_TX renamed 2040_UART0.TX
- new net RP2040_UART_1_RX: U?.7 (GPIO5)
- new net RP2040_UART_1_TX: U?.6 (GPIO4)
- no-connect marks 2 -> 4

Commit message: sync
Parts:
- removed LED1: ~, symbol Device:LED
- removed U3: W25Q128JVS, Package_SO:SOIC-8_5.3x5.3mm_P1.27mm, symbol Memory_Flash:W25Q128JVS
- added C47: 2.2uf, Capacitor_SMD:C_0603_1608Metric_Pad1.08x0.95mm_HandSolder, symbol Device:C_Small
- added D2: LED, symbol Device:LED
- added Q3: BC847CT, Package_TO_SOT_SMD:SOT-23, symbol a_giraffe_symbols:BC847AT
- added R26, R27, R28: ?Ω, symbol Device:R
- added U8: W25Q16JVUXIQ TR, USON-8_UX_2x3x0p6_WIN, symbol a_giraffe_symbols:W25Q16JVUXIQ_TR
- C19: footprint (none) -> Capacitor_SMD:C_0603_1608Metric_Pad1.08x0.95mm_HandSolder; Size (none) -> 0603
- SW1: now not fitted
- gave numbers to parts that had none: 2
Connections:
- net RP2040_SPI0_RX is gone; now on net RP2040_SPI0_RX SD_DO: U5.27 (GPIO16)
- net RP2040_SPI0_SCK is gone; now on net RP2040_SPI0_SCK SD_SCLK: U5.29 (GPIO18)
- net SD_CS is gone; now on net RP2040_SPI0_~{CS} SD_CS: J4.2 (DAT3/CD)
- net SD_DI is gone; now on net RP2040_SPI0_TX SD_DI: J4.3 (CMD)
- net 3V3_PICO: now also C19.2, C47.2, D2.2 (A), R27.1, R28.1, U8.8 (VCC); no longer C19.1
- net ADC0_INPUT_VOLTAGE_SIGNAL: now also U5.40 (GPIO28_ADC2); no longer U5.39 (GPIO27_ADC1)
- net ADC1_INPUT_CURRENT_SENSE_SIGNAL: now also U5.41 (GPIO29_ADC3); no longer U5.40 (GPIO28_ADC2)
- net GND: now also C19.1, C47.1, Q3.2 (E), U8.4 (GND); no longer C19.2
- net PRIMARY_POWER_SUPPLY_DISABLE: now also U5.17 (GPIO14)
- net QSPI_SCLK: now also U8.6 (CLK)
- net QSPI_SD0: now also U8.5 (DI(IO0))
- net QSPI_SD1: now also U8.2 (DO(IO1))
- net QSPI_SD2: now also U8.3 (/WP(IO2))
- net QSPI_SD3: now also U8.7 (RESET(IO3))
- net QSPI_SS: no longer R10.2, R11.2
- net at R16.2: now also Q3.1 (B)
- net HW_ID: now reaches U5.38 (GPIO26_ADC0)
- net RP2040_SPI0_SCK SD_SCLK: now reaches J4.5 (CLK)
- net RP2040_SPI0_RX SD_DO: now reaches J4.7 (DAT0)
- net RP2040_I2C_0_SCL renamed 2040_I2C0_WSPR.SCL
- net 2040_I2C0_WSPR.SCL: now also R27.2
- net RP2040_I2C_0_SDA renamed 2040_I2C0_WSPR.SDA
- net 2040_I2C0_WSPR.SDA: now also R28.2
- net RP2040_I2C_1_SCL renamed 2040_I2C1.SCL
- net RP2040_I2C_1_SDA renamed 2040_I2C1.SDA
- net RP2040_SPI0_TX renamed RP2040_SPI0_TX SD_DI
- net RP2040_SPI0_~{CS} renamed RP2040_SPI0_~{CS} SD_CS
- net RP2040_SPI1_RX renamed 2040_SPI1.RX
- net RP2040_SPI1_SCK renamed 2040_SPI1.SCK
- net RP2040_SPI1_TX renamed 2040_SPI1.TX
- net RP2040_SPI1_~{CS} renamed 2040_SPI1.~{CS}
- net RP2040_UART_1_RX renamed 2040_UART1.RX
- net RP2040_UART_1_TX renamed 2040_UART1.TX
- new net: R10.2, R11.2, U8.1 (/CS)
- new net: D2.1 (K), R26.1
- new net: Q3.3 (C), R26.2
- no-connect marks 4 -> 12
Other:
- added sheet WSPR Transmitter (wspr_transmitter.kicad_sch)
- note added: "BOOTSEL Jumper"
- note added: "Optional I2C0 Pullups"
- note added: "https://www.electroniccircuitsdesign.com/pinout/sd-microsd-card-pinout.html https://youtu.be/JrYT7aJnP_I"
- note removed: "https://www.electroniccircuitsdesign.com/pinout/sd-microsd-card-pinout.html"
- moved on the sheet: C1, C10, C11, C12, C13, C14, C15, C16, C17, C3, C33, C34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

Commit message: sync
Parts:
- D2: value LED -> 0603 Green; footprint (none) -> LED_SMD:LED_0603_1608Metric
- R16, R26: footprint (none) -> Resistor_SMD:R_0603_1608Metric
Connections:
- net 3V3_PICO: no longer D2.2 (A)
- net GND: now also D2.1 (K); no longer Q3.2 (E)
- net at R26.1: now also Q3.2 (E); no longer D2.1 (K)
- net at R26.2: now also D2.2 (A); no longer Q3.3 (C)
- new net 3V3_RP2040: Q3.3 (C)
Other:
- note added: "RP2040 Status LED"
- note added: "https://electronics.stackexchange.com/a/151328"
- moved on the sheet: C19, C47, D2, JP2, Q3, R10, R11, R16, R26, U8

Commit message: sync
Connections:
- net 2040_I2C0_WSPR.SDA renamed WSPR.SDA
Other:
- sheet WSPR Transmitter ports: added WSPR{SDA SCL}; removed 2040_I2C0_WSPR{SDA SCL}
- note added: "I2C0 SCL"
- note added: "I2C0 SDA"
- moved on the sheet: R27, R28

Commit message: sync complete hardware
Parts:
- removed J4: Micro_SD_Card, symbol a_giraffe_symbols:Micro_SD_Card
- removed R10: 1kΩ, symbol Device:R
- added R12: 1kΩ, symbol Device:R
Connections:
- net 2040_I2C1.SDA is gone; now on net WSPR.SDA: U5.4 (GPIO2)
- net 3V3_PICO: no longer C10.2, C11.2, C12.2, C19.2, C33.2, C34.2, C35.2, C47.2, C6.2, C7.2, C8.2, C9.2, R11.1, U5.1 (IOVDD), U5.10 (IOVDD), U5.22 (IOVDD), U5.33 (IOVDD), U5.42 (IOVDD), U5.43 (ADC_AVDD), U5.44 (VREG_IN), U5.48 (USB_VDD), U5.49 (IOVDD), U8.8 (VCC)
- net 3V3_RP2040: now also C10.2, C11.2, C12.2, C19.2, C33.2, C34.2, C35.2, C47.2, C6.2, C7.2, C8.2, C9.2, R11.1, U5.1 (IOVDD), U5.10 (IOVDD), U5.22 (IOVDD), U5.33 (IOVDD), U5.42 (IOVDD), U5.43 (ADC_AVDD), U5.44 (VREG_IN), U5.48 (USB_VDD), U5.49 (IOVDD), U8.8 (VCC)
- net QSPI_SS: now also R11.2, U8.1 (/CS), R12.1
- net WSPR.SDA: no longer U5.15 (GPIO12)
- net 5V_CONTROLED_FAULT_GPIO: now reaches U5.18 (GPIO15)
- net WSPR_POWER_ENABLE: now reaches U5.8 (GPIO6)
- net WSPR_POWER_FAULT: now reaches U5.9 (GPIO7)
- net at JP2.2 (B): now also R12.2
- net 2040_I2C0_WSPR.SCL renamed KS_BACKPLANE_IO.I2C_SCL
- net KS_BACKPLANE_IO.I2C_SCL: no longer R27.2
- net 2040_I2C1.SCL renamed WSPR.SCL
- net WSPR.SCL: now also R27.2
- net HW_ID renamed HW_ID_ADC
- net PRIMARY_POWER_SUPPLY_DISABLE renamed 5V_KS_ENABLE_GPIO
- net RP2040_SPI0_RX SD_DO renamed SD_SPI0.RX
- net RP2040_SPI0_SCK SD_SCLK renamed SD_SPI0.SCK
- net RP2040_SPI0_TX SD_DI renamed SD_SPI0.TX
- net RP2040_SPI0_~{CS} SD_CS renamed SD_SPI0.~{CS}
- new net KS_BACKPLANE_IO.I2C_SDA: U5.15 (GPIO12)
- no-connect marks 12 -> 7
Other:
- added sheet RP2040 SD Card (rp2040_sd_card.kicad_sch)
- note added: "SPI0 CS/SD CS"
- note added: "SPI0 RX/SD DO"
- note added: "SPI0 SCK/SD SCLK"
- note added: "SPI0 TX/SD DI"
- moved on the sheet: C19, C47, JP2, R11, R27, R28, U8
